Commit message: converted to xacro

File: huron_description/urdf/huron_visuals.xacro (robot description, xacro)
@@ -8,7 +8,5 @@
             <mesh filename="package://huron_description/meshes/base_link.STL" scale="1 1 1" />
         </geometry>
-        <material name="">
-            <color rgba="0.75294 0.75294 0.75294 1" />
-        </material>
+        <material name="grey"/>
     </xacro:macro>
     <!-- left hip yaw link -->
@@ -18,7 +16,5 @@
             <mesh filename="package://huron_description/meshes/l_hip_yaw_link.STL" scale="1 1 1" />
         </geometry>
-        <material name="">
-            <color rgba="0.75294 0.75294 0.75294 1" />
-        </material>
+        <material name="grey"/>
     </xacro:macro>
     <!-- left hip roll link -->
@@ -28,7 +24,5 @@
             <mesh filename="package://huron_description/meshes/l_hip_roll_link.STL" scale="1 1 1" />
         </geometry>
-        <material name="">
-            <color rgba="0.75294 0.75294 0.75294 1" />
-        </material>
+        <material name="grey"/>
     </xacro:macro>
     <!-- left hip pitch link -->
@@ -38,7 +32,5 @@
             <mesh filename="package://huron_description/meshes/l_hip_pitch_link.STL" scale="1 1 1" />
         </geometry>
-        <material name="">
-            <color rgba="0.75294 0.75294 0.75294 1" />
-        </material>
+        <material name="grey"/>
     </xacro:macro>
     <!-- left knee pitch link -->
@@ -48,7 +40,5 @@
             <mesh filename="package://huron_description/meshes/l_knee_pitch_link.STL" scale="1 1 1" />
         </geometry>
-        <material name="">
-            <color rgba="0.75294 0.75294 0.75294 1" />
-        </material>
+        <material name="grey"/>
     </xacro:macro>
     <!-- left ankle pitch link -->
@@ -72,4 +62,5 @@
         </material>
     </xacro:macro>
+    <?comment
     <!-- l1_foot_ft link -->
     <xacro:macro name="insert_mesh_l1_foot_ft_link">
@@ -104,9 +95,10 @@
         <material name="grey"/>
     </xacro:macro>
+        ?>
     <!-- right hip yaw link -->
     <xacro:macro name="insert_mesh_r_hip_yaw_link">
         <origin xyz="0 0 0" rpy="0 0 0" />
         <geometry>
-            <mesh filename="package://uthai_description/meshes/r_hip_yaw.STL" scale="1 1 1" />
+            <mesh filename="package://huron_description/meshes/r_hip_yaw_link.STL" scale="1 1 1" />
         </geometry>
         <material name="grey"/>
@@ -116,5 +108,5 @@
         <origin xyz="0 0 0" rpy="0 0 0" />
         <geometry>
-            <mesh filename="package://uthai_description/meshes/r_hip_roll.STL" scale="1 1 1" />
+            <mesh filename="package://huron_description/meshes/r_hip_roll_link.STL" scale="1 1 1" />
         </geometry>
         <material name="grey"/>
@@ -124,5 +116,5 @@
         <origin xyz="0 0 0" rpy="0 0 0" />
         <geometry>
-            <mesh filename="package://uthai_description/meshes/r_hip_pitch.STL" scale="1 1 1" />
+            <mesh filename="package://huron_description/meshes/r_hip_pitch_link.STL" scale="1 1 1" />
         </geometry>
         <material name="grey"/>
@@ -132,5 +124,5 @@
         <origin xyz="0 0 0" rpy="0 0 0" />
         <geometry>
-            <mesh filename="package://uthai_description/meshes/r_knee_pitch.STL" scale="1 1 1" />
+            <mesh filename="package://huron_description/meshes/r_knee_pitch_link.STL" scale="1 1 1" />
         </geometry>
         <material name="grey"/>
@@ -140,7 +132,9 @@
         <origin xyz="0 0 0" rpy="0 0 0" />
         <geometry>
-            <mesh filename="package://uthai_description/meshes/r_ankle_pitch.STL" scale="1 1 1" />
+            <mesh filename="package://huron_description/meshes/r_ankle_pitch_link.STL" scale="1 1 1" />
         </geometry>
-        <material name="grey"/>
+        <material name="">
+            <color rgba="0.77647 0.75686 0.73725 1" />
+        </material>
     </xacro:macro>
     <!-- right ankle roll link -->
@@ -148,39 +142,44 @@
         <origin xyz="0 0 0" rpy="0 0 0" />
         <geometry>
-            <mesh filename="package://uthai_description/meshes/r_ankle_roll.STL" scale="1 1 1" />
+            <mesh filename="package://huron_description/meshes/r_ankle_roll_link.STL" scale="1 1 1" />
         </geometry>
-        <material name="grey"/>
+        <material name="">
+            <color rgba="0.77647 0.75686 0.73725 1" />
+        </material>
     </xacro:macro>
+    <!-- Right foot sensors -->
+    <?comment
     <!-- r1_foot_ft link -->
     <xacro:macro name="insert_mesh_r1_foot_ft_link">
         <origin xyz="0 0 0" rpy=" 0 0 0" />
         <geometry>
-            <mesh filename="package://uthai_description/meshes/r_foot_ft.STL" scale="0.05 0.05 0.05" />
+            <mesh filename="package://huron_description/meshes/r_foot_ft.STL" scale="0.05 0.05 0.05" />
         </geometry>
         <material name="grey"/>
     </xacro:macro>
-        <!-- r2_foot_ft link  -->
+    <!-- r2_foot_ft link  -->
     <xacro:macro name="insert_mesh_r2_foot_ft_link">
         <origin xyz="0 0 0" rpy=" 0 0 0" />
         <geometry>
-            <mesh filename="package://uthai_description/meshes/r_foot_ft.STL" scale="0.05 0.05 0.05" />
+            <mesh filename="package://huron_description/meshes/r_foot_ft.STL" scale="0.05 0.05 0.05" />
         </geometry>
         <material name="grey"/>
     </xacro:macro>
-        <!-- r3_foot_ft link 3-->
+    <!-- r3_foot_ft link 3-->
     <xacro:macro name="insert_mesh_r3_foot_ft_link">
         <origin xyz="0 0 0" rpy=" 0 0 0" />
         <geometry>
-            <mesh filename="package://uthai_description/meshes/r_foot_ft.STL" scale="0.05 0.05 0.05" />
+            <mesh filename="package://huron_description/meshes/r_foot_ft.STL" scale="0.05 0.05 0.05" />
         </geometry>
         <material name="grey"/>
     </xacro:macro>
-            <!-- r4_foot_ft link 4 -->
+    <!-- r4_foot_ft link 4 -->
     <xacro:macro name="insert_mesh_r4_foot_ft_link">
         <origin xyz="0 0 0" rpy=" 0 0 0" />
         <geometry>
-            <mesh filename="package://uthai_description/meshes/r_foot_ft.STL" scale="0.05 0.05 0.05" />
+            <mesh filename="package://huron_description/meshes/r_foot_ft.STL" scale="0.05 0.05 0.05" />
         </geometry>
         <material name="grey"/>
     </xacro:macro>
+        ?>
 </robot>
