Commit message: Fix joint limits

File: huron_description/urdf/huron_left_leg.xacro (robot description, xacro)
@@ -46,6 +46,6 @@
             xyz="0 0 1" />
           <limit
-            lower="-3.1416"
-            upper="3.1416"
+            lower="-0.01"
+            upper="0.5236"
             effort="${dxl_effort}"
             velocity="${dxl_speed}" />
@@ -81,6 +81,6 @@
             xyz="0 0 1" />
           <limit
-            lower="-3.1416"
-            upper="3.1416"
+            lower="-1.2217"
+            upper="1.2217"
             effort="${dxl_effort}"
             velocity="${dxl_speed}" />
@@ -116,6 +116,6 @@
             xyz="0 0 1" />
           <limit
-            lower="-3.1416"
-            upper="3.1416"
+            lower="${-pi/2}"
+            upper="${pi/2}"
             effort="${dxl_effort}"
             velocity="${dxl_speed}" />
@@ -151,11 +151,11 @@
             xyz="0 0 1" />
           <limit
-            lower="-3.1416"
-            upper="3.1416"
-            effort="${dxl_effort}"
-            velocity="${dxl_speed}" />
-          <dynamics
-            damping="0.5"
-            friction="2.5" />
+            lower="-0.5236"
+            upper="0.1745"
+            effort="${dxl_effort}"
+            velocity="${dxl_speed}" />
+          <dynamics
+            damping="0.5"
+            friction="2.0" />
         </joint>
         <xacro:insert_transmission name="l_ankle_pitch_joint"/>
@@ -186,11 +186,11 @@
             xyz="0 0 1" />
           <limit
-            lower="-3.1416"
-            upper="3.1416"
-            effort="${dxl_effort}"
-            velocity="${dxl_speed}" />
-          <dynamics
-            damping="0.5"
-            friction="2.5" />
+            lower="-0.3491"
+            upper="0.3491"
+            effort="${dxl_effort}"
+            velocity="${dxl_speed}" />
+          <dynamics
+            damping="0.5"
+            friction="2.0" />
         </joint>
         <xacro:insert_transmission name="l_ankle_roll_joint"/>

File: huron_description/urdf/huron_right_leg.xacro (robot description, xacro)
@@ -53,6 +53,6 @@
             xyz="0 0 1" />
           <limit
-            lower="-3.1416"
-            upper="3.1416"
+            lower="-0.5236"
+            upper="0.01"
             effort="${dxl_effort}"
             velocity="${dxl_speed}" />
@@ -88,6 +88,6 @@
             xyz="0 0 1" />
           <limit
-            lower="-3.1416"
-            upper="3.1416"
+            lower="-1.2217"
+            upper="1.2217"
             effort="${dxl_effort}"
             velocity="${dxl_speed}" />
@@ -123,6 +123,6 @@
             xyz="0 0 1" />
           <limit
-            lower="-3.1416"
-            upper="3.1416"
+            lower="-${pi/2}"
+            upper="${pi/2}"
             effort="${dxl_effort}"
             velocity="${dxl_speed}" />
@@ -158,11 +158,11 @@
             xyz="0 0 1" />
           <limit
-            lower="-3.1416"
-            upper="3.1416"
-            effort="${dxl_effort}"
-            velocity="${dxl_speed}" />
-          <dynamics
-            damping="0.5"
-            friction="2.5" />
+            lower="-0.5236"
+            upper="0.1745"
+            effort="${dxl_effort}"
+            velocity="${dxl_speed}" />
+          <dynamics
+            damping="0.5"
+            friction="2.0" />
         </joint>
         <xacro:insert_transmission name="r_ankle_pitch_joint"/>
@@ -193,11 +193,11 @@
             xyz="0 0 1" />
           <limit
-            lower="-3.1416"
-            upper="3.1416"
-            effort="${dxl_effort}"
-            velocity="${dxl_speed}" />
-          <dynamics
-            damping="0.5"
-            friction="2.5" />
+            lower="-0.3491"
+            upper="0.3491"
+            effort="${dxl_effort}"
+            velocity="${dxl_speed}" />
+          <dynamics
+            damping="0.5"
+            friction="2.0" />
         </joint>
         <xacro:insert_transmission name="r_ankle_roll_joint"/>
