Commit message: control

File: huron_description/urdf/huron_gazebo.xacro (robot description, xacro)
@@ -36,94 +36,4 @@
         </sensor>
     </gazebo>
-    <?comment
-    <gazebo reference ="r1_ft_fixed">
-    	<provideFeedback> true</provideFeedback>
-    </gazebo>
-    <gazebo>
-    <plugin name="r1_ft_sensor" filename="libgazebo_ros_ft_sensor.so">
-        <updateRate>100.0</updateRate>
-        <topicName>/robotis/sensor/r1_ft_sensor</topicName>
-        <jointName>r1_ft_fixed</jointName>
-        <gaussianNoise>0.0</gaussianNoise>
-    </plugin>
-    </gazebo>
-    <gazebo reference ="r2_ft_fixed">
-    	<provideFeedback> true</provideFeedback>
-    </gazebo>
-    <gazebo>
-    <plugin name="r2_ft_sensor" filename="libgazebo_ros_ft_sensor.so">
-        <updateRate>100.0</updateRate>
-        <topicName>/robotis/sensor/r2_ft_sensor</topicName>
-        <jointName>r2_ft_fixed</jointName>
-        <gaussianNoise>0.0</gaussianNoise>
-    </plugin>
-    </gazebo>
-    <gazebo reference ="r3_ft_fixed">
-    	<provideFeedback> true</provideFeedback>
-    </gazebo>
-    <gazebo>
-    <plugin name="r3_ft_sensor" filename="libgazebo_ros_ft_sensor.so">
-        <updateRate>100.0</updateRate>
-        <topicName>/robotis/sensor/r3_ft_sensor</topicName>
-        <jointName>r3_ft_fixed</jointName>
-        <gaussianNoise>0.0</gaussianNoise>
-    </plugin>
-    </gazebo>
-    <gazebo reference ="r4_ft_fixed">
-    	<provideFeedback> true</provideFeedback>
-    </gazebo>
-    <gazebo>
-    <plugin name="r4_ft_sensor" filename="libgazebo_ros_ft_sensor.so">
-        <updateRate>100.0</updateRate>
-        <topicName>/robotis/sensor/r4_ft_sensor</topicName>
-        <jointName>r4_ft_fixed</jointName>
-        <gaussianNoise>0.0</gaussianNoise>
-    </plugin>
-    </gazebo>
-    <gazebo reference ="l1_ft_fixed">
-    	<provideFeedback> true</provideFeedback>
-    </gazebo>
-    <gazebo>
-    <plugin name="l1_ft_sensor" filename="libgazebo_ros_ft_sensor.so">
-        <updateRate>100.0</updateRate>
-        <topicName>/robotis/sensor/l1_ft_sensor</topicName>
-        <jointName>l1_ft_fixed</jointName>
-        <gaussianNoise>0.0</gaussianNoise>
-    </plugin>
-    </gazebo>
-    <gazebo reference ="l2_ft_fixed">
-    	<provideFeedback> true</provideFeedback>
-    </gazebo>
-    <gazebo>
-    <plugin name="l2_ft_sensor" filename="libgazebo_ros_ft_sensor.so">
-        <updateRate>100.0</updateRate>
-        <topicName>/robotis/sensor/l2_ft_sensor</topicName>
-        <jointName>l2_ft_fixed</jointName>
-        <gaussianNoise>0.0</gaussianNoise>
-    </plugin>
-    </gazebo>
-    <gazebo reference ="l3_ft_fixed">
-    	<provideFeedback> true</provideFeedback>
-    </gazebo>
-    <gazebo>
-    <plugin name="l3_ft_sensor" filename="libgazebo_ros_ft_sensor.so">
-        <updateRate>100.0</updateRate>
-        <topicName>/robotis/sensor/l3_ft_sensor</topicName>
-        <jointName>l3_ft_fixed</jointName>
-        <gaussianNoise>0.0</gaussianNoise>
-    </plugin>
-    </gazebo>
-    <gazebo reference ="l4_ft_fixed">
-    	<provideFeedback> true</provideFeedback>
-    </gazebo>
-    <gazebo>
-    <plugin name="r4_ft_sensor" filename="libgazebo_ros_ft_sensor.so">
-        <updateRate>100.0</updateRate>
-        <topicName>/robotis/sensor/l4_ft_sensor</topicName>
-        <jointName>l4_ft_fixed</jointName>
-        <gaussianNoise>0.0</gaussianNoise>
-    </plugin>
-    </gazebo>
-      ?>
     <!-- World -->
     <gazebo reference="world"></gazebo>
@@ -183,50 +93,4 @@
         <material>Gazebo/Blue</material>
     </gazebo>
-    <?comment
-    <gazebo reference="l1_foot_ft_link">
-        <kp>100000.0</kp>
-        <kd>100.0</kd>
-        <mu1>0.9</mu1>
-        <mu2>0.9</mu2>
-        <!--<maxContacts>30</maxContacts>-->
-        <fdir1>1 1 0</fdir1>
-         <maxVel>1.0</maxVel>
-        <minDepth>0.0001</minDepth>
-        <material>Gazebo/white</material>
-    </gazebo>
-    <gazebo reference="l2_foot_ft_link">
-        <kp>100000.0</kp>
-        <kd>100.0</kd>
-        <mu1>0.9</mu1>
-        <mu2>0.9</mu2>
-        <!--<maxContacts>30</maxContacts>-->
-        <fdir1>1 1 0</fdir1>
-         <maxVel>1.0</maxVel>
-        <minDepth>0.0001</minDepth>
-        <material>Gazebo/white</material>
-    </gazebo>
-    <gazebo reference="l3_foot_ft_link">
-        <kp>100000.0</kp>
-        <kd>100.0</kd>
-        <mu1>0.9</mu1>
-        <mu2>0.9</mu2>
-        <!--<maxContacts>30</maxContacts>-->
-        <fdir1>1 1 0</fdir1>
-         <maxVel>1.0</maxVel>
-        <minDepth>0.0001</minDepth>
-        <material>Gazebo/white</material>
-    </gazebo>
-    <gazebo reference="l4_foot_ft_link">
-        <kp>100000.0</kp>
-        <kd>100.0</kd>
-        <mu1>0.9</mu1>
-        <mu2>0.9</mu2>
-        <!--<maxContacts>30</maxContacts>-->
-        <fdir1>1 1 0</fdir1>
-         <maxVel>1.0</maxVel>
-        <minDepth>0.0001</minDepth>
-        <material>Gazebo/white</material>
-    </gazebo>
-    ?>
     <!-- Right Leg -->
     <gazebo reference="r_hip_yaw_link">
@@ -271,49 +135,3 @@
         <material>Gazebo/Blue</material>
     </gazebo>
-    <?comment
-    <gazebo reference="r1_foot_ft_link">
-        <kp>100000.0</kp>
-        <kd>100.0</kd>
-        <mu1>0.9</mu1>
-        <mu2>0.9</mu2>
-        <!--<maxContacts>30</maxContacts>-->
-        <fdir1>1 1 0</fdir1>
-         <maxVel>1.0</maxVel>
-        <minDepth>0.0001</minDepth>
-        <material>Gazebo/white</material>
-    </gazebo>
-    <gazebo reference="r2_foot_ft_link">
-        <kp>100000.0</kp>
-        <kd>100.0</kd>
-        <mu1>0.9</mu1>
-        <mu2>0.9</mu2>
-        <!--<maxContacts>30</maxContacts>-->
-        <fdir1>1 1 0</fdir1>
-         <maxVel>1.0</maxVel>
-        <minDepth>0.0001</minDepth>
-        <material>Gazebo/white</material>
-    </gazebo>
-    <gazebo reference="r3_foot_ft_link">
-        <kp>100000.0</kp>
-        <kd>100.0</kd>
-        <mu1>0.9</mu1>
-        <mu2>0.9</mu2>
-        <!--<maxContacts>30</maxContacts>-->
-        <fdir1>1 1 0</fdir1>
-         <maxVel>1.0</maxVel>
-        <minDepth>0.0001</minDepth>
-        <material>Gazebo/white</material>
-    </gazebo>
-    <gazebo reference="r4_foot_ft_link">
-        <kp>100000.0</kp>
-        <kd>100.0</kd>
-        <mu1>0.9</mu1>
-        <mu2>0.9</mu2>
-        <!--<maxContacts>30</maxContacts>-->
-        <fdir1>1 1 0</fdir1>
-         <maxVel>1.0</maxVel>
-        <minDepth>0.0001</minDepth>
-        <material>Gazebo/white</material>
-    </gazebo>
-    ?>
 </robot>
