Commit message: Standing

File: huron_description/urdf/huron_gazebo.xacro (robot description, xacro)
@@ -181,80 +181,4 @@
         <material>Gazebo/Blue</material>
     </gazebo>
-    <gazebo reference="l1_foot_ft_link">
-        <kp>100000.0</kp>
-        <kd>100.0</kd>
-        <mu1>0.9</mu1>
-        <mu2>0.9</mu2>
-        <surface>
-          <contact>
-              <ode>
-                <kp>1e15</kp>
-                <kd>1e13</kd>
-              </ode>
-            </contact>
-        </surface>
-        <!--<maxContacts>30</maxContacts>-->
-        <fdir1>1 1 0</fdir1>
-         <maxVel>1.0</maxVel>
-        <minDepth>0.0001</minDepth>
-        <material>Gazebo/Black</material>
-    </gazebo>
-    <gazebo reference="l2_foot_ft_link">
-        <kp>100000.0</kp>
-        <kd>100.0</kd>
-        <mu1>0.9</mu1>
-        <mu2>0.9</mu2>
-        <surface>
-          <contact>
-              <ode>
-                <kp>1e15</kp>
-                <kd>1e13</kd>
-              </ode>
-            </contact>
-        </surface>
-        <!--<maxContacts>30</maxContacts>-->
-        <fdir1>1 1 0</fdir1>
-         <maxVel>1.0</maxVel>
-        <minDepth>0.0001</minDepth>
-        <material>Gazebo/Black</material>
-    </gazebo>
-    <gazebo reference="l3_foot_ft_link">
-        <kp>100000.0</kp>
-        <kd>100.0</kd>
-        <mu1>0.9</mu1>
-        <mu2>0.9</mu2>
-        <surface>
-          <contact>
-              <ode>
-                <kp>1e15</kp>
-                <kd>1e13</kd>
-              </ode>
-            </contact>
-        </surface>
-        <!--<maxContacts>30</maxContacts>-->
-        <fdir1>1 1 0</fdir1>
-         <maxVel>1.0</maxVel>
-        <minDepth>0.0001</minDepth>
-        <material>Gazebo/Black</material>
-    </gazebo>
-    <gazebo reference="l4_foot_ft_link">
-        <kp>100000.0</kp>
-        <kd>100.0</kd>
-        <mu1>0.9</mu1>
-        <mu2>0.9</mu2>
-        <surface>
-          <contact>
-              <ode>
-                <kp>1e15</kp>
-                <kd>1e13</kd>
-              </ode>
-            </contact>
-        </surface>
-        <!--<maxContacts>30</maxContacts>-->
-        <fdir1>1 1 0</fdir1>
-         <maxVel>1.0</maxVel>
-        <minDepth>0.0001</minDepth>
-        <material>Gazebo/Black</material>
-    </gazebo>
     <!-- Right Leg -->
     <gazebo reference="r_hip_yaw_link">
@@ -299,79 +223,3 @@
         <material>Gazebo/Blue</material>
     </gazebo>
-    <gazebo reference="r1_foot_ft_link">
-        <kp>100000.0</kp>
-        <kd>100.0</kd>
-        <mu1>0.9</mu1>
-        <mu2>0.9</mu2>
-        <surface>
-          <contact>
-              <ode>
-                <kp>1e15</kp>
-                <kd>1e13</kd>
-              </ode>
-            </contact>
-        </surface>
-        <!--<maxContacts>30</maxContacts>-->
-        <fdir1>1 1 0</fdir1>
-         <maxVel>1.0</maxVel>
-        <minDepth>0.0001</minDepth>
-        <material>Gazebo/Black</material>
-    </gazebo>
-    <gazebo reference="r2_foot_ft_link">
-        <kp>100000.0</kp>
-        <kd>100.0</kd>
-        <mu1>0.9</mu1>
-        <mu2>0.9</mu2>
-        <surface>
-          <contact>
-              <ode>
-                <kp>1e15</kp>
-                <kd>1e13</kd>
-              </ode>
-            </contact>
-        </surface>
-        <!--<maxContacts>30</maxContacts>-->
-        <fdir1>1 1 0</fdir1>
-         <maxVel>1.0</maxVel>
-        <minDepth>0.0001</minDepth>
-        <material>Gazebo/Black</material>
-    </gazebo>
-    <gazebo reference="r3_foot_ft_link">
-        <kp>100000.0</kp>
-        <kd>100.0</kd>
-        <mu1>0.9</mu1>
-        <mu2>0.9</mu2>
-        <surface>
-          <contact>
-              <ode>
-                <kp>1e15</kp>
-                <kd>1e13</kd>
-              </ode>
-            </contact>
-        </surface>
-        <!--<maxContacts>30</maxContacts>-->
-        <fdir1>1 1 0</fdir1>
-         <maxVel>1.0</maxVel>
-        <minDepth>0.0001</minDepth>
-        <material>Gazebo/Black</material>
-    </gazebo>
-    <gazebo reference="r4_foot_ft_link">
-        <kp>100000.0</kp>
-        <kd>100.0</kd>
-        <mu1>0.9</mu1>
-        <mu2>0.9</mu2>
-        <surface>
-          <contact>
-              <ode>
-                <kp>1e15</kp>
-                <kd>1e13</kd>
-              </ode>
-            </contact>
-        </surface>
-        <!--<maxContacts>30</maxContacts>-->
-        <fdir1>1 1 0</fdir1>
-         <maxVel>1.0</maxVel>
-        <minDepth>0.0001</minDepth>
-        <material>Gazebo/Black</material>
-    </gazebo>
 </robot>

File: huron_description/urdf/huron_inertia.xacro (robot description, xacro)
@@ -108,64 +108,4 @@
     </xacro:macro>
     <!-- Left foot sensors -->
-    <!-- l1_foot_ft link -->
-    <xacro:macro name="insert_inertia_l1_foot_ft_link">
-      <origin
-        xyz="6.5681E-06 0.0048368 0.00012069"
-        rpy="0 0 0" />
-      <mass
-        value="0.0086322" />
-      <inertia
-        ixx="3.8994E-07"
-        ixy="2.5351E-10"
-        ixz="3.0416E-10"
-        iyy="5.8206E-07"
-        iyz="5.9744E-09"
-        izz="3.4276E-07" />
-    </xacro:macro>
-    <!-- l2_foot_ft link  -->
-    <xacro:macro name="insert_inertia_l2_foot_ft_link">
-      <origin
-        xyz="6.56809560273253E-06 0.00483682139671537 0.000120685375128327"
-        rpy="0 0 0" />
-      <mass
-        value="0.00863223621815319" />
-      <inertia
-        ixx="3.89940248965647E-07"
-        ixy="2.53506346419819E-10"
-        ixz="3.04161588773098E-10"
-        iyy="5.82064646347941E-07"
-        iyz="5.97441467814794E-09"
-        izz="3.42755265424868E-07" />
-    </xacro:macro>
-    <!-- l3_foot_ft link 3 -->
-    <xacro:macro name="insert_inertia_l3_foot_ft_link">
-      <origin
-        xyz="6.56809560273253E-06 0.00483682139671548 0.000120685375128382"
-        rpy="0 0 0" />
-      <mass
-        value="0.00863223621815319" />
-      <inertia
-        ixx="3.89940248965648E-07"
-        ixy="2.53506346419837E-10"
-        ixz="3.04161588773088E-10"
-        iyy="5.82064646347941E-07"
-        iyz="5.97441467814795E-09"
-        izz="3.42755265424868E-07" />
-    </xacro:macro>
-    <!-- l4_foot_ft link 4 -->
-    <xacro:macro name="insert_inertia_l4_foot_ft_link">
-      <origin
-        xyz="6.5681E-06 0.0048368 0.00012069"
-        rpy="0 0 0" />
-      <mass
-        value="0.0086322" />
-      <inertia
-        ixx="3.8994E-07"
-        ixy="2.5351E-10"
-        ixz="3.0416E-10"
-        iyy="5.8206E-07"
-        iyz="5.9744E-09"
-        izz="3.4276E-07" />
-    </xacro:macro>
     <!-- Right leg -->
     <!-- right hip yaw link -->
@@ -260,63 +200,3 @@
     </xacro:macro>
     <!-- Right foot sensors -->
-    <!-- r1_foot_ft link -->
-    <xacro:macro name="insert_inertia_r1_foot_ft_link">
-      <origin
-        xyz="-9.3029E-06 0.0048381 4.6013E-05"
-        rpy="0 0 0" />
-      <mass
-        value="0.0086322" />
-      <inertia
-        ixx="3.8994E-07"
-        ixy="-3.7469E-10"
-        ixz="5.2298E-10"
-        iyy="5.8219E-07"
-        iyz="2.2796E-09"
-        izz="3.4263E-07" />
-    </xacro:macro>
-    <!-- r2_foot_ft link  -->
-    <xacro:macro name="insert_inertia_r2_foot_ft_link">
-      <origin
-        xyz="-9.3029E-06 0.0048381 4.6013E-05"
-        rpy="0 0 0" />
-      <mass
-        value="0.0086322" />
-      <inertia
-        ixx="3.8994E-07"
-        ixy="-3.7469E-10"
-        ixz="5.2298E-10"
-        iyy="5.8219E-07"
-        iyz="2.2796E-09"
-        izz="3.4263E-07" />
-    </xacro:macro>
-    <!-- r_foot_ft link 3 -->
-    <xacro:macro name="insert_inertia_r3_foot_ft_link">
-      <origin
-        xyz="-9.3029E-06 0.0048381 4.6013E-05"
-        rpy="0 0 0" />
-      <mass
-        value="0.0086322" />
-      <inertia
-        ixx="3.8994E-07"
-        ixy="-3.7469E-10"
-        ixz="5.2298E-10"
-        iyy="5.8219E-07"
-        iyz="2.2796E-09"
-        izz="3.4263E-07" />
-    </xacro:macro>
-    <!-- r_foot_ft link 4 -->
-    <xacro:macro name="insert_inertia_r4_foot_ft_link">
-      <origin
-        xyz="-9.3029E-06 0.0048381 4.6013E-05"
-        rpy="0 0 0" />
-      <mass
-        value="0.0086322" />
-      <inertia
-        ixx="3.8994E-07"
-        ixy="-3.7469E-10"
-        ixz="5.2298E-10"
-        iyy="5.8219E-07"
-        iyz="2.2796E-09"
-        izz="3.4263E-07" />
-    </xacro:macro>
 </robot>

File: huron_description/urdf/huron_left_leg.xacro (robot description, xacro)
@@ -207,116 +207,4 @@
             </inertial>
         </link>
-        <!-- left ft fixed joint 1 -->
-        <joint name="l1_ft_fixed" type="revolute">
-            <origin
-              xyz="0.096 0.020682 0.13788"
-              rpy="-0.0 0.0 ${pi/2}" />
-            <axis xyz="0 0 1"/>
-            <parent link="l_ankle_roll_link"/>
-            <child link="l1_foot_ft_link"/>
-            <limit
-            lower="0"
-            upper="0"
-            effort="100"
-            velocity="100" />
-        </joint>
-        <!-- left foot ft link 1 -->
-        <link name="l1_foot_ft_link">
-	    <visual>
-		<xacro:insert_mesh_l1_foot_ft_link />
-	    </visual>
-            <collision>
-                <xacro:insert_mesh_l1_foot_ft_link />
-            </collision>
-	    <inertial>
-		<xacro:insert_inertia_l1_foot_ft_link />
-	    </inertial>
-        </link>
-        <!-- left ft fixed joint 2 -->
-        <joint name="l2_ft_fixed" type="revolute">
-            <origin
-              xyz="0.096 -0.014318 0.13788"
-              rpy="-0.0 0.0 ${pi/2}" />
-            <axis xyz="0 0 1"/>
-            <parent link="l_ankle_roll_link"/>
-            <child link="l2_foot_ft_link"/>
-            <limit
-            lower="0"
-            upper="0"
-            effort="100"
-            velocity="100" />
-        </joint>
-        <!-- left foot ft link 2 -->
-        <link name="l2_foot_ft_link">
-	    <visual>
-		<xacro:insert_mesh_l2_foot_ft_link />
-	    </visual>
-            <collision>
-                <xacro:insert_mesh_l2_foot_ft_link />
-            </collision>
-	    <inertial>
-		<xacro:insert_inertia_l2_foot_ft_link />
-	    </inertial>
-        </link>
-        <!-- left ft fixed joint 3 -->
-        <joint name="l3_ft_fixed" type="revolute">
-            <origin
-              xyz="0.096 -0.016649 -0.026"
-              rpy="-0.0 0.0 ${pi/2}" />
-            <axis xyz="0 0 1"/>
-            <parent link="l_ankle_roll_link"/>
-            <child link="l3_foot_ft_link"/>
-            <limit
-            lower="0"
-            upper="0"
-            effort="100"
-            velocity="100" />
-        </joint>
-        <!-- left foot ft link 3 -->
-        <link name="l3_foot_ft_link">
-	    <visual>
-		<xacro:insert_mesh_l3_foot_ft_link />
-	    </visual>
-            <collision>
-                <xacro:insert_mesh_l3_foot_ft_link />
-            </collision>
-	    <inertial>
-		<xacro:insert_inertia_l3_foot_ft_link />
-	    </inertial>
-        </link>
-        <!-- left ft fixed joint 4 -->
-        <joint name="l4_ft_fixed" type="revolute">
-            <origin
-              xyz="0.096 0.01686 -0.026"
-              rpy="-0.0 0.0 ${pi/2}" />
-            <axis xyz="0 0 1"/>
-            <parent link="l_ankle_roll_link"/>
-            <child link="l4_foot_ft_link"/>
-            <limit
-            lower="0"
-            upper="0"
-            effort="100"
-            velocity="100" />
-        </joint>
-        <!-- left foot ft link 4 -->
-        <link name="l4_foot_ft_link">
-	    <visual>
-		<xacro:insert_mesh_l4_foot_ft_link />
-	    </visual>
-            <collision>
-                <xacro:insert_mesh_l4_foot_ft_link />
-            </collision>
-	    <inertial>
-		<xacro:insert_inertia_l4_foot_ft_link />
-	    </inertial>
-        </link>
-        <!-- left ft fixed joint -->
-        <joint name="lv_ft_fixed" type="fixed">
-            <origin xyz="0.045 0.0 0.0" rpy="0 ${-pi/2} 0"/>
-            <parent link="l4_foot_ft_link"/>
-            <child link="l_foot_v_ft_link"/>
-        </joint>
-        <!-- left foot ft link -->
-        <link name="l_foot_v_ft_link"></link>
     </xacro:macro>
 </robot>

File: huron_description/urdf/huron_right_leg.xacro (robot description, xacro)
@@ -214,123 +214,4 @@
             </inertial>
         </link>
-        <!-- Right foot sensors -->
-        <!-- right ft fixed joint 1 -->
-        <joint name="r1_ft_fixed" type="revolute">
-            <origin
-              xyz="0.096 0.014348 0.13788"
-              rpy="-0.0 0.0 ${pi/2}" />
-            <axis xyz="0 0 1"/>
-            <parent link="r_ankle_roll_link"/>
-            <child link="r1_foot_ft_link"/>
-            <limit
-            lower="0"
-            upper="0"
-            effort="100"
-            velocity="100" />
-        </joint>
-        <!-- right foot ft link 1 -->
-        <link name="r1_foot_ft_link">
-	    <visual>
-		<xacro:insert_mesh_r1_foot_ft_link />
-	    </visual>
-            <collision>
-                <xacro:insert_mesh_r1_foot_ft_link />
-            </collision>
-	    <inertial>
-		<xacro:insert_inertia_r1_foot_ft_link />
-	    </inertial>
-        </link>
-        <!-- right ft fixed joint 2 -->
-        <joint name="r2_ft_fixed" type="revolute">
-            <origin
-              xyz="0.096 -0.020652 0.13788"
-              rpy="-0.0 0.0 ${pi/2}" />
-            <axis xyz="0 0 1"/>
-            <parent link="r_ankle_roll_link"/>
-            <child link="r2_foot_ft_link"/>
-            <limit
-            lower="0"
-            upper="0"
-            effort="100"
-            velocity="100" />
-        </joint>
-        <!-- right foot ft link 2 -->
-        <link name="r2_foot_ft_link">
-	    <visual>
-		<xacro:insert_mesh_r2_foot_ft_link />
-	    </visual>
-            <collision>
-                <xacro:insert_mesh_r2_foot_ft_link />
-            </collision>
-	    <inertial>
-		<xacro:insert_inertia_r2_foot_ft_link />
-	    </inertial>
-        </link>
-        <!-- right ft fixed joint 3 -->
-        <joint name="r3_ft_fixed" type="revolute">
-            <origin
-              xyz="0.096 -0.01683 -0.026"
-              rpy="-0.0 0.0 ${pi/2}" />
-            <axis xyz="0 0 1"/>
-            <parent link="r_ankle_roll_link"/>
-            <child link="r3_foot_ft_link"/>
-            <limit
-            lower="0"
-            upper="0"
-            effort="100"
-            velocity="100" />
-        </joint>
-        <!-- right foot ft link 3 -->
-        <link name="r3_foot_ft_link">
-	    <visual>
-		<xacro:insert_mesh_r3_foot_ft_link />
-	    </visual>
-            <collision>
-                <xacro:insert_mesh_r3_foot_ft_link />
-            </collision>
-	    <inertial>
-		<xacro:insert_inertia_r3_foot_ft_link />
-	    </inertial>
-        </link>
-        <!-- right ft fixed joint 4 -->
-        <joint name="r4_ft_fixed" type="revolute">
-            <origin
-              xyz="0.096 0.016679 -0.026"
-              rpy="-0.0 0.0 ${pi/2}" />
-            <axis xyz="0 0 1"/>
-            <parent link="r_ankle_roll_link"/>
-            <child link="r4_foot_ft_link"/>
-            <limit
-            lower="0"
-            upper="0"
-            effort="100"
-            velocity="100" />
-        </joint>
-        <!-- right4 foot ft link 4 -->
-        <link name="r4_foot_ft_link">
-	    <visual>
-		<xacro:insert_mesh_r4_foot_ft_link />
-	    </visual>
-            <collision>
-                <xacro:insert_mesh_r4_foot_ft_link />
-            </collision>
-	    <inertial>
-		<xacro:insert_inertia_r4_foot_ft_link />
-	    </inertial>
-        </link>
-        <!-- right ft fixed joint -->
-        <joint name="rv_ft_fixed" type="fixed">
-            <origin xyz="0.0 0.0 0.0" rpy="0 0 0"/>
-            <axis xyz="0 0 0"/>
-            <parent link="r4_foot_ft_link"/>
-            <child link="r_foot_v_ft_link"/>
-            <limit
-            lower="0"
-            upper="0"
-            effort="100"
-            velocity="100" />
-        </joint>
-        <!-- right foot ft link -->
-        <link name="r_foot_v_ft_link"></link>
     </xacro:macro>
 </robot>

File: huron_description/urdf/huron_visuals.xacro (robot description, xacro)
@@ -62,36 +62,4 @@
         </material>
     </xacro:macro>
-    <!-- l1_foot_ft link -->
-    <xacro:macro name="insert_mesh_l1_foot_ft_link">
-        <origin xyz="0 0 0" rpy=" 0 0 0" />
-        <geometry>
-            <mesh filename="package://huron_description/meshes/r_foot_ft.STL" scale="1 1 1" />
-        </geometry>
-        <material name="grey"/>
-    </xacro:macro>
-    <!-- l2_foot_ft link  -->
-    <xacro:macro name="insert_mesh_l2_foot_ft_link">
-        <origin xyz="0 0 0" rpy=" 0 0 0" />
-        <geometry>
-            <mesh filename="package://huron_description/meshes/r_foot_ft.STL" scale="1 1 1" />
-        </geometry>
-        <material name="grey"/>
-    </xacro:macro>
-    <!-- l3_foot_ft link 3 -->
-    <xacro:macro name="insert_mesh_l3_foot_ft_link">
-        <origin xyz="0 0 0" rpy=" 0 0 0" />
-        <geometry>
-            <mesh filename="package://huron_description/meshes/r_foot_ft.STL" scale="1 1 1" />
-        </geometry>
-        <material name="grey"/>
-    </xacro:macro>
-    <!-- l4_foot_ft link 4 -->
-    <xacro:macro name="insert_mesh_l4_foot_ft_link">
-        <origin xyz="0 0 0" rpy=" 0 0 0" />
-        <geometry>
-            <mesh filename="package://huron_description/meshes/r_foot_ft.STL" scale="1 1 1" />
-        </geometry>
-        <material name="grey"/>
-    </xacro:macro>
     <!-- right hip yaw link -->
     <xacro:macro name="insert_mesh_r_hip_yaw_link">
@@ -147,35 +115,3 @@
     </xacro:macro>
     <!-- Right foot sensors -->
-    <!-- r1_foot_ft link -->
-    <xacro:macro name="insert_mesh_r1_foot_ft_link">
-        <origin xyz="0 0 0" rpy=" 0 0 0" />
-        <geometry>
-            <mesh filename="package://huron_description/meshes/r_foot_ft.STL" scale="1 1 1" />
-        </geometry>
-        <material name="grey"/>
-    </xacro:macro>
-    <!-- r2_foot_ft link  -->
-    <xacro:macro name="insert_mesh_r2_foot_ft_link">
-        <origin xyz="0 0 0" rpy=" 0 0 0" />
-        <geometry>
-            <mesh filename="package://huron_description/meshes/r_foot_ft.STL" scale="1 1 1" />
-        </geometry>
-        <material name="grey"/>
-    </xacro:macro>
-    <!-- r3_foot_ft link 3-->
-    <xacro:macro name="insert_mesh_r3_foot_ft_link">
-        <origin xyz="0 0 0" rpy=" 0 0 0" />
-        <geometry>
-            <mesh filename="package://huron_description/meshes/r_foot_ft.STL" scale="1 1 1" />
-        </geometry>
-        <material name="grey"/>
-    </xacro:macro>
-    <!-- r4_foot_ft link 4 -->
-    <xacro:macro name="insert_mesh_r4_foot_ft_link">
-        <origin xyz="0 0 0" rpy=" 0 0 0" />
-        <geometry>
-            <mesh filename="package://huron_description/meshes/r_foot_ft.STL" scale="1 1 1" />
-        </geometry>
-        <material name="grey"/>
-    </xacro:macro>
 </robot>

Commit message: Original design working

File: huron_description/urdf/huron_gazebo.xacro (robot description, xacro)
@@ -316,25 +316,3 @@
         <material>Gazebo/Orange</material>
     </gazebo>
-    <gazebo reference="l_foot_base_link">
-        <kp>100000.0</kp>
-        <kd>100.0</kd>
-        <mu1>0.9</mu1>
-        <mu2>0.9</mu2>
-        <!--<maxContacts>30</maxContacts>-->
-        <!-- <fdir1>1 0 0</fdir1> -->
-         <maxVel>1.0</maxVel>
-        <minDepth>0.0001</minDepth>
-        <material>Gazebo/Green</material>
-    </gazebo>
-    <gazebo reference="r_foot_base_link">
-        <kp>100000.0</kp>
-        <kd>100.0</kd>
-        <mu1>0.9</mu1>
-        <mu2>0.9</mu2>
-        <!--<maxContacts>30</maxContacts>-->
-        <!-- <fdir1>1 0 0</fdir1> -->
-         <maxVel>1.0</maxVel>
-        <minDepth>0.0001</minDepth>
-        <material>Gazebo/Green</material>
-    </gazebo>
 </robot>

File: huron_description/urdf/huron_left_leg.xacro (robot description, xacro)
@@ -319,21 +319,4 @@
         <!-- left foot ft link -->
         <link name="l_foot_v_ft_link"></link>
-        <!-- Foot base -->
-        <link name="l_foot_base_link">
-	    <visual>
-		<xacro:insert_mesh_foot_base_link />
-	    </visual>
-            <collision>
-                <xacro:insert_mesh_foot_base_link />
-            </collision>
-	    <inertial>
-		<xacro:insert_inertia_foot_base_link />
-	    </inertial>
-        </link>
-        <joint name="l_foot_base_fixed" type="fixed">
-            <origin xyz="-0.0175 -0.0025 -0.06395" rpy="0 0 0"/>
-            <parent link="l1_foot_ft_link"/>
-            <child link="l_foot_base_link"/>
-        </joint>
     </xacro:macro>
 </robot>

File: huron_description/urdf/huron_right_leg.xacro (robot description, xacro)
@@ -332,21 +332,4 @@
         <!-- right foot ft link -->
         <link name="r_foot_v_ft_link"></link>
-        <!-- Foot base -->
-        <link name="r_foot_base_link">
-	    <visual>
-		<xacro:insert_mesh_foot_base_link />
-	    </visual>
-            <collision>
-                <xacro:insert_mesh_foot_base_link />
-            </collision>
-	    <inertial>
-		<xacro:insert_inertia_foot_base_link />
-	    </inertial>
-        </link>
-        <joint name="r_foot_base_fixed" type="fixed">
-            <origin xyz="-0.0175 -0.0025 -0.06395" rpy="0 0 0"/>
-            <parent link="r1_foot_ft_link"/>
-            <child link="r_foot_base_link"/>
-        </joint>
     </xacro:macro>
 </robot>
