Commit message: Replace 8 force sensors by 2 6-DoF load cells

File: huron_description/urdf/huron_gazebo.xacro (robot description, xacro)
@@ -36,5 +36,5 @@
         </sensor>
     </gazebo>
-    <gazebo reference ="r1_ft_fixed">
+    <gazebo reference ="r_ankle_roll_joint">
     	<provideFeedback>true</provideFeedback>
     </gazebo>
@@ -43,42 +43,9 @@
         <updateRate>100.0</updateRate>
         <topicName>/huron/sensor/r1_ft_sensor</topicName>
-        <jointName>r1_ft_fixed</jointName>
+        <jointName>r_ankle_roll_joint</jointName>
         <gaussianNoise>0.0</gaussianNoise>
     </plugin>
     </gazebo>
-    <gazebo reference ="r2_ft_fixed">
-    	<provideFeedback>true</provideFeedback>
-    </gazebo>
-    <gazebo>
-    <plugin name="r2_ft_sensor" filename="libgazebo_ros_ft_sensor.so">
-        <updateRate>100.0</updateRate>
-        <topicName>/huron/sensor/r2_ft_sensor</topicName>
-        <jointName>r2_ft_fixed</jointName>
-        <gaussianNoise>0.0</gaussianNoise>
-    </plugin>
-    </gazebo>
-    <gazebo reference ="r3_ft_fixed">
-    	<provideFeedback>true</provideFeedback>
-    </gazebo>
-    <gazebo>
-    <plugin name="r3_ft_sensor" filename="libgazebo_ros_ft_sensor.so">
-        <updateRate>100.0</updateRate>
-        <topicName>/huron/sensor/r3_ft_sensor</topicName>
-        <jointName>r3_ft_fixed</jointName>
-        <gaussianNoise>0.0</gaussianNoise>
-    </plugin>
-    </gazebo>
-    <gazebo reference ="r4_ft_fixed">
-    	<provideFeedback>true</provideFeedback>
-    </gazebo>
-    <gazebo>
-    <plugin name="r4_ft_sensor" filename="libgazebo_ros_ft_sensor.so">
-        <updateRate>100.0</updateRate>
-        <topicName>/huron/sensor/r4_ft_sensor</topicName>
-        <jointName>r4_ft_fixed</jointName>
-        <gaussianNoise>0.0</gaussianNoise>
-    </plugin>
-    </gazebo>
-    <gazebo reference ="l1_ft_fixed">
+    <gazebo reference ="l_ankle_roll_joint">
     	<provideFeedback>true</provideFeedback>
     </gazebo>
@@ -87,38 +54,5 @@
         <updateRate>100.0</updateRate>
         <topicName>/huron/sensor/l1_ft_sensor</topicName>
-        <jointName>l1_ft_fixed</jointName>
-        <gaussianNoise>0.0</gaussianNoise>
-    </plugin>
-    </gazebo>
-    <gazebo reference ="l2_ft_fixed">
-    	<provideFeedback>true</provideFeedback>
-    </gazebo>
-    <gazebo>
-    <plugin name="l2_ft_sensor" filename="libgazebo_ros_ft_sensor.so">
-        <updateRate>100.0</updateRate>
-        <topicName>/huron/sensor/l2_ft_sensor</topicName>
-        <jointName>l2_ft_fixed</jointName>
-        <gaussianNoise>0.0</gaussianNoise>
-    </plugin>
-    </gazebo>
-    <gazebo reference ="l3_ft_fixed">
-    	<provideFeedback>true</provideFeedback>
-    </gazebo>
-    <gazebo>
-    <plugin name="l3_ft_sensor" filename="libgazebo_ros_ft_sensor.so">
-        <updateRate>100.0</updateRate>
-        <topicName>/huron/sensor/l3_ft_sensor</topicName>
-        <jointName>l3_ft_fixed</jointName>
-        <gaussianNoise>0.0</gaussianNoise>
-    </plugin>
-    </gazebo>
-    <gazebo reference ="l4_ft_fixed">
-    	<provideFeedback>true</provideFeedback>
-    </gazebo>
-    <gazebo>
-    <plugin name="r4_ft_sensor" filename="libgazebo_ros_ft_sensor.so">
-        <updateRate>100.0</updateRate>
-        <topicName>/huron/sensor/l4_ft_sensor</topicName>
-        <jointName>l4_ft_fixed</jointName>
+        <jointName>l_ankle_roll_joint</jointName>
         <gaussianNoise>0.0</gaussianNoise>
     </plugin>
@@ -176,57 +110,14 @@
     </gazebo>
     <gazebo reference="l_ankle_roll_link">
-        <!-- <kp>100000.0</kp> -->
-        <!-- <kd>100.0</kd> -->
+        <kp>1e15</kp>
+        <kd>1e13</kd>
         <mu1>0.9</mu1>
         <mu2>0.9</mu2>
+        <!-- <mu>0.9</mu> -->
         <!--<maxContacts>30</maxContacts>-->
-        <!-- <fdir1>1 0 0</fdir1> -->
+        <fdir1>0 -1 0</fdir1>
         <!-- <maxVel>1.0</maxVel> -->
         <!-- <minDepth>0.001</minDepth> -->
         <material>Gazebo/Blue</material>
-    </gazebo>
-    <gazebo reference="l1_foot_ft_link">
-        <kp>1e7</kp>
-        <kd>1e5</kd>
-        <mu1>1.5</mu1>
-        <mu2>1.5</mu2>
-        <!--<maxContacts>30</maxContacts>-->
-        <fdir1>1 0 0</fdir1>
-         <maxVel>0.0</maxVel>
-        <minDepth>0.001</minDepth>
-        <material>Gazebo/Orange</material>
-    </gazebo>
-    <gazebo reference="l2_foot_ft_link">
-        <kp>1e7</kp>
-        <kd>1e5</kd>
-        <mu1>1.5</mu1>
-        <mu2>1.5</mu2>
-        <!--<maxContacts>30</maxContacts>-->
-        <fdir1>1 0 0</fdir1>
-         <maxVel>0.0</maxVel>
-        <minDepth>0.001</minDepth>
-        <material>Gazebo/Orange</material>
-    </gazebo>
-    <gazebo reference="l3_foot_ft_link">
-        <kp>1e7</kp>
-        <kd>1e5</kd>
-        <mu1>1.5</mu1>
-        <mu2>1.5</mu2>
-        <!--<maxContacts>30</maxContacts>-->
-        <fdir1>1 0 0</fdir1>
-         <maxVel>0.0</maxVel>
-        <minDepth>0.001</minDepth>
-        <material>Gazebo/Orange</material>
-    </gazebo>
-    <gazebo reference="l4_foot_ft_link">
-        <kp>1e7</kp>
-        <kd>1e5</kd>
-        <mu1>1.5</mu1>
-        <mu2>1.5</mu2>
-        <!--<maxContacts>30</maxContacts>-->
-        <fdir1>1 0 0</fdir1>
-         <maxVel>0.0</maxVel>
-        <minDepth>0.001</minDepth>
-        <material>Gazebo/Orange</material>
     </gazebo>
     <!-- Right Leg -->
@@ -262,57 +153,14 @@
     </gazebo>
     <gazebo reference="r_ankle_roll_link">
-        <!-- <kp>100000.0</kp> -->
-        <!-- <kd>100.0</kd> -->
+        <kp>1e15</kp>
+        <kd>1e13</kd>
         <mu1>0.9</mu1>
         <mu2>0.9</mu2>
+        <!-- <mu>0.9</mu> -->
         <!--<maxContacts>30</maxContacts>-->
-        <!-- <fdir1>1 0 0</fdir1> -->
+        <fdir1>0 -1 0</fdir1>
         <!--  <maxVel>1.0</maxVel>  -->
         <!-- <minDepth>0.0001</minDepth> -->
         <material>Gazebo/Blue</material>
     </gazebo>
-    <gazebo reference="r1_foot_ft_link">
-        <kp>1e7</kp>
-        <kd>1e5</kd>
-        <mu1>1.5</mu1>
-        <mu2>1.5</mu2>
-        <!--<maxContacts>30</maxContacts>-->
-        <fdir1>1 0 0</fdir1>
-         <maxVel>0.0</maxVel>
-        <minDepth>0.001</minDepth>
-        <material>Gazebo/Orange</material>
-    </gazebo>
-    <gazebo reference="r2_foot_ft_link">
-        <kp>1e7</kp>
-        <kd>1e5</kd>
-        <mu1>1.5</mu1>
-        <mu2>1.5</mu2>
-        <!--<maxContacts>30</maxContacts>-->
-        <fdir1>1 0 0</fdir1>
-         <maxVel>0.0</maxVel>
-        <minDepth>0.001</minDepth>
-        <material>Gazebo/Orange</material>
-    </gazebo>
-    <gazebo reference="r3_foot_ft_link">
-        <kp>1e7</kp>
-        <kd>1e5</kd>
-        <mu1>1.5</mu1>
-        <mu2>1.5</mu2>
-        <!--<maxContacts>30</maxContacts>-->
-        <fdir1>1 0 0</fdir1>
-         <maxVel>0.0</maxVel>
-        <minDepth>0.001</minDepth>
-        <material>Gazebo/Orange</material>
-    </gazebo>
-    <gazebo reference="r4_foot_ft_link">
-        <kp>1e7</kp>
-        <kd>1e5</kd>
-        <mu1>1.5</mu1>
-        <mu2>1.5</mu2>
-        <!--<maxContacts>30</maxContacts>-->
-        <fdir1>1 0 0</fdir1>
-         <maxVel>0.0</maxVel>
-        <minDepth>0.001</minDepth>
-        <material>Gazebo/Orange</material>
-    </gazebo>
 </robot>

File: huron_description/urdf/huron_left_leg.xacro (robot description, xacro)
@@ -159,5 +159,5 @@
           <dynamics
             damping="0.5"
-            friction="4" />
+            friction="2" />
         </joint>
         <xacro:insert_transmission name="l_ankle_pitch_joint"/>
@@ -194,5 +194,5 @@
           <dynamics
             damping="0.5"
-            friction="4" />
+            friction="2" />
         </joint>
         <xacro:insert_transmission name="l_ankle_roll_joint"/>
@@ -209,116 +209,4 @@
             </inertial>
         </link>
-        <!-- left ft fixed joint 1 -->
-        <joint name="l1_ft_fixed" type="revolute">
-            <origin
-              xyz="0.098297 0.02083 0.12788"
-              rpy="0 0 ${pi/2}" />
-            <axis xyz="0 0 1"/>
-            <parent link="l_ankle_roll_link"/>
-            <child link="l1_foot_ft_link"/>
-            <limit
-            lower="0"
-            upper="0"
-            effort="100"
-            velocity="100" />
-        </joint>
-        <!-- left foot ft link 1 -->
-        <link name="l1_foot_ft_link">
-	    <visual>
-		<xacro:insert_mesh_l1_foot_ft_link />
-	    </visual>
-            <collision>
-                <xacro:insert_mesh_l1_foot_ft_link />
-            </collision>
-	    <inertial>
-		<xacro:insert_inertia_l1_foot_ft_link />
-	    </inertial>
-        </link>
-        <!-- left ft fixed joint 2 -->
-        <joint name="l2_ft_fixed" type="revolute">
-            <origin
-              xyz="0.098297 -0.01417 0.12788"
-              rpy="0 0 ${pi/2}" />
-            <axis xyz="0 0 1"/>
-            <parent link="l_ankle_roll_link"/>
-            <child link="l2_foot_ft_link"/>
-            <limit
-            lower="0"
-            upper="0"
-            effort="100"
-            velocity="100" />
-        </joint>
-        <!-- left foot ft link 2 -->
-        <link name="l2_foot_ft_link">
-	    <visual>
-		<xacro:insert_mesh_l2_foot_ft_link />
-	    </visual>
-            <collision>
-                <xacro:insert_mesh_l2_foot_ft_link />
-            </collision>
-	    <inertial>
-		<xacro:insert_inertia_l2_foot_ft_link />
-	    </inertial>
-        </link>
-        <!-- left ft fixed joint 3 -->
-        <joint name="l3_ft_fixed" type="revolute">
-            <origin
-              xyz="0.098297 -0.0165 0"
-              rpy="0 0 ${pi/2}" />
-            <axis xyz="0 0 1"/>
-            <parent link="l_ankle_roll_link"/>
-            <child link="l3_foot_ft_link"/>
-            <limit
-            lower="0"
-            upper="0"
-            effort="100"
-            velocity="100" />
-        </joint>
-        <!-- left foot ft link 3 -->
-        <link name="l3_foot_ft_link">
-	    <visual>
-		<xacro:insert_mesh_l3_foot_ft_link />
-	    </visual>
-            <collision>
-                <xacro:insert_mesh_l3_foot_ft_link />
-            </collision>
-	    <inertial>
-		<xacro:insert_inertia_l3_foot_ft_link />
-	    </inertial>
-        </link>
-        <!-- left ft fixed joint 4 -->
-        <joint name="l4_ft_fixed" type="revolute">
-            <origin
-              xyz="0.098297 0.017008 0"
-              rpy="0 0 ${pi/2}" />
-            <axis xyz="0 0 1"/>
-            <parent link="l_ankle_roll_link"/>
-            <child link="l4_foot_ft_link"/>
-            <limit
-            lower="0"
-            upper="0"
-            effort="100"
-            velocity="100" />
-        </joint>
-        <!-- left foot ft link 4 -->
-        <link name="l4_foot_ft_link">
-	    <visual>
-		<xacro:insert_mesh_l4_foot_ft_link />
-	    </visual>
-            <collision>
-                <xacro:insert_mesh_l4_foot_ft_link />
-            </collision>
-	    <inertial>
-		<xacro:insert_inertia_l4_foot_ft_link />
-	    </inertial>
-        </link>
-        <!-- left ft fixed joint -->
-        <joint name="lv_ft_fixed" type="fixed">
-            <origin xyz="0.045 0.0 0.0" rpy="0 ${-pi/2} 0"/>
-            <parent link="l4_foot_ft_link"/>
-            <child link="l_foot_v_ft_link"/>
-        </joint>
-        <!-- left foot ft link -->
-        <link name="l_foot_v_ft_link"></link>
     </xacro:macro>
 </robot>

File: huron_description/urdf/huron_right_leg.xacro (robot description, xacro)
@@ -164,5 +164,5 @@
           <dynamics
             damping="0.5"
-            friction="4" />
+            friction="2" />
         </joint>
         <xacro:insert_transmission name="r_ankle_pitch_joint"/>
@@ -199,5 +199,5 @@
           <dynamics
             damping="0.5"
-            friction="4" />
+            friction="2" />
         </joint>
         <xacro:insert_transmission name="r_ankle_roll_joint"/>
@@ -214,122 +214,4 @@
             </inertial>
         </link>
-       <!-- right ft fixed joint 1 -->
-        <joint name="r1_ft_fixed" type="revolute">
-            <origin
-              xyz="0.098297 0.01417 0.12788"
-              rpy="0 0 ${pi/2}" />
-            <axis xyz="0 0 1"/>
-            <parent link="r_ankle_roll_link"/>
-            <child link="r1_foot_ft_link"/>
-            <limit
-            lower="0"
-            upper="0"
-            effort="100"
-            velocity="100" />
-        </joint>
-        <!-- right foot ft link 1 -->
-        <link name="r1_foot_ft_link">
-	    <visual>
-		<xacro:insert_mesh_r1_foot_ft_link />
-	    </visual>
-            <collision>
-                <xacro:insert_mesh_r1_foot_ft_link />
-            </collision>
-	    <inertial>
-		<xacro:insert_inertia_r1_foot_ft_link />
-	    </inertial>
-        </link>
-        <!-- right ft fixed joint 2 -->
-        <joint name="r2_ft_fixed" type="revolute">
-            <origin
-              xyz="0.098297 -0.02083 0.12788"
-              rpy="0 0 ${pi/2}" />
-            <axis xyz="0 0 1"/>
-            <parent link="r_ankle_roll_link"/>
-            <child link="r2_foot_ft_link"/>
-            <limit
-            lower="0"
-            upper="0"
-            effort="100"
-            velocity="100" />
-        </joint>
-        <!-- right foot ft link 2 -->
-        <link name="r2_foot_ft_link">
-	    <visual>
-		<xacro:insert_mesh_r2_foot_ft_link />
-	    </visual>
-            <collision>
-                <xacro:insert_mesh_r2_foot_ft_link />
-            </collision>
-	    <inertial>
-		<xacro:insert_inertia_r2_foot_ft_link />
-	    </inertial>
-        </link>
-        <!-- right ft fixed joint 3 -->
-        <joint name="r3_ft_fixed" type="revolute">
-            <origin
-              xyz="0.098297 -0.017008 0"
-              rpy="0 0 ${pi/2}" />
-            <axis xyz="0 0 1"/>
-            <parent link="r_ankle_roll_link"/>
-            <child link="r3_foot_ft_link"/>
-            <limit
-            lower="0"
-            upper="0"
-            effort="100"
-            velocity="100" />
-        </joint>
-        <!-- right foot ft link 3 -->
-        <link name="r3_foot_ft_link">
-	    <visual>
-		<xacro:insert_mesh_r3_foot_ft_link />
-	    </visual>
-            <collision>
-                <xacro:insert_mesh_r3_foot_ft_link />
-            </collision>
-	    <inertial>
-		<xacro:insert_inertia_r3_foot_ft_link />
-	    </inertial>
-        </link>
-        <!-- right ft fixed joint 4 -->
-        <joint name="r4_ft_fixed" type="revolute">
-            <origin
-              xyz="0.098297 0.0165 0"
-              rpy="0 0 ${pi/2}" />
-            <axis xyz="0 0 1"/>
-            <parent link="r_ankle_roll_link"/>
-            <child link="r4_foot_ft_link"/>
-            <limit
-            lower="0"
-            upper="0"
-            effort="100"
-            velocity="100" />
-        </joint>
-        <!-- right4 foot ft link 4 -->
-        <link name="r4_foot_ft_link">
-	    <visual>
-		<xacro:insert_mesh_r4_foot_ft_link />
-	    </visual>
-            <collision>
-                <xacro:insert_mesh_r4_foot_ft_link />
-            </collision>
-	    <inertial>
-		<xacro:insert_inertia_r4_foot_ft_link />
-	    </inertial>
-        </link>
-        <!-- right ft fixed joint -->
-        <joint name="rv_ft_fixed" type="fixed">
-            <origin xyz="0.0 0.0 0.0" rpy="0 0 0"/>
-            <axis xyz="0 0 0"/>
-            <parent link="r4_foot_ft_link"/>
-            <child link="r_foot_v_ft_link"/>
-            <limit
-            lower="0"
-            upper="0"
-            effort="100"
-            velocity="100" />
-        </joint>
-        <!-- right foot ft link -->
-        <link name="r_foot_v_ft_link"></link>
     </xacro:macro>
 </robot>
