Commit message: test

File: huron_description/urdf/huron.urdf (robot description, URDF)
Before this commit: robot huron, 25 links, 24 joints
Joints:
- joint imu_fixed: origin xyz=0.0 0 0.45 rpy=0 0 0 -> xyz=0 0 0 rpy=0 0 0
- joint l1_ft_fixed: origin xyz=0.098328 0.020682 0.12788 rpy=-0.024938 0.00629 1.5706 -> xyz=0.095 0.020682 0.13788 rpy=-0.024938 0.00629 1.5706
- joint l2_ft_fixed: origin xyz=0.098275 -0.014318 0.12788 rpy=-0.024938 0.00629 1.5706 -> xyz=0.095 -0.014318 0.13788 rpy=-0.024938 0.00629 1.5706
- joint l3_ft_fixed: origin xyz=0.098272 -0.016649 0 rpy=-0.024938 0.00629 1.5706 -> xyz=0.095 -0.016649 -0.026 rpy=-0.024938 0.00629 1.5706
- joint l4_ft_fixed: origin xyz=0.098322 0.01686 0 rpy=-0.024938 0.00629 1.5706 -> xyz=0.095 0.01686 -0.026 rpy=-0.024938 0.00629 1.5706
- joint r1_ft_fixed: origin xyz=0.098271 0.014348 0.12788 rpy=-0.0095317 0.011124 1.5707 -> xyz=0.096 0.014348 0.13788 rpy=-0.0095317 0.011124 1.5707
- joint r2_ft_fixed: origin xyz=0.098334 -0.020652 0.12788 rpy=-0.0095317 0.011124 1.5707 -> xyz=0.096 -0.020652 0.13788 rpy=-0.0095317 0.011124 1.5707
- joint r3_ft_fixed: origin xyz=0.098328 -0.01683 0 rpy=-0.0095317 0.011124 1.5707 -> xyz=0.096 -0.01683 -0.026 rpy=-0.0095317 0.011124 1.5707
- joint r4_ft_fixed: origin xyz=0.098267 0.016679 0 rpy=-0.0095317 0.011124 1.5707 -> xyz=0.096 0.016679 -0.026 rpy=-0.0095317 0.011124 1.5707

File: huron_description/urdf/huron_gazebo.xacro (robot description, xacro)
@@ -186,4 +186,12 @@
         <mu1>0.9</mu1>
         <mu2>0.9</mu2>
+        <surface>
+          <contact>
+              <ode>
+                <kp>1e15</kp>
+                <kd>1e13</kd>
+              </ode>
+            </contact>
+        </surface>
         <!--<maxContacts>30</maxContacts>-->
         <fdir1>1 1 0</fdir1>
@@ -197,4 +205,12 @@
         <mu1>0.9</mu1>
         <mu2>0.9</mu2>
+        <surface>
+          <contact>
+              <ode>
+                <kp>1e15</kp>
+                <kd>1e13</kd>
+              </ode>
+            </contact>
+        </surface>
         <!--<maxContacts>30</maxContacts>-->
         <fdir1>1 1 0</fdir1>
@@ -208,4 +224,12 @@
         <mu1>0.9</mu1>
         <mu2>0.9</mu2>
+        <surface>
+          <contact>
+              <ode>
+                <kp>1e15</kp>
+                <kd>1e13</kd>
+              </ode>
+            </contact>
+        </surface>
         <!--<maxContacts>30</maxContacts>-->
         <fdir1>1 1 0</fdir1>
@@ -219,4 +243,12 @@
         <mu1>0.9</mu1>
         <mu2>0.9</mu2>
+        <surface>
+          <contact>
+              <ode>
+                <kp>1e15</kp>
+                <kd>1e13</kd>
+              </ode>
+            </contact>
+        </surface>
         <!--<maxContacts>30</maxContacts>-->
         <fdir1>1 1 0</fdir1>
@@ -272,4 +304,12 @@
         <mu1>0.9</mu1>
         <mu2>0.9</mu2>
+        <surface>
+          <contact>
+              <ode>
+                <kp>1e15</kp>
+                <kd>1e13</kd>
+              </ode>
+            </contact>
+        </surface>
         <!--<maxContacts>30</maxContacts>-->
         <fdir1>1 1 0</fdir1>
@@ -283,4 +323,12 @@
         <mu1>0.9</mu1>
         <mu2>0.9</mu2>
+        <surface>
+          <contact>
+              <ode>
+                <kp>1e15</kp>
+                <kd>1e13</kd>
+              </ode>
+            </contact>
+        </surface>
         <!--<maxContacts>30</maxContacts>-->
         <fdir1>1 1 0</fdir1>
@@ -294,4 +342,12 @@
         <mu1>0.9</mu1>
         <mu2>0.9</mu2>
+        <surface>
+          <contact>
+              <ode>
+                <kp>1e15</kp>
+                <kd>1e13</kd>
+              </ode>
+            </contact>
+        </surface>
         <!--<maxContacts>30</maxContacts>-->
         <fdir1>1 1 0</fdir1>
@@ -305,4 +361,12 @@
         <mu1>0.9</mu1>
         <mu2>0.9</mu2>
+        <surface>
+          <contact>
+              <ode>
+                <kp>1e15</kp>
+                <kd>1e13</kd>
+              </ode>
+            </contact>
+        </surface>
         <!--<maxContacts>30</maxContacts>-->
         <fdir1>1 1 0</fdir1>

File: huron_description/urdf/huron_inertia.xacro (robot description, xacro)
@@ -250,5 +250,5 @@
         rpy="0 0 0" />
       <mass
-        value="1.8531" />
+        value="1.8533" />
       <inertia
         ixx="0.0086813"

File: huron_description/urdf/huron_left_leg.xacro (robot description, xacro)
@@ -6,5 +6,5 @@
         <!-- left hip yaw joint -->
         <joint name="l_hip_yaw_joint" type="revolute">
-          <origin xyz="-0.0775 0 -0.14512" rpy="0 0 -0.0062919" />
+          <origin xyz="-0.0775 0 -0.14512" rpy="0 0 -0.0" />
           <parent link="${parent}" />
           <child link="l_hip_yaw_link" />
@@ -17,5 +17,5 @@
           <dynamics
             damping="0.5"
-            friction="100" />
+            friction="5" />
         </joint>
         <xacro:insert_transmission name="l_hip_yaw_joint"/>
@@ -38,5 +38,5 @@
           <origin
             xyz="0 0 0"
-            rpy="1.5708 0 3.1416" />
+            rpy="${pi/2} 0 ${pi}" />
           <parent
             link="l_hip_yaw_link" />
@@ -52,5 +52,5 @@
           <dynamics
             damping="0.5"
-            friction="100" />
+            friction="5" />
         </joint>
         <xacro:insert_transmission name="l_hip_roll_joint"/>
@@ -73,5 +73,5 @@
           <origin
             xyz="0 0 0"
-            rpy="-1.5707963267949 0 -1.5707963267949" />
+            rpy="${-pi/2} 0 ${-pi/2}" />
           <parent
             link="l_hip_roll_link" />
@@ -87,5 +87,5 @@
           <dynamics
             damping="0.5"
-            friction="100" />
+            friction="5" />
         </joint>
         <xacro:insert_transmission name="l_hip_pitch_joint"/>
@@ -107,5 +107,5 @@
           type="revolute">
           <origin
-            xyz="0.511278478308803 4.99999997527478E-05 1.66647320021251E-05"
+            xyz="0.512778478308813 4.99999997527478E-05 1.66647320021251E-05"
             rpy="0 0 0" />
           <parent
@@ -122,5 +122,5 @@
           <dynamics
             damping="0.5"
-            friction="100" />
+            friction="5" />
         </joint>
         <xacro:insert_transmission name="l_knee_pitch_joint"/>
@@ -143,5 +143,5 @@
           <origin
             xyz="0.370000000000016 3.16358752296964E-05 0.00249999999999911"
-            rpy="0 0 0.0249371730038869" />
+            rpy="0 0 0.0" />
           <parent
             link="l_knee_pitch_link" />
@@ -157,5 +157,5 @@
           <dynamics
             damping="0.5"
-            friction="100" />
+            friction="0.9" />
         </joint>
         <xacro:insert_transmission name="l_ankle_pitch_joint"/>
@@ -178,5 +178,5 @@
           <origin
             xyz="0 0 0"
-            rpy="1.57079632679489 0 0" />
+            rpy="${pi/2} 0 0" />
           <parent
             link="l_ankle_pitch_link" />
@@ -192,5 +192,5 @@
           <dynamics
             damping="0.5"
-            friction="100" />
+            friction="0.9" />
         </joint>
         <xacro:insert_transmission name="l_ankle_roll_joint"/>
@@ -210,6 +210,6 @@
         <joint name="l1_ft_fixed" type="revolute">
             <origin
-              xyz="0.098328 0.020682 0.12788"
-              rpy="-0.024938 0.00629 1.5706" />
+              xyz="0.096 0.020682 0.13788"
+              rpy="-0.0 0.0 ${pi/2}" />
             <axis xyz="0 0 1"/>
             <parent link="l_ankle_roll_link"/>
@@ -236,6 +236,6 @@
         <joint name="l2_ft_fixed" type="revolute">
             <origin
-              xyz="0.098275 -0.014318 0.12788"
-              rpy="-0.024938 0.00629 1.5706" />
+              xyz="0.096 -0.014318 0.13788"
+              rpy="-0.0 0.0 ${pi/2}" />
             <axis xyz="0 0 1"/>
             <parent link="l_ankle_roll_link"/>
@@ -262,6 +262,6 @@
         <joint name="l3_ft_fixed" type="revolute">
             <origin
-              xyz="0.098272 -0.016649 0"
-              rpy="-0.024938 0.00629 1.5706" />
+              xyz="0.096 -0.016649 -0.026"
+              rpy="-0.0 0.0 ${pi/2}" />
             <axis xyz="0 0 1"/>
             <parent link="l_ankle_roll_link"/>
@@ -288,6 +288,6 @@
         <joint name="l4_ft_fixed" type="revolute">
             <origin
-              xyz="0.098322 0.01686 0"
-              rpy="-0.024938 0.00629 1.5706" />
+              xyz="0.096 0.01686 -0.026"
+              rpy="-0.0 0.0 ${pi/2}" />
             <axis xyz="0 0 1"/>
             <parent link="l_ankle_roll_link"/>

File: huron_description/urdf/huron_right_leg.xacro (robot description, xacro)
@@ -10,5 +10,5 @@
           <origin
             xyz="0.0774999999999944 0 -0.1451242"
-            rpy="0 0 3.13046853298182" />
+            rpy="0 0 ${pi}" />
           <parent
             link="${parent}" />
@@ -24,5 +24,5 @@
           <dynamics
             damping="0.5"
-            friction="100" />
+            friction="5" />
         </joint>
         <xacro:insert_transmission name="r_hip_yaw_joint"/>
@@ -45,5 +45,5 @@
           <origin
             xyz="0 0 0"
-            rpy="1.5708 0 0" />
+            rpy="${pi/2} 0 0" />
           <parent
             link="r_hip_yaw_link" />
@@ -59,5 +59,5 @@
           <dynamics
             damping="0.5"
-            friction="100" />
+            friction="5" />
         </joint>
         <xacro:insert_transmission name="r_hip_roll_joint"/>
@@ -80,5 +80,5 @@
           <origin
             xyz="0 0 0"
-            rpy="-1.5708 0 -1.5708" />
+            rpy="${-pi/2} 0 ${-pi/2}" />
           <parent
             link="r_hip_roll_link" />
@@ -94,5 +94,5 @@
           <dynamics
             damping="0.5"
-            friction="100" />
+            friction="5" />
         </joint>
         <xacro:insert_transmission name="r_hip_pitch_joint"/>
@@ -129,5 +129,5 @@
           <dynamics
             damping="0.5"
-            friction="100" />
+            friction="5" />
         </joint>
         <xacro:insert_transmission name="r_knee_pitch_joint"/>
@@ -150,5 +150,5 @@
           <origin
             xyz="0.370000000000006 -3.16358749707368E-05 -0.00249999999999918"
-            rpy="0 0 0.0095311367408488" />
+            rpy="0 0 0.0" />
           <parent
             link="r_knee_pitch_link" />
@@ -164,5 +164,5 @@
           <dynamics
             damping="0.5"
-            friction="100" />
+            friction="0.9" />
         </joint>
         <xacro:insert_transmission name="r_ankle_pitch_joint"/>
@@ -185,5 +185,5 @@
           <origin
             xyz="0 0 0"
-            rpy="1.57079632679489 0 0" />
+            rpy="${pi/2} 0 0" />
           <parent
             link="r_ankle_pitch_link" />
@@ -199,5 +199,5 @@
           <dynamics
             damping="0.5"
-            friction="100" />
+            friction="0.9" />
         </joint>
         <xacro:insert_transmission name="r_ankle_roll_joint"/>
@@ -218,6 +218,6 @@
         <joint name="r1_ft_fixed" type="revolute">
             <origin
-              xyz="0.098271 0.014348 0.12788"
-              rpy="-0.0095317 0.011124 1.5707" />
+              xyz="0.096 0.014348 0.13788"
+              rpy="-0.0 0.0 ${pi/2}" />
             <axis xyz="0 0 1"/>
             <parent link="r_ankle_roll_link"/>
@@ -244,6 +244,6 @@
         <joint name="r2_ft_fixed" type="revolute">
             <origin
-              xyz="0.098334 -0.020652 0.12788"
-              rpy="-0.0095317 0.011124 1.5707" />
+              xyz="0.096 -0.020652 0.13788"
+              rpy="-0.0 0.0 ${pi/2}" />
             <axis xyz="0 0 1"/>
             <parent link="r_ankle_roll_link"/>
@@ -270,6 +270,6 @@
         <joint name="r3_ft_fixed" type="revolute">
             <origin
-              xyz="0.098328 -0.01683 0"
-              rpy="-0.0095317 0.011124 1.5707" />
+              xyz="0.096 -0.01683 -0.026"
+              rpy="-0.0 0.0 ${pi/2}" />
             <axis xyz="0 0 1"/>
             <parent link="r_ankle_roll_link"/>
@@ -296,6 +296,6 @@
         <joint name="r4_ft_fixed" type="revolute">
             <origin
-              xyz="0.098267 0.016679 0"
-              rpy="-0.0095317 0.011124 1.5707" />
+              xyz="0.096 0.016679 -0.026"
+              rpy="-0.0 0.0 ${pi/2}" />
             <axis xyz="0 0 1"/>
             <parent link="r_ankle_roll_link"/>

Commit message: Added battery

File: huron_description/urdf/huron.urdf (robot description, URDF)
Before this commit: robot huron, 25 links, 24 joints
Links:
- removed link l1_foot_ft_link
- removed link l2_foot_ft_link
- removed link l3_foot_ft_link
- removed link l4_foot_ft_link
- removed link l_foot_v_ft_link
- removed link r1_foot_ft_link
- removed link r2_foot_ft_link
- removed link r3_foot_ft_link
- removed link r4_foot_ft_link
- removed link r_foot_v_ft_link
- added link battery_link, mass 3.90089; collision box size=0.065 0.188 0.151; visual box size=0.065 0.188 0.151
- link r_ankle_roll_link: mass 1.8531 -> 1.8533
Joints:
- removed joint l1_ft_fixed
- removed joint l2_ft_fixed
- removed joint l3_ft_fixed
- removed joint l4_ft_fixed
- removed joint lv_ft_fixed
- removed joint r1_ft_fixed
- removed joint r2_ft_fixed
- removed joint r3_ft_fixed
- removed joint r4_ft_fixed
- removed joint rv_ft_fixed
- added joint battery_fixed: type fixed, parent base_footprint, child battery_link, origin xyz=0 0 0.0895 rpy=0 0 0
- joint l_ankle_pitch_joint: origin xyz=0.370000000000016 3.16358752296964E-05 0.00249999999999911 rpy=0 0 0.0249371730038869 -> xyz=0.370000000000016 3.16358752296964E-05 0.00249999999999911 rpy=0 0 0.0
- joint l_ankle_roll_joint: origin xyz=0 0 0 rpy=1.57079632679489 0 0 -> xyz=0 0 0 rpy=1.570796327 0 0
- joint l_hip_pitch_joint: origin xyz=0 0 0 rpy=-1.5707963267949 0 -1.5707963267949 -> xyz=0 0 0 rpy=-1.570796327 0 -1.570796327
- joint l_hip_roll_joint: origin xyz=0 0 0 rpy=1.5708 0 3.1416 -> xyz=0 0 0 rpy=1.570796327 0 3.141592654
- joint l_hip_yaw_joint: origin xyz=-0.0775 0 -0.14512 rpy=0 0 -0.0062919 -> xyz=-0.0775 0 -0.14512 rpy=0 0 -0.0
- joint l_knee_pitch_joint: origin xyz=0.511278478308803 4.99999997527478E-05 1.66647320021251E-05 rpy=0 0 0 -> xyz=0.512778478308813 4.99999997527478E-05 1.66647320021251E-05 rpy=0 0 0
- joint r_ankle_pitch_joint: origin xyz=0.370000000000006 -3.16358749707368E-05 -0.00249999999999918 rpy=0 0 0.0095311367408488 -> xyz=0.370000000000006 -3.16358749707368E-05 -0.00249999999999918 rpy=0 0 0.0
- joint r_ankle_roll_joint: origin xyz=0 0 0 rpy=1.57079632679489 0 0 -> xyz=0 0 0 rpy=1.570796327 0 0
- joint r_hip_pitch_joint: origin xyz=0 0 0 rpy=-1.5708 0 -1.5708 -> xyz=0 0 0 rpy=-1.570796327 0 -1.570796327
- joint r_hip_roll_joint: origin xyz=0 0 0 rpy=1.5708 0 0 -> xyz=0 0 0 rpy=1.570796327 0 0
- joint r_hip_yaw_joint: origin xyz=0.0774999999999944 0 -0.1451242 rpy=0 0 3.13046853298182 -> xyz=0.0774999999999944 0 -0.1451242 rpy=0 0 3.141592654

File: huron_description/urdf/huron.xacro (robot description, xacro)
@@ -36,4 +36,21 @@
         </inertial>
     </link>
+    <!-- Battery -->
+    <link name="battery_link">
+        <visual>
+            <xacro:insert_mesh_battery_link />
+        </visual>
+        <collision>
+            <xacro:insert_mesh_battery_link />
+        </collision>
+        <inertial>
+            <xacro:insert_inertia_battery_link />
+        </inertial>
+    </link>
+    <joint name="battery_fixed" type="fixed">
+        <origin xyz="0 0 0.0895" rpy="0 0 0"/>
+        <parent link="base_footprint"/>
+        <child link="battery_link"/>
+    </joint>
     <!-- imu joint -->
     <joint name="imu_fixed" type="fixed">

File: huron_description/urdf/huron_gazebo.xacro (robot description, xacro)
@@ -139,4 +139,9 @@
         <selfCollide>true</selfCollide>
     </gazebo>
+    <!-- Battery -->
+    <gazebo reference="battery_link">
+        <material>Gazebo/Cyan</material>
+        <selfCollide>true</selfCollide>
+    </gazebo>
     <!-- Left Leg -->
     <gazebo reference="l_hip_yaw_link">

File: huron_description/urdf/huron_inertia.xacro (robot description, xacro)
@@ -17,4 +17,19 @@
         izz="0.012315" />
     </xacro:macro>
+    <!-- Battery link -->
+    <xacro:macro name="insert_inertia_battery_link">
+      <origin
+        xyz="0 0 0"
+        rpy="0 0 0" />
+      <mass
+        value="3.90089" />
+      <inertia
+        ixx="0.01890143742"
+        ixy="0"
+        ixz="0"
+        iyy="0.0128628597"
+        iyz="0"
+        izz="0.008785454428" />
+    </xacro:macro>
     <!-- left hip yaw link -->
     <xacro:macro name="insert_inertia_l_hip_yaw_link">

File: huron_description/urdf/huron_left_leg.xacro (robot description, xacro)
@@ -157,5 +157,5 @@
           <dynamics
             damping="0.5"
-            friction="0.9" />
+            friction="2.5" />
         </joint>
         <xacro:insert_transmission name="l_ankle_pitch_joint"/>
@@ -192,5 +192,5 @@
           <dynamics
             damping="0.5"
-            friction="0.9" />
+            friction="2.5" />
         </joint>
         <xacro:insert_transmission name="l_ankle_roll_joint"/>

File: huron_description/urdf/huron_right_leg.xacro (robot description, xacro)
@@ -164,5 +164,5 @@
           <dynamics
             damping="0.5"
-            friction="0.9" />
+            friction="2.5" />
         </joint>
         <xacro:insert_transmission name="r_ankle_pitch_joint"/>
@@ -199,5 +199,5 @@
           <dynamics
             damping="0.5"
-            friction="0.9" />
+            friction="2.5" />
         </joint>
         <xacro:insert_transmission name="r_ankle_roll_joint"/>

File: huron_description/urdf/huron_visuals.xacro (robot description, xacro)
@@ -9,4 +9,12 @@
         </geometry>
         <material name="grey"/>
+    </xacro:macro>
+    <!-- Battery -->
+    <xacro:macro name="insert_mesh_battery_link">
+        <origin xyz="0 0 0" rpy="0 0 0" />
+        <geometry>
+            <box size="0.065 0.188 0.151" />
+        </geometry>
+        <material name="blue"/>
     </xacro:macro>
     <!-- left hip yaw link -->
