Commit message: Fixed CAD model and re-added force sensors

File: huron_description/urdf/huron.urdf (robot description, URDF)
Before this commit: robot huron, 16 links, 15 joints
Links:
- added link l1_foot_ft_link, mass 0.0086322; collision mesh filename=package://huron_description/meshes/r_foot_ft.STL scale=1 1 1; visual mesh filename=package://huron_description/meshes/r_foot_ft.STL scale=1 1 1
- added link l2_foot_ft_link, mass 0.00863223621815312; collision mesh filename=package://huron_description/meshes/r_foot_ft.STL scale=1 1 1; visual mesh filename=package://huron_description/meshes/r_foot_ft.STL scale=1 1 1
- added link l3_foot_ft_link, mass 0.00863223621815312; collision mesh filename=package://huron_description/meshes/r_foot_ft.STL scale=1 1 1; visual mesh filename=package://huron_description/meshes/r_foot_ft.STL scale=1 1 1
- added link l4_foot_ft_link, mass 0.00863223621815312; collision mesh filename=package://huron_description/meshes/r_foot_ft.STL scale=1 1 1; visual mesh filename=package://huron_description/meshes/r_foot_ft.STL scale=1 1 1
- added link l_foot_v_ft_link
- added link r1_foot_ft_link, mass 0.0086322; collision mesh filename=package://huron_description/meshes/r_foot_ft.STL scale=1 1 1; visual mesh filename=package://huron_description/meshes/r_foot_ft.STL scale=1 1 1
- added link r2_foot_ft_link, mass 0.00863223621815318; collision mesh filename=package://huron_description/meshes/r_foot_ft.STL scale=1 1 1; visual mesh filename=package://huron_description/meshes/r_foot_ft.STL scale=1 1 1
- added link r3_foot_ft_link, mass 0.00863223621815318; collision mesh filename=package://huron_description/meshes/r_foot_ft.STL scale=1 1 1; visual mesh filename=package://huron_description/meshes/r_foot_ft.STL scale=1 1 1
- added link r4_foot_ft_link, mass 0.00863223621815318; collision mesh filename=package://huron_description/meshes/r_foot_ft.STL scale=1 1 1; visual mesh filename=package://huron_description/meshes/r_foot_ft.STL scale=1 1 1
- added link r_foot_v_ft_link
Joints:
- added joint l1_ft_fixed: type revolute, parent l_ankle_roll_link, child l1_foot_ft_link, origin xyz=0.098328 0.020682 0.12788 rpy=-0.024938 0.00629 1.5706, axis 0 0 1, limit lower=0 upper=0 effort=100 velocity=100
- added joint l2_ft_fixed: type revolute, parent l_ankle_roll_link, child l2_foot_ft_link, origin xyz=0.098275 -0.014318 0.12788 rpy=-0.024938 0.00629 1.5706, axis 0 0 1, limit lower=0 upper=0 effort=100 velocity=100
- added joint l3_ft_fixed: type revolute, parent l_ankle_roll_link, child l3_foot_ft_link, origin xyz=0.098272 -0.016649 0 rpy=-0.024938 0.00629 1.5706, axis 0 0 1, limit lower=0 upper=0 effort=100 velocity=100
- added joint l4_ft_fixed: type revolute, parent l_ankle_roll_link, child l4_foot_ft_link, origin xyz=0.098322 0.01686 0 rpy=-0.024938 0.00629 1.5706, axis 0 0 1, limit lower=0 upper=0 effort=100 velocity=100
- added joint lv_ft_fixed: type fixed, parent l4_foot_ft_link, child l_foot_v_ft_link, origin xyz=0.045 0.0 0.0 rpy=0 -1.570796327 0
- added joint r1_ft_fixed: type revolute, parent r_ankle_roll_link, child r1_foot_ft_link, origin xyz=0.098271 0.014348 0.12788 rpy=-0.0095317 0.011124 1.5707, axis 0 0 1, limit lower=0 upper=0 effort=100 velocity=100
- added joint r2_ft_fixed: type revolute, parent r_ankle_roll_link, child r2_foot_ft_link, origin xyz=0.098334 -0.020652 0.12788 rpy=-0.0095317 0.011124 1.5707, axis 0 0 1, limit lower=0 upper=0 effort=100 velocity=100
- added joint r3_ft_fixed: type revolute, parent r_ankle_roll_link, child r3_foot_ft_link, origin xyz=0.098328 -0.01683 0 rpy=-0.0095317 0.011124 1.5707, axis 0 0 1, limit lower=0 upper=0 effort=100 velocity=100
- added joint r4_ft_fixed: type revolute, parent r_ankle_roll_link, child r4_foot_ft_link, origin xyz=0.098267 0.016679 0 rpy=-0.0095317 0.011124 1.5707, axis 0 0 1, limit lower=0 upper=0 effort=100 velocity=100
- added joint rv_ft_fixed: type fixed, parent r4_foot_ft_link, child r_foot_v_ft_link, origin xyz=0.0 0.0 0.0 rpy=0 0 0, axis 0 0 0, limit lower=0 upper=0 effort=100 velocity=100
- joint l_ankle_pitch_joint: limit lower=-3.1416 upper=3.1416 effort=1000 velocity=3 -> lower=-0.5236 upper=0.1745 effort=1000 velocity=3; origin xyz=0.370000000000016 3.16358752296964E-05 0.00249999999999911 rpy=0 0 0.0 -> xyz=0.3715 3.1633E-05 0.0025 rpy=0 0 0.0
- joint l_ankle_roll_joint: limit lower=-3.1416 upper=3.1416 effort=1000 velocity=3 -> lower=-0.3491 upper=0.3491 effort=1000 velocity=3
- joint l_hip_pitch_joint: limit lower=-3.1416 upper=3.1416 effort=1000 velocity=3 -> lower=-1.2217 upper=1.2217 effort=1000 velocity=3
- joint l_hip_roll_joint: limit lower=-3.1416 upper=3.1416 effort=1000 velocity=3 -> lower=-0.01 upper=0.5236 effort=1000 velocity=3
- joint l_knee_pitch_joint: limit lower=-3.1416 upper=3.1416 effort=1000 velocity=3 -> lower=-1.570796327 upper=1.570796327 effort=1000 velocity=3; origin xyz=0.512778478308813 4.99999997527478E-05 1.66647320021251E-05 rpy=0 0 0 -> xyz=0.511278478308821 5.00027201116859E-05 1.66647320003488E-05 rpy=0 0 0
- joint r_ankle_pitch_joint: limit lower=-3.1416 upper=3.1416 effort=1000 velocity=3 -> lower=-0.5236 upper=0.1745 effort=1000 velocity=3; origin xyz=0.370000000000006 -3.16358749707368E-05 -0.00249999999999918 rpy=0 0 0.0 -> xyz=0.370000000000006 -3.16358749707368E-05 -0.00249999999999943 rpy=0 0 0.0
- joint r_ankle_roll_joint: limit lower=-3.1416 upper=3.1416 effort=1000 velocity=3 -> lower=-0.3491 upper=0.3491 effort=1000 velocity=3
- joint r_hip_pitch_joint: limit lower=-3.1416 upper=3.1416 effort=1000 velocity=3 -> lower=-1.2217 upper=1.2217 effort=1000 velocity=3
- joint r_hip_roll_joint: limit lower=-3.1416 upper=3.1416 effort=1000 velocity=3 -> lower=-0.5236 upper=0.01 effort=1000 velocity=3
- joint r_knee_pitch_joint: limit lower=-3.1416 upper=3.1416 effort=1000 velocity=3 -> lower=-1.570796327 upper=1.570796327 effort=1000 velocity=3

File: huron_description/urdf/huron_gazebo.xacro (robot description, xacro)
@@ -141,5 +141,5 @@
     <!-- Battery -->
     <gazebo reference="battery_link">
-        <material>Gazebo/Cyan</material>
+        <material>Gazebo/SkyBlue</material>
         <selfCollide>true</selfCollide>
     </gazebo>
@@ -181,9 +181,53 @@
         <mu2>0.9</mu2>
         <!--<maxContacts>30</maxContacts>-->
-        <fdir1>1 1 0</fdir1>
+        <fdir1>1 0 0</fdir1>
         <maxVel>1.0</maxVel>
         <minDepth>0.001</minDepth>
         <material>Gazebo/Blue</material>
     </gazebo>
+    <gazebo reference="l1_foot_ft_link">
+        <kp>1e15</kp>
+        <kd>1e13</kd>
+        <mu1>0.9</mu1>
+        <mu2>0.9</mu2>
+        <!--<maxContacts>30</maxContacts>-->
+        <fdir1>1 0 0</fdir1>
+         <maxVel>1.0</maxVel>
+        <minDepth>0.0001</minDepth>
+        <material>Gazebo/Orange</material>
+    </gazebo>
+    <gazebo reference="l2_foot_ft_link">
+        <kp>1e15</kp>
+        <kd>1e13</kd>
+        <mu1>0.9</mu1>
+        <mu2>0.9</mu2>
+        <!--<maxContacts>30</maxContacts>-->
+        <fdir1>1 0 0</fdir1>
+         <maxVel>1.0</maxVel>
+        <minDepth>0.0001</minDepth>
+        <material>Gazebo/Orange</material>
+    </gazebo>
+    <gazebo reference="l3_foot_ft_link">
+        <kp>1e15</kp>
+        <kd>1e13</kd>
+        <mu1>0.9</mu1>
+        <mu2>0.9</mu2>
+        <!--<maxContacts>30</maxContacts>-->
+        <fdir1>1 0 0</fdir1>
+         <maxVel>1.0</maxVel>
+        <minDepth>0.0001</minDepth>
+        <material>Gazebo/Orange</material>
+    </gazebo>
+    <gazebo reference="l4_foot_ft_link">
+        <kp>1e15</kp>
+        <kd>1e13</kd>
+        <mu1>0.9</mu1>
+        <mu2>0.9</mu2>
+        <!--<maxContacts>30</maxContacts>-->
+        <fdir1>1 0 0</fdir1>
+         <maxVel>1.0</maxVel>
+        <minDepth>0.0001</minDepth>
+        <material>Gazebo/Orange</material>
+    </gazebo>
     <!-- Right Leg -->
     <gazebo reference="r_hip_yaw_link">
@@ -223,8 +267,52 @@
         <mu2>0.9</mu2>
         <!--<maxContacts>30</maxContacts>-->
-        <fdir1>1 1 0</fdir1>
+        <fdir1>1 0 0</fdir1>
          <maxVel>1.0</maxVel>
         <minDepth>0.0001</minDepth>
         <material>Gazebo/Blue</material>
     </gazebo>
+    <gazebo reference="r1_foot_ft_link">
+        <kp>1e15</kp>
+        <kd>1e13</kd>
+        <mu1>0.9</mu1>
+        <mu2>0.9</mu2>
+        <!--<maxContacts>30</maxContacts>-->
+        <fdir1>1 0 0</fdir1>
+         <maxVel>1.0</maxVel>
+        <minDepth>0.0001</minDepth>
+        <material>Gazebo/Orange</material>
+    </gazebo>
+    <gazebo reference="r2_foot_ft_link">
+        <kp>1e15</kp>
+        <kd>1e13</kd>
+        <mu1>0.9</mu1>
+        <mu2>0.9</mu2>
+        <!--<maxContacts>30</maxContacts>-->
+        <fdir1>1 0 0</fdir1>
+         <maxVel>1.0</maxVel>
+        <minDepth>0.0001</minDepth>
+        <material>Gazebo/Orange</material>
+    </gazebo>
+    <gazebo reference="r3_foot_ft_link">
+        <kp>1e15</kp>
+        <kd>1e13</kd>
+        <mu1>0.9</mu1>
+        <mu2>0.9</mu2>
+        <!--<maxContacts>30</maxContacts>-->
+        <fdir1>1 0 0</fdir1>
+         <maxVel>1.0</maxVel>
+        <minDepth>0.0001</minDepth>
+        <material>Gazebo/Orange</material>
+    </gazebo>
+    <gazebo reference="r4_foot_ft_link">
+        <kp>1e15</kp>
+        <kd>1e13</kd>
+        <mu1>0.9</mu1>
+        <mu2>0.9</mu2>
+        <!--<maxContacts>30</maxContacts>-->
+        <fdir1>1 0 0</fdir1>
+         <maxVel>1.0</maxVel>
+        <minDepth>0.0001</minDepth>
+        <material>Gazebo/Orange</material>
+    </gazebo>
 </robot>

File: huron_description/urdf/huron_inertia.xacro (robot description, xacro)
@@ -65,5 +65,5 @@
     <xacro:macro name="insert_inertia_l_hip_pitch_link">
       <origin
-        xyz="0.26603 4.6212E-05 0.053152"
+        xyz="0.26752 4.6211E-05 0.053152"
         rpy="0 0 0" />
       <mass
@@ -71,8 +71,8 @@
       <inertia
         ixx="0.0034527"
-        ixy="-3.1046E-08"
+        ixy="-3.1056E-08"
         ixz="0.0019797"
         iyy="0.010032"
-        iyz="-1.4492E-10"
+        iyz="-1.4618E-10"
         izz="0.01009" />
     </xacro:macro>
@@ -80,14 +80,14 @@
     <xacro:macro name="insert_inertia_l_knee_pitch_link">
       <origin
-        xyz="0.13395 0.00068098 0.00486"
+        xyz="0.13547 0.00068516 0.00486"
         rpy="0 0 0" />
       <mass
         value="3.4875" />
       <inertia
-        ixx="0.0064808"
-        ixy="1.3685E-05"
-        ixz="-2.8221E-05"
-        iyy="0.019763"
-        iyz="1.0351E-05"
+        ixx="0.0064814"
+        ixy="1.2524E-05"
+        ixz="-2.7966E-05"
+        iyy="0.019762"
+        iyz="1.0417E-05"
         izz="0.017354" />
     </xacro:macro>
@@ -102,7 +102,7 @@
         ixx="0.0025143"
         ixy="-0.00025651"
-        ixz="1.1648E-12"
+        ixz="1.1633E-12"
         iyy="0.0045125"
-        iyz="6.7198E-10"
+        iyz="6.7196E-10"
         izz="0.0049235" />
     </xacro:macro>
@@ -123,4 +123,64 @@
     </xacro:macro>
     <!-- Left foot sensors -->
+    <!-- l1_foot_ft link -->
+    <xacro:macro name="insert_inertia_l1_foot_ft_link">
+      <origin
+        xyz="7.3272E-06 0.0048383 4.6103E-08"
+        rpy="0 0 0" />
+      <mass
+        value="0.0086322" />
+      <inertia
+        ixx="3.8994E-07"
+        ixy="2.9118E-10"
+        ixz="2.9784E-10"
+        iyy="5.8221E-07"
+        iyz="1.8321E-12"
+        izz="3.4261E-07" />
+    </xacro:macro>
+    <!-- l2_foot_ft link  -->
+    <xacro:macro name="insert_inertia_l2_foot_ft_link">
+      <origin
+        xyz="7.32716003928879E-06 0.00483832570565201 4.61026197218217E-08"
+        rpy="0 0 0" />
+      <mass
+        value="0.00863223621815312" />
+      <inertia
+        ixx="3.89940334430996E-07"
+        ixy="2.91176476412897E-10"
+        ixz="2.9783895900032E-10"
+        iyy="5.82213619517231E-07"
+        iyz="1.83208753538184E-12"
+        izz="3.4260620679022E-07" />
+    </xacro:macro>
+    <!-- l3_foot_ft link 3 -->
+    <xacro:macro name="insert_inertia_l3_foot_ft_link">
+      <origin
+        xyz="7.32716003956635E-06 0.00483832570565224 4.61026188336433E-08"
+        rpy="0 0 0" />
+      <mass
+        value="0.00863223621815312" />
+      <inertia
+        ixx="3.89940334430996E-07"
+        ixy="2.9117647641293E-10"
+        ixz="2.97838959000262E-10"
+        iyy="5.82213619517231E-07"
+        iyz="1.83208753540344E-12"
+        izz="3.4260620679022E-07" />
+    </xacro:macro>
+    <!-- l4_foot_ft link 4 -->
+    <xacro:macro name="insert_inertia_l4_foot_ft_link">
+      <origin
+        xyz="7.32716003670753E-06 0.00483832570565246 4.61026209985782E-08"
+        rpy="0 0 0" />
+      <mass
+        value="0.00863223621815312" />
+      <inertia
+        ixx="3.89940334430996E-07"
+        ixy="2.91176476412812E-10"
+        ixz="2.97838959000613E-10"
+        iyy="5.82213619517231E-07"
+        iyz="1.83208753537968E-12"
+        izz="3.42606206790219E-07" />
+    </xacro:macro>
     <!-- Right leg -->
     <!-- right hip yaw link -->
@@ -163,8 +223,8 @@
       <inertia
         ixx="0.0034501"
-        ixy="-2.7561E-09"
+        ixy="-2.7593E-09"
         ixz="-0.0019797"
         iyy="0.010035"
-        iyz="2.5263E-10"
+        iyz="2.5351E-10"
         izz="0.01009" />
     </xacro:macro>
@@ -215,3 +275,63 @@
     </xacro:macro>
     <!-- Right foot sensors -->
+    <!-- r1_foot_ft link -->
+    <xacro:macro name="insert_inertia_r1_foot_ft_link">
+      <origin
+        xyz="-8.7899E-06 0.0048383 -9.7784E-08"
+        rpy="0 0 0" />
+      <mass
+        value="0.0086322" />
+      <inertia
+        ixx="3.8994E-07"
+        ixy="-3.4931E-10"
+        ixz="5.2655E-10"
+        iyy="5.8221E-07"
+        iyz="-3.8859E-12"
+        izz="3.4261E-07" />
+    </xacro:macro>
+    <!-- r2_foot_ft link  -->
+    <xacro:macro name="insert_inertia_r2_foot_ft_link">
+      <origin
+        xyz="-8.78991381628169E-06 0.00483832326857458 -9.77840948768183E-08"
+        rpy="0 0 0" />
+      <mass
+        value="0.00863223621815318" />
+      <inertia
+        ixx="3.89936544476746E-07"
+        ixy="-3.49305164752985E-10"
+        ixz="5.26550951245735E-10"
+        iyy="5.82213425821568E-07"
+        iyz="-3.88587306925662E-12"
+        izz="3.42610190440137E-07" />
+    </xacro:macro>
+    <!-- r_foot_ft link 3 -->
+    <xacro:macro name="insert_inertia_r3_foot_ft_link">
+      <origin
+        xyz="-8.78991381587924E-06 0.00483832326857436 -9.7784095154374E-08"
+        rpy="0 0 0" />
+      <mass
+        value="0.00863223621815318" />
+      <inertia
+        ixx="3.89936544476746E-07"
+        ixy="-3.49305164752997E-10"
+        ixz="5.26550951245753E-10"
+        iyy="5.82213425821568E-07"
+        iyz="-3.88587306930208E-12"
+        izz="3.42610190440137E-07" />
+    </xacro:macro>
+    <!-- r_foot_ft link 4 -->
+    <xacro:macro name="insert_inertia_r4_foot_ft_link">
+      <origin
+        xyz="-8.78991381597638E-06 0.00483832326857403 -9.7784095154374E-08"
+        rpy="0 0 0" />
+      <mass
+        value="0.00863223621815318" />
+      <inertia
+        ixx="3.89936544476746E-07"
+        ixy="-3.49305164753006E-10"
+        ixz="5.26550951245779E-10"
+        iyy="5.82213425821568E-07"
+        iyz="-3.88587306929652E-12"
+        izz="3.42610190440137E-07" />
+    </xacro:macro>
 </robot>

File: huron_description/urdf/huron_left_leg.xacro (robot description, xacro)
@@ -107,5 +107,5 @@
           type="revolute">
           <origin
-            xyz="0.512778478308813 4.99999997527478E-05 1.66647320021251E-05"
+            xyz="0.511278478308821 5.00027201116859E-05 1.66647320003488E-05"
             rpy="0 0 0" />
           <parent
@@ -142,5 +142,5 @@
           type="revolute">
           <origin
-            xyz="0.370000000000016 3.16358752296964E-05 0.00249999999999911"
+            xyz="0.3715 3.1633E-05 0.0025"
             rpy="0 0 0.0" />
           <parent
@@ -207,4 +207,116 @@
             </inertial>
         </link>
+        <!-- left ft fixed joint 1 -->
+        <joint name="l1_ft_fixed" type="revolute">
+            <origin
+              xyz="0.098328 0.020682 0.12788"
+              rpy="-0.024938 0.00629 1.5706" />
+            <axis xyz="0 0 1"/>
+            <parent link="l_ankle_roll_link"/>
+            <child link="l1_foot_ft_link"/>
+            <limit
+            lower="0"
+            upper="0"
+            effort="100"
+            velocity="100" />
+        </joint>
+        <!-- left foot ft link 1 -->
+        <link name="l1_foot_ft_link">
+	    <visual>
+		<xacro:insert_mesh_l1_foot_ft_link />
+	    </visual>
+            <collision>
+                <xacro:insert_mesh_l1_foot_ft_link />
+            </collision>
+	    <inertial>
+		<xacro:insert_inertia_l1_foot_ft_link />
+	    </inertial>
+        </link>
+        <!-- left ft fixed joint 2 -->
+        <joint name="l2_ft_fixed" type="revolute">
+            <origin
+              xyz="0.098275 -0.014318 0.12788"
+              rpy="-0.024938 0.00629 1.5706" />
+            <axis xyz="0 0 1"/>
+            <parent link="l_ankle_roll_link"/>
+            <child link="l2_foot_ft_link"/>
+            <limit
+            lower="0"
+            upper="0"
+            effort="100"
+            velocity="100" />
+        </joint>
+        <!-- left foot ft link 2 -->
+        <link name="l2_foot_ft_link">
+	    <visual>
+		<xacro:insert_mesh_l2_foot_ft_link />
+	    </visual>
+            <collision>
+                <xacro:insert_mesh_l2_foot_ft_link />
+            </collision>
+	    <inertial>
+		<xacro:insert_inertia_l2_foot_ft_link />
+	    </inertial>
+        </link>
+        <!-- left ft fixed joint 3 -->
+        <joint name="l3_ft_fixed" type="revolute">
+            <origin
+              xyz="0.098272 -0.016649 0"
+              rpy="-0.024938 0.00629 1.5706" />
+            <axis xyz="0 0 1"/>
+            <parent link="l_ankle_roll_link"/>
+            <child link="l3_foot_ft_link"/>
+            <limit
+            lower="0"
+            upper="0"
+            effort="100"
+            velocity="100" />
+        </joint>
+        <!-- left foot ft link 3 -->
+        <link name="l3_foot_ft_link">
+	    <visual>
+		<xacro:insert_mesh_l3_foot_ft_link />
+	    </visual>
+            <collision>
+                <xacro:insert_mesh_l3_foot_ft_link />
+            </collision>
+	    <inertial>
+		<xacro:insert_inertia_l3_foot_ft_link />
+	    </inertial>
+        </link>
+        <!-- left ft fixed joint 4 -->
+        <joint name="l4_ft_fixed" type="revolute">
+            <origin
+              xyz="0.098322 0.01686 0"
+              rpy="-0.024938 0.00629 1.5706" />
+            <axis xyz="0 0 1"/>
+            <parent link="l_ankle_roll_link"/>
+            <child link="l4_foot_ft_link"/>
+            <limit
+            lower="0"
+            upper="0"
+            effort="100"
+            velocity="100" />
+        </joint>
+        <!-- left foot ft link 4 -->
+        <link name="l4_foot_ft_link">
+	    <visual>
+		<xacro:insert_mesh_l4_foot_ft_link />
+	    </visual>
+            <collision>
+                <xacro:insert_mesh_l4_foot_ft_link />
+            </collision>
+	    <inertial>
+		<xacro:insert_inertia_l4_foot_ft_link />
+	    </inertial>
+        </link>
+        <!-- left ft fixed joint -->
+        <joint name="lv_ft_fixed" type="fixed">
+            <origin xyz="0.045 0.0 0.0" rpy="0 ${-pi/2} 0"/>
+            <parent link="l4_foot_ft_link"/>
+            <child link="l_foot_v_ft_link"/>
+        </joint>
+        <!-- left foot ft link -->
+        <link name="l_foot_v_ft_link"></link>
     </xacro:macro>
 </robot>
