Commit message: Fixed CAD model and re-added force sensors

File: huron_description/urdf/huron_right_leg.xacro (robot description, xacro)
@@ -149,5 +149,5 @@
           type="revolute">
           <origin
-            xyz="0.370000000000006 -3.16358749707368E-05 -0.00249999999999918"
+            xyz="0.370000000000006 -3.16358749707368E-05 -0.00249999999999943"
             rpy="0 0 0.0" />
           <parent
@@ -214,4 +214,122 @@
             </inertial>
         </link>
+       <!-- right ft fixed joint 1 -->
+        <joint name="r1_ft_fixed" type="revolute">
+            <origin
+              xyz="0.098271 0.014348 0.12788"
+              rpy="-0.0095317 0.011124 1.5707" />
+            <axis xyz="0 0 1"/>
+            <parent link="r_ankle_roll_link"/>
+            <child link="r1_foot_ft_link"/>
+            <limit
+            lower="0"
+            upper="0"
+            effort="100"
+            velocity="100" />
+        </joint>
+        <!-- right foot ft link 1 -->
+        <link name="r1_foot_ft_link">
+	    <visual>
+		<xacro:insert_mesh_r1_foot_ft_link />
+	    </visual>
+            <collision>
+                <xacro:insert_mesh_r1_foot_ft_link />
+            </collision>
+	    <inertial>
+		<xacro:insert_inertia_r1_foot_ft_link />
+	    </inertial>
+        </link>
+        <!-- right ft fixed joint 2 -->
+        <joint name="r2_ft_fixed" type="revolute">
+            <origin
+              xyz="0.098334 -0.020652 0.12788"
+              rpy="-0.0095317 0.011124 1.5707" />
+            <axis xyz="0 0 1"/>
+            <parent link="r_ankle_roll_link"/>
+            <child link="r2_foot_ft_link"/>
+            <limit
+            lower="0"
+            upper="0"
+            effort="100"
+            velocity="100" />
+        </joint>
+        <!-- right foot ft link 2 -->
+        <link name="r2_foot_ft_link">
+	    <visual>
+		<xacro:insert_mesh_r2_foot_ft_link />
+	    </visual>
+            <collision>
+                <xacro:insert_mesh_r2_foot_ft_link />
+            </collision>
+	    <inertial>
+		<xacro:insert_inertia_r2_foot_ft_link />
+	    </inertial>
+        </link>
+        <!-- right ft fixed joint 3 -->
+        <joint name="r3_ft_fixed" type="revolute">
+            <origin
+              xyz="0.098328 -0.01683 0"
+              rpy="-0.0095317 0.011124 1.5707" />
+            <axis xyz="0 0 1"/>
+            <parent link="r_ankle_roll_link"/>
+            <child link="r3_foot_ft_link"/>
+            <limit
+            lower="0"
+            upper="0"
+            effort="100"
+            velocity="100" />
+        </joint>
+        <!-- right foot ft link 3 -->
+        <link name="r3_foot_ft_link">
+	    <visual>
+		<xacro:insert_mesh_r3_foot_ft_link />
+	    </visual>
+            <collision>
+                <xacro:insert_mesh_r3_foot_ft_link />
+            </collision>
+	    <inertial>
+		<xacro:insert_inertia_r3_foot_ft_link />
+	    </inertial>
+        </link>
+        <!-- right ft fixed joint 4 -->
+        <joint name="r4_ft_fixed" type="revolute">
+            <origin
+              xyz="0.098267 0.016679 0"
+              rpy="-0.0095317 0.011124 1.5707" />
+            <axis xyz="0 0 1"/>
+            <parent link="r_ankle_roll_link"/>
+            <child link="r4_foot_ft_link"/>
+            <limit
+            lower="0"
+            upper="0"
+            effort="100"
+            velocity="100" />
+        </joint>
+        <!-- right4 foot ft link 4 -->
+        <link name="r4_foot_ft_link">
+	    <visual>
+		<xacro:insert_mesh_r4_foot_ft_link />
+	    </visual>
+            <collision>
+                <xacro:insert_mesh_r4_foot_ft_link />
+            </collision>
+	    <inertial>
+		<xacro:insert_inertia_r4_foot_ft_link />
+	    </inertial>
+        </link>
+        <!-- right ft fixed joint -->
+        <joint name="rv_ft_fixed" type="fixed">
+            <origin xyz="0.0 0.0 0.0" rpy="0 0 0"/>
+            <axis xyz="0 0 0"/>
+            <parent link="r4_foot_ft_link"/>
+            <child link="r_foot_v_ft_link"/>
+            <limit
+            lower="0"
+            upper="0"
+            effort="100"
+            velocity="100" />
+        </joint>
+        <!-- right foot ft link -->
+        <link name="r_foot_v_ft_link"></link>
     </xacro:macro>
 </robot>

File: huron_description/urdf/huron_visuals.xacro (robot description, xacro)
@@ -70,4 +70,36 @@
         </material>
     </xacro:macro>
+    <!-- l1_foot_ft link -->
+    <xacro:macro name="insert_mesh_l1_foot_ft_link">
+        <origin xyz="0 0 0" rpy=" 0 0 0" />
+        <geometry>
+            <mesh filename="package://huron_description/meshes/r_foot_ft.STL" scale="1 1 1" />
+        </geometry>
+        <material name="green"/>
+    </xacro:macro>
+    <!-- l2_foot_ft link  -->
+    <xacro:macro name="insert_mesh_l2_foot_ft_link">
+        <origin xyz="0 0 0" rpy=" 0 0 0" />
+        <geometry>
+            <mesh filename="package://huron_description/meshes/r_foot_ft.STL" scale="1 1 1" />
+        </geometry>
+        <material name="green"/>
+    </xacro:macro>
+    <!-- l3_foot_ft link 3 -->
+    <xacro:macro name="insert_mesh_l3_foot_ft_link">
+        <origin xyz="0 0 0" rpy=" 0 0 0" />
+        <geometry>
+            <mesh filename="package://huron_description/meshes/r_foot_ft.STL" scale="1 1 1" />
+        </geometry>
+        <material name="green"/>
+    </xacro:macro>
+    <!-- l4_foot_ft link 4 -->
+    <xacro:macro name="insert_mesh_l4_foot_ft_link">
+        <origin xyz="0 0 0" rpy=" 0 0 0" />
+        <geometry>
+            <mesh filename="package://huron_description/meshes/r_foot_ft.STL" scale="1 1 1" />
+        </geometry>
+        <material name="green"/>
+    </xacro:macro>
     <!-- right hip yaw link -->
     <xacro:macro name="insert_mesh_r_hip_yaw_link">
@@ -123,3 +155,35 @@
     </xacro:macro>
     <!-- Right foot sensors -->
+    <!-- r1_foot_ft link -->
+    <xacro:macro name="insert_mesh_r1_foot_ft_link">
+        <origin xyz="0 0 0" rpy=" 0 0 0" />
+        <geometry>
+            <mesh filename="package://huron_description/meshes/r_foot_ft.STL" scale="1 1 1" />
+        </geometry>
+        <material name="grey"/>
+    </xacro:macro>
+    <!-- r2_foot_ft link  -->
+    <xacro:macro name="insert_mesh_r2_foot_ft_link">
+        <origin xyz="0 0 0" rpy=" 0 0 0" />
+        <geometry>
+            <mesh filename="package://huron_description/meshes/r_foot_ft.STL" scale="1 1 1" />
+        </geometry>
+        <material name="grey"/>
+    </xacro:macro>
+    <!-- r3_foot_ft link 3-->
+    <xacro:macro name="insert_mesh_r3_foot_ft_link">
+        <origin xyz="0 0 0" rpy=" 0 0 0" />
+        <geometry>
+            <mesh filename="package://huron_description/meshes/r_foot_ft.STL" scale="1 1 1" />
+        </geometry>
+        <material name="grey"/>
+    </xacro:macro>
+    <!-- r4_foot_ft link 4 -->
+    <xacro:macro name="insert_mesh_r4_foot_ft_link">
+        <origin xyz="0 0 0" rpy=" 0 0 0" />
+        <geometry>
+            <mesh filename="package://huron_description/meshes/r_foot_ft.STL" scale="1 1 1" />
+        </geometry>
+        <material name="grey"/>
+    </xacro:macro>
 </robot>

Commit message: Base not fully attached to sensors

File: huron_description/urdf/huron.urdf (robot description, URDF)
Before this commit: robot huron, 26 links, 25 joints
Links:
- added link l_foot_base_link, mass 0.01; collision box size=0.078 0.005 0.221; visual box size=0.078 0.005 0.221
- added link r_foot_base_link, mass 0.01; collision box size=0.078 0.005 0.221; visual box size=0.078 0.005 0.221
Joints:
- added joint l_foot_base_fixed: type fixed, parent l1_foot_ft_link, child l_foot_base_link, origin xyz=-0.0175 -0.0025 -0.06395 rpy=0 0 0
- added joint r_foot_base_fixed: type fixed, parent r1_foot_ft_link, child r_foot_base_link, origin xyz=-0.0175 -0.0025 -0.06395 rpy=0 0 0
- joint l_knee_pitch_joint: origin xyz=0.511278478308821 5.00027201116859E-05 1.66647320003488E-05 rpy=0 0 0 -> xyz=0.512778478308813 5.00027201116859E-05 1.66647320003488E-05 rpy=0 0 0

File: huron_description/urdf/huron_gazebo.xacro (robot description, xacro)
@@ -176,5 +176,5 @@
     </gazebo>
     <gazebo reference="l_ankle_roll_link">
-         <kp>100000.0</kp>
+        <kp>100000.0</kp>
         <kd>100.0</kd>
         <mu1>0.9</mu1>
@@ -187,10 +187,10 @@
     </gazebo>
     <gazebo reference="l1_foot_ft_link">
-        <kp>1e15</kp>
-        <kd>1e13</kd>
-        <mu1>0.9</mu1>
-        <mu2>0.9</mu2>
-        <!--<maxContacts>30</maxContacts>-->
-        <fdir1>1 0 0</fdir1>
+        <kp>100000.0</kp>
+        <kd>100.0</kd>
+        <mu1>0.9</mu1>
+        <mu2>0.9</mu2>
+        <!--<maxContacts>30</maxContacts>-->
+        <!-- <fdir1>1 0 0</fdir1> -->
          <maxVel>1.0</maxVel>
         <minDepth>0.0001</minDepth>
@@ -198,10 +198,10 @@
     </gazebo>
     <gazebo reference="l2_foot_ft_link">
-        <kp>1e15</kp>
-        <kd>1e13</kd>
-        <mu1>0.9</mu1>
-        <mu2>0.9</mu2>
-        <!--<maxContacts>30</maxContacts>-->
-        <fdir1>1 0 0</fdir1>
+        <kp>100000.0</kp>
+        <kd>100.0</kd>
+        <mu1>0.9</mu1>
+        <mu2>0.9</mu2>
+        <!--<maxContacts>30</maxContacts>-->
+        <!-- <fdir1>1 0 0</fdir1> -->
          <maxVel>1.0</maxVel>
         <minDepth>0.0001</minDepth>
@@ -209,10 +209,10 @@
     </gazebo>
     <gazebo reference="l3_foot_ft_link">
-        <kp>1e15</kp>
-        <kd>1e13</kd>
-        <mu1>0.9</mu1>
-        <mu2>0.9</mu2>
-        <!--<maxContacts>30</maxContacts>-->
-        <fdir1>1 0 0</fdir1>
+        <kp>100000.0</kp>
+        <kd>100.0</kd>
+        <mu1>0.9</mu1>
+        <mu2>0.9</mu2>
+        <!--<maxContacts>30</maxContacts>-->
+        <!-- <fdir1>1 0 0</fdir1> -->
          <maxVel>1.0</maxVel>
         <minDepth>0.0001</minDepth>
@@ -220,10 +220,10 @@
     </gazebo>
     <gazebo reference="l4_foot_ft_link">
-        <kp>1e15</kp>
-        <kd>1e13</kd>
-        <mu1>0.9</mu1>
-        <mu2>0.9</mu2>
-        <!--<maxContacts>30</maxContacts>-->
-        <fdir1>1 0 0</fdir1>
+        <kp>100000.0</kp>
+        <kd>100.0</kd>
+        <mu1>0.9</mu1>
+        <mu2>0.9</mu2>
+        <!--<maxContacts>30</maxContacts>-->
+        <!-- <fdir1>1 0 0</fdir1> -->
          <maxVel>1.0</maxVel>
         <minDepth>0.0001</minDepth>
@@ -273,10 +273,10 @@
     </gazebo>
     <gazebo reference="r1_foot_ft_link">
-        <kp>1e15</kp>
-        <kd>1e13</kd>
-        <mu1>0.9</mu1>
-        <mu2>0.9</mu2>
-        <!--<maxContacts>30</maxContacts>-->
-        <fdir1>1 0 0</fdir1>
+        <kp>100000.0</kp>
+        <kd>100.0</kd>
+        <mu1>0.9</mu1>
+        <mu2>0.9</mu2>
+        <!--<maxContacts>30</maxContacts>-->
+        <!-- <fdir1>1 0 0</fdir1> -->
          <maxVel>1.0</maxVel>
         <minDepth>0.0001</minDepth>
@@ -284,10 +284,10 @@
     </gazebo>
     <gazebo reference="r2_foot_ft_link">
-        <kp>1e15</kp>
-        <kd>1e13</kd>
-        <mu1>0.9</mu1>
-        <mu2>0.9</mu2>
-        <!--<maxContacts>30</maxContacts>-->
-        <fdir1>1 0 0</fdir1>
+        <kp>100000.0</kp>
+        <kd>100.0</kd>
+        <mu1>0.9</mu1>
+        <mu2>0.9</mu2>
+        <!--<maxContacts>30</maxContacts>-->
+        <!-- <fdir1>1 0 0</fdir1> -->
          <maxVel>1.0</maxVel>
         <minDepth>0.0001</minDepth>
@@ -295,10 +295,10 @@
     </gazebo>
     <gazebo reference="r3_foot_ft_link">
-        <kp>1e15</kp>
-        <kd>1e13</kd>
-        <mu1>0.9</mu1>
-        <mu2>0.9</mu2>
-        <!--<maxContacts>30</maxContacts>-->
-        <fdir1>1 0 0</fdir1>
+        <kp>100000.0</kp>
+        <kd>100.0</kd>
+        <mu1>0.9</mu1>
+        <mu2>0.9</mu2>
+        <!--<maxContacts>30</maxContacts>-->
+        <!-- <fdir1>1 0 0</fdir1> -->
          <maxVel>1.0</maxVel>
         <minDepth>0.0001</minDepth>
@@ -306,13 +306,35 @@
     </gazebo>
     <gazebo reference="r4_foot_ft_link">
-        <kp>1e15</kp>
-        <kd>1e13</kd>
-        <mu1>0.9</mu1>
-        <mu2>0.9</mu2>
-        <!--<maxContacts>30</maxContacts>-->
-        <fdir1>1 0 0</fdir1>
-         <maxVel>1.0</maxVel>
-        <minDepth>0.0001</minDepth>
-        <material>Gazebo/Orange</material>
+        <kp>100000.0</kp>
+        <kd>100.0</kd>
+        <mu1>0.9</mu1>
+        <mu2>0.9</mu2>
+        <!--<maxContacts>30</maxContacts>-->
+        <!-- <fdir1>1 0 0</fdir1> -->
+         <maxVel>1.0</maxVel>
+        <minDepth>0.0001</minDepth>
+        <material>Gazebo/Orange</material>
+    </gazebo>
+    <gazebo reference="l_foot_base_link">
+        <kp>100000.0</kp>
+        <kd>100.0</kd>
+        <mu1>0.9</mu1>
+        <mu2>0.9</mu2>
+        <!--<maxContacts>30</maxContacts>-->
+        <!-- <fdir1>1 0 0</fdir1> -->
+         <maxVel>1.0</maxVel>
+        <minDepth>0.0001</minDepth>
+        <material>Gazebo/Green</material>
+    </gazebo>
+    <gazebo reference="r_foot_base_link">
+        <kp>100000.0</kp>
+        <kd>100.0</kd>
+        <mu1>0.9</mu1>
+        <mu2>0.9</mu2>
+        <!--<maxContacts>30</maxContacts>-->
+        <!-- <fdir1>1 0 0</fdir1> -->
+         <maxVel>1.0</maxVel>
+        <minDepth>0.0001</minDepth>
+        <material>Gazebo/Green</material>
     </gazebo>
 </robot>

File: huron_description/urdf/huron_inertia.xacro (robot description, xacro)
@@ -335,3 +335,18 @@
         izz="3.42610190440137E-07" />
     </xacro:macro>
+    <!-- Foot base link -->
+    <xacro:macro name="insert_inertia_foot_base_link">
+      <origin
+        xyz="0 0 0"
+        rpy="0 0 0" />
+      <mass
+        value="0.01" />
+      <inertia
+        ixx="4.448833333E-05"
+        ixy="0"
+        ixz="0"
+        iyy="4.95375E-05"
+        iyz="0"
+        izz="5.090833333E-06" />
+    </xacro:macro>
 </robot>

File: huron_description/urdf/huron_left_leg.xacro (robot description, xacro)
@@ -107,5 +107,5 @@
           type="revolute">
           <origin
-            xyz="0.511278478308821 5.00027201116859E-05 1.66647320003488E-05"
+            xyz="0.512778478308813 5.00027201116859E-05 1.66647320003488E-05"
             rpy="0 0 0" />
           <parent
@@ -210,6 +210,6 @@
         <joint name="l1_ft_fixed" type="revolute">
             <origin
-              xyz="0.098328 0.020682 0.12788"
-              rpy="-0.024938 0.00629 1.5706" />
+              xyz="0.0983282135717449 0.0206816111121677 0.127875866180865"
+              rpy="0 0 ${pi/2}" />
             <axis xyz="0 0 1"/>
             <parent link="l_ankle_roll_link"/>
@@ -236,6 +236,6 @@
         <joint name="l2_ft_fixed" type="revolute">
             <origin
-              xyz="0.098275 -0.014318 0.12788"
-              rpy="-0.024938 0.00629 1.5706" />
+              xyz="0.0982752085863122 -0.0143183487516882 0.127875866180865"
+              rpy="0 0 ${pi/2}" />
             <axis xyz="0 0 1"/>
             <parent link="l_ankle_roll_link"/>
@@ -262,6 +262,6 @@
         <joint name="l3_ft_fixed" type="revolute">
             <origin
-              xyz="0.098272 -0.016649 0"
-              rpy="-0.024938 0.00629 1.5706" />
+              xyz="0.0982716792139032 -0.0166488444898757 0"
+              rpy="0 0 ${pi/2}" />
             <axis xyz="0 0 1"/>
             <parent link="l_ankle_roll_link"/>
@@ -288,6 +288,6 @@
         <joint name="l4_ft_fixed" type="revolute">
             <origin
-              xyz="0.098322 0.01686 0"
-              rpy="-0.024938 0.00629 1.5706" />
+              xyz="0.0983224252792114 0.0168595176863209 0"
+              rpy="0 0 ${pi/2}" />
             <axis xyz="0 0 1"/>
             <parent link="l_ankle_roll_link"/>
@@ -319,4 +319,21 @@
         <!-- left foot ft link -->
         <link name="l_foot_v_ft_link"></link>
+        <!-- Foot base -->
+        <link name="l_foot_base_link">
+	    <visual>
+		<xacro:insert_mesh_foot_base_link />
+	    </visual>
+            <collision>
+                <xacro:insert_mesh_foot_base_link />
+            </collision>
+	    <inertial>
+		<xacro:insert_inertia_foot_base_link />
+	    </inertial>
+        </link>
+        <joint name="l_foot_base_fixed" type="fixed">
+            <origin xyz="-0.0175 -0.0025 -0.06395" rpy="0 0 0"/>
+            <parent link="l1_foot_ft_link"/>
+            <child link="l_foot_base_link"/>
+        </joint>
     </xacro:macro>
 </robot>

File: huron_description/urdf/huron_right_leg.xacro (robot description, xacro)
@@ -217,6 +217,6 @@
         <joint name="r1_ft_fixed" type="revolute">
             <origin
-              xyz="0.098271 0.014348 0.12788"
-              rpy="-0.0095317 0.011124 1.5707" />
+              xyz="0.0982708740959065 0.0143480673989493 0.127875866180863"
+              rpy="0 0 ${pi/2}" />
             <axis xyz="0 0 1"/>
             <parent link="r_ankle_roll_link"/>
@@ -243,6 +243,6 @@
         <joint name="r2_ft_fixed" type="revolute">
             <origin
-              xyz="0.098334 -0.020652 0.12788"
-              rpy="-0.0095317 0.011124 1.5707" />
+              xyz="0.0983344633797905 -0.0206518748353312 0.127875866180863"
+              rpy="0 0 ${pi/2}" />
             <axis xyz="0 0 1"/>
             <parent link="r_ankle_roll_link"/>
@@ -269,6 +269,6 @@
         <joint name="r3_ft_fixed" type="revolute">
             <origin
-              xyz="0.098328 -0.01683 0"
-              rpy="-0.0095317 0.011124 1.5707" />
+              xyz="0.0983275192522874 -0.0168297833346846 0"
+              rpy="0 0 ${pi/2}" />
             <axis xyz="0 0 1"/>
             <parent link="r_ankle_roll_link"/>
@@ -295,6 +295,6 @@
         <joint name="r4_ft_fixed" type="revolute">
             <origin
-              xyz="0.098267 0.016679 0"
-              rpy="-0.0095317 0.011124 1.5707" />
+              xyz="0.0982666399609057 0.0166785619632585 0"
+              rpy="0 0 ${pi/2}" />
             <axis xyz="0 0 1"/>
             <parent link="r_ankle_roll_link"/>
@@ -332,4 +332,21 @@
         <!-- right foot ft link -->
         <link name="r_foot_v_ft_link"></link>
+        <!-- Foot base -->
+        <link name="r_foot_base_link">
+	    <visual>
+		<xacro:insert_mesh_foot_base_link />
+	    </visual>
+            <collision>
+                <xacro:insert_mesh_foot_base_link />
+            </collision>
+	    <inertial>
+		<xacro:insert_inertia_foot_base_link />
+	    </inertial>
+        </link>
+        <joint name="r_foot_base_fixed" type="fixed">
+            <origin xyz="-0.0175 -0.0025 -0.06395" rpy="0 0 0"/>
+            <parent link="r1_foot_ft_link"/>
+            <child link="r_foot_base_link"/>
+        </joint>
     </xacro:macro>
 </robot>

File: huron_description/urdf/huron_visuals.xacro (robot description, xacro)
@@ -187,3 +187,11 @@
         <material name="grey"/>
     </xacro:macro>
+    <!-- Foot base -->
+    <xacro:macro name="insert_mesh_foot_base_link">
+        <origin xyz="0 0 0" rpy="0 0 0" />
+        <geometry>
+            <box size="0.078 0.005 0.231" />
+        </geometry>
+        <material name="green"/>
+    </xacro:macro>
 </robot>
