Commit message: Completely fixed CAD model

File: huron_description/urdf/huron.urdf (robot description, URDF)
Before this commit: robot huron, 28 links, 27 joints
Links:
- removed link l_foot_base_link
- removed link r_foot_base_link
- link l1_foot_ft_link: mass 0.0086322 -> 0.0061011; geometry collision mesh filename=package://huron_description/meshes/l1_foot_ft_link.STL scale=1 1 1; visual mesh filename=package://huron_description/meshes/l1_foot_ft_link.STL scale=1 1 1
- link l2_foot_ft_link: mass 0.00863223621815312 -> 0.00610112058812606; geometry collision mesh filename=package://huron_description/meshes/l2_foot_ft_link.STL scale=1 1 1; visual mesh filename=package://huron_description/meshes/l2_foot_ft_link.STL scale=1 1 1
- link l3_foot_ft_link: mass 0.00863223621815312 -> 0.00610112058812606; geometry collision mesh filename=package://huron_description/meshes/l3_foot_ft_link.STL scale=1 1 1; visual mesh filename=package://huron_description/meshes/l3_foot_ft_link.STL scale=1 1 1
- link l4_foot_ft_link: mass 0.00863223621815312 -> 0.00610112058812606; geometry collision mesh filename=package://huron_description/meshes/l4_foot_ft_link.STL scale=1 1 1; visual mesh filename=package://huron_description/meshes/l4_foot_ft_link.STL scale=1 1 1
- link l_ankle_roll_link: mass 1.8533 -> 1.8633
- link r1_foot_ft_link: mass 0.0086322 -> 0.00610112058812607; geometry collision mesh filename=package://huron_description/meshes/r1_foot_ft_link.STL scale=1 1 1; visual mesh filename=package://huron_description/meshes/r1_foot_ft_link.STL scale=1 1 1
- link r2_foot_ft_link: mass 0.00863223621815318 -> 0.00610112058812607; geometry collision mesh filename=package://huron_description/meshes/r2_foot_ft_link.STL scale=1 1 1; visual mesh filename=package://huron_description/meshes/r2_foot_ft_link.STL scale=1 1 1
- link r3_foot_ft_link: mass 0.00863223621815318 -> 0.00610112058812607; geometry collision mesh filename=package://huron_description/meshes/r3_foot_ft_link.STL scale=1 1 1; visual mesh filename=package://huron_description/meshes/r3_foot_ft_link.STL scale=1 1 1
- link r4_foot_ft_link: mass 0.00863223621815318 -> 0.00610112058812607; geometry collision mesh filename=package://huron_description/meshes/r4_foot_ft_link.STL scale=1 1 1; visual mesh filename=package://huron_description/meshes/r4_foot_ft_link.STL scale=1 1 1
- link r_ankle_roll_link: mass 1.8533 -> 1.8633
Joints:
- removed joint l_foot_base_fixed
- removed joint r_foot_base_fixed
- joint l1_ft_fixed: origin xyz=0.098328 0.020682 0.12788 rpy=-0.024938 0.00629 1.5706 -> xyz=0.098297 0.02083 0.12788 rpy=0 0 1.570796327
- joint l2_ft_fixed: origin xyz=0.098275 -0.014318 0.12788 rpy=-0.024938 0.00629 1.5706 -> xyz=0.098297 -0.01417 0.12788 rpy=0 0 1.570796327
- joint l3_ft_fixed: origin xyz=0.098272 -0.016649 0 rpy=-0.024938 0.00629 1.5706 -> xyz=0.098297 -0.0165 0 rpy=0 0 1.570796327
- joint l4_ft_fixed: origin xyz=0.098322 0.01686 0 rpy=-0.024938 0.00629 1.5706 -> xyz=0.098297 0.017008 0 rpy=0 0 1.570796327
- joint l_ankle_pitch_joint: origin xyz=0.3715 3.1633E-05 0.0025 rpy=0 0 0.0 -> xyz=0.37 0 0 rpy=0 0 0.0
- joint l_hip_pitch_joint: origin xyz=0 0 0 rpy=-1.570796327 0 -1.570796327 -> xyz=1.6665E-05 -0.0165 -5E-05 rpy=-1.570796327 0 -1.570796327
- joint l_hip_yaw_joint: origin xyz=-0.0775 0 -0.14512 rpy=0 0 -0.0 -> xyz=-0.0775000000000011 0 -0.1451242 rpy=0 0 0
- joint l_knee_pitch_joint: origin xyz=0.512778478308813 5.00027201116859E-05 1.66647320003488E-05 rpy=0 0 0 -> xyz=0.49628 0 0 rpy=0 0 0
- joint r1_ft_fixed: origin xyz=0.098271 0.014348 0.12788 rpy=-0.0095317 0.011124 1.5707 -> xyz=0.098297 0.01417 0.12788 rpy=0 0 1.570796327
- joint r2_ft_fixed: origin xyz=0.098334 -0.020652 0.12788 rpy=-0.0095317 0.011124 1.5707 -> xyz=0.098297 -0.02083 0.12788 rpy=0 0 1.570796327
- joint r3_ft_fixed: origin xyz=0.098328 -0.01683 0 rpy=-0.0095317 0.011124 1.5707 -> xyz=0.098297 -0.017008 0 rpy=0 0 1.570796327
- joint r4_ft_fixed: origin xyz=0.098267 0.016679 0 rpy=-0.0095317 0.011124 1.5707 -> xyz=0.098297 0.0165 0 rpy=0 0 1.570796327
- joint r_ankle_pitch_joint: origin xyz=0.370000000000006 -3.16358749707368E-05 -0.00249999999999943 rpy=0 0 0.0 -> xyz=0.37 0 0 rpy=0 0 0.0
- joint r_hip_pitch_joint: origin xyz=0 0 0 rpy=-1.570796327 0 -1.570796327 -> xyz=-1.6665E-05 -0.0165 -5E-05 rpy=-1.570796327 0 -1.570796327
- joint r_hip_yaw_joint: origin xyz=0.0774999999999944 0 -0.1451242 rpy=0 0 3.141592654 -> xyz=0.0775 0 -0.14512 rpy=0 0 3.141592654
- joint r_knee_pitch_joint: origin xyz=0.512778478308813 4.99999999867273E-05 -1.66647320091612E-05 rpy=0 0 0 -> xyz=0.49628 0 0 rpy=0 0 0

File: huron_description/urdf/huron_gazebo.xacro (robot description, xacro)
@@ -137,10 +137,10 @@
         <mu2>0.2</mu2>
         <material>Gazebo/Grey</material>
-        <selfCollide>true</selfCollide>
+        <selfCollide>false</selfCollide>
     </gazebo>
     <!-- Battery -->
     <gazebo reference="battery_link">
         <material>Gazebo/SkyBlue</material>
-        <selfCollide>true</selfCollide>
+        <selfCollide>false</selfCollide>
     </gazebo>
     <!-- Left Leg -->
@@ -149,5 +149,5 @@
         <mu2>0.2</mu2>
         <material>Gazebo/Grey</material>
-        <selfCollide>true</selfCollide>
+        <selfCollide>false</selfCollide>
     </gazebo>
     <gazebo reference="l_hip_roll_link">
@@ -155,5 +155,5 @@
         <mu2>0.2</mu2>
         <material>Gazebo/Grey</material>
-        <selfCollide>true</selfCollide>
+        <selfCollide>false</selfCollide>
     </gazebo>
     <gazebo reference="l_hip_pitch_link">
@@ -161,5 +161,5 @@
         <mu2>0.2</mu2>
         <material>Gazebo/Grey</material>
-        <selfCollide>true</selfCollide>
+        <selfCollide>false</selfCollide>
     </gazebo>
     <gazebo reference="l_knee_pitch_link">
@@ -167,5 +167,5 @@
         <mu2>0.2</mu2>
         <material>Gazebo/Grey</material>
-        <selfCollide>true</selfCollide>
+        <selfCollide>false</selfCollide>
     </gazebo>
     <gazebo reference="l_ankle_pitch_link">
@@ -173,145 +173,145 @@
         <mu2>0.2</mu2>
         <material>Gazebo/Grey</material>
-        <selfCollide>true</selfCollide>
+        <selfCollide>false</selfCollide>
     </gazebo>
     <gazebo reference="l_ankle_roll_link">
-        <kp>100000.0</kp>
-        <kd>100.0</kd>
+        <!-- <kp>100000.0</kp> -->
+        <!-- <kd>100.0</kd> -->
         <mu1>0.9</mu1>
         <mu2>0.9</mu2>
         <!--<maxContacts>30</maxContacts>-->
-        <fdir1>1 0 0</fdir1>
-        <maxVel>1.0</maxVel>
-        <minDepth>0.001</minDepth>
+        <!-- <fdir1>1 0 0</fdir1> -->
+        <!-- <maxVel>1.0</maxVel> -->
+        <!-- <minDepth>0.001</minDepth> -->
         <material>Gazebo/Blue</material>
     </gazebo>
     <gazebo reference="l1_foot_ft_link">
-        <kp>100000.0</kp>
-        <kd>100.0</kd>
+        <kp>1e7</kp>
+        <kd>1e5</kd>
+        <mu1>1.5</mu1>
+        <mu2>1.5</mu2>
+        <!--<maxContacts>30</maxContacts>-->
+        <fdir1>1 0 0</fdir1>
+         <maxVel>0.0</maxVel>
+        <minDepth>0.001</minDepth>
+        <material>Gazebo/Orange</material>
+    </gazebo>
+    <gazebo reference="l2_foot_ft_link">
+        <kp>1e7</kp>
+        <kd>1e5</kd>
+        <mu1>1.5</mu1>
+        <mu2>1.5</mu2>
+        <!--<maxContacts>30</maxContacts>-->
+        <fdir1>1 0 0</fdir1>
+         <maxVel>0.0</maxVel>
+        <minDepth>0.001</minDepth>
+        <material>Gazebo/Orange</material>
+    </gazebo>
+    <gazebo reference="l3_foot_ft_link">
+        <kp>1e7</kp>
+        <kd>1e5</kd>
+        <mu1>1.5</mu1>
+        <mu2>1.5</mu2>
+        <!--<maxContacts>30</maxContacts>-->
+        <fdir1>1 0 0</fdir1>
+         <maxVel>0.0</maxVel>
+        <minDepth>0.001</minDepth>
+        <material>Gazebo/Orange</material>
+    </gazebo>
+    <gazebo reference="l4_foot_ft_link">
+        <kp>1e7</kp>
+        <kd>1e5</kd>
+        <mu1>1.5</mu1>
+        <mu2>1.5</mu2>
+        <!--<maxContacts>30</maxContacts>-->
+        <fdir1>1 0 0</fdir1>
+         <maxVel>0.0</maxVel>
+        <minDepth>0.001</minDepth>
+        <material>Gazebo/Orange</material>
+    </gazebo>
+    <!-- Right Leg -->
+    <gazebo reference="r_hip_yaw_link">
+        <mu1>0.2</mu1>
+        <mu2>0.2</mu2>
+        <material>Gazebo/Grey</material>
+        <selfCollide>false</selfCollide>
+    </gazebo>
+    <gazebo reference="r_hip_roll_link">
+        <mu1>0.2</mu1>
+        <mu2>0.2</mu2>
+        <material>Gazebo/Grey</material>
+        <selfCollide>false</selfCollide>
+    </gazebo>
+    <gazebo reference="r_hip_pitch_link">
+        <mu1>0.2</mu1>
+        <mu2>0.2</mu2>
+        <material>Gazebo/Grey</material>
+        <selfCollide>false</selfCollide>
+    </gazebo>
+    <gazebo reference="r_knee_pitch_link">
+        <mu1>0.2</mu1>
+        <mu2>0.2</mu2>
+        <material>Gazebo/Grey</material>
+        <selfCollide>false</selfCollide>
+    </gazebo>
+    <gazebo reference="r_ankle_pitch_link">
+        <mu1>0.2</mu1>
+        <mu2>0.2</mu2>
+        <material>Gazebo/Grey</material>
+        <selfCollide>false</selfCollide>
+    </gazebo>
+    <gazebo reference="r_ankle_roll_link">
+        <!-- <kp>100000.0</kp> -->
+        <!-- <kd>100.0</kd> -->
         <mu1>0.9</mu1>
         <mu2>0.9</mu2>
         <!--<maxContacts>30</maxContacts>-->
         <!-- <fdir1>1 0 0</fdir1> -->
-         <maxVel>1.0</maxVel>
-        <minDepth>0.0001</minDepth>
-        <material>Gazebo/Orange</material>
-    </gazebo>
-    <gazebo reference="l2_foot_ft_link">
-        <kp>100000.0</kp>
-        <kd>100.0</kd>
-        <mu1>0.9</mu1>
-        <mu2>0.9</mu2>
-        <!--<maxContacts>30</maxContacts>-->
-        <!-- <fdir1>1 0 0</fdir1> -->
-         <maxVel>1.0</maxVel>
-        <minDepth>0.0001</minDepth>
-        <material>Gazebo/Orange</material>
-    </gazebo>
-    <gazebo reference="l3_foot_ft_link">
-        <kp>100000.0</kp>
-        <kd>100.0</kd>
-        <mu1>0.9</mu1>
-        <mu2>0.9</mu2>
-        <!--<maxContacts>30</maxContacts>-->
-        <!-- <fdir1>1 0 0</fdir1> -->
-         <maxVel>1.0</maxVel>
-        <minDepth>0.0001</minDepth>
-        <material>Gazebo/Orange</material>
-    </gazebo>
-    <gazebo reference="l4_foot_ft_link">
-        <kp>100000.0</kp>
-        <kd>100.0</kd>
-        <mu1>0.9</mu1>
-        <mu2>0.9</mu2>
-        <!--<maxContacts>30</maxContacts>-->
-        <!-- <fdir1>1 0 0</fdir1> -->
-         <maxVel>1.0</maxVel>
-        <minDepth>0.0001</minDepth>
-        <material>Gazebo/Orange</material>
-    </gazebo>
-    <!-- Right Leg -->
-    <gazebo reference="r_hip_yaw_link">
-        <mu1>0.2</mu1>
-        <mu2>0.2</mu2>
-        <material>Gazebo/Grey</material>
-        <selfCollide>true</selfCollide>
-    </gazebo>
-    <gazebo reference="r_hip_roll_link">
-        <mu1>0.2</mu1>
-        <mu2>0.2</mu2>
-        <material>Gazebo/Grey</material>
-        <selfCollide>true</selfCollide>
-    </gazebo>
-    <gazebo reference="r_hip_pitch_link">
-        <mu1>0.2</mu1>
-        <mu2>0.2</mu2>
-        <material>Gazebo/Grey</material>
-        <selfCollide>true</selfCollide>
-    </gazebo>
-    <gazebo reference="r_knee_pitch_link">
-        <mu1>0.2</mu1>
-        <mu2>0.2</mu2>
-        <material>Gazebo/Grey</material>
-        <selfCollide>true</selfCollide>
-    </gazebo>
-    <gazebo reference="r_ankle_pitch_link">
-        <mu1>0.2</mu1>
-        <mu2>0.2</mu2>
-        <material>Gazebo/Grey</material>
-        <selfCollide>true</selfCollide>
-    </gazebo>
-    <gazebo reference="r_ankle_roll_link">
-        <kp>100000.0</kp>
-        <kd>100.0</kd>
-        <mu1>0.9</mu1>
-        <mu2>0.9</mu2>
-        <!--<maxContacts>30</maxContacts>-->
-        <fdir1>1 0 0</fdir1>
-         <maxVel>1.0</maxVel>
-        <minDepth>0.0001</minDepth>
+        <!--  <maxVel>1.0</maxVel>  -->
+        <!-- <minDepth>0.0001</minDepth> -->
         <material>Gazebo/Blue</material>
     </gazebo>
     <gazebo reference="r1_foot_ft_link">
-        <kp>100000.0</kp>
-        <kd>100.0</kd>
-        <mu1>0.9</mu1>
-        <mu2>0.9</mu2>
-        <!--<maxContacts>30</maxContacts>-->
-        <!-- <fdir1>1 0 0</fdir1> -->
-         <maxVel>1.0</maxVel>
-        <minDepth>0.0001</minDepth>
+        <kp>1e7</kp>
+        <kd>1e5</kd>
+        <mu1>1.5</mu1>
+        <mu2>1.5</mu2>
+        <!--<maxContacts>30</maxContacts>-->
+        <fdir1>1 0 0</fdir1>
+         <maxVel>0.0</maxVel>
+        <minDepth>0.001</minDepth>
         <material>Gazebo/Orange</material>
     </gazebo>
     <gazebo reference="r2_foot_ft_link">
-        <kp>100000.0</kp>
-        <kd>100.0</kd>
-        <mu1>0.9</mu1>
-        <mu2>0.9</mu2>
-        <!--<maxContacts>30</maxContacts>-->
-        <!-- <fdir1>1 0 0</fdir1> -->
-         <maxVel>1.0</maxVel>
-        <minDepth>0.0001</minDepth>
+        <kp>1e7</kp>
+        <kd>1e5</kd>
+        <mu1>1.5</mu1>
+        <mu2>1.5</mu2>
+        <!--<maxContacts>30</maxContacts>-->
+        <fdir1>1 0 0</fdir1>
+         <maxVel>0.0</maxVel>
+        <minDepth>0.001</minDepth>
         <material>Gazebo/Orange</material>
     </gazebo>
     <gazebo reference="r3_foot_ft_link">
-        <kp>100000.0</kp>
-        <kd>100.0</kd>
-        <mu1>0.9</mu1>
-        <mu2>0.9</mu2>
-        <!--<maxContacts>30</maxContacts>-->
-        <!-- <fdir1>1 0 0</fdir1> -->
-         <maxVel>1.0</maxVel>
-        <minDepth>0.0001</minDepth>
+        <kp>1e7</kp>
+        <kd>1e5</kd>
+        <mu1>1.5</mu1>
+        <mu2>1.5</mu2>
+        <!--<maxContacts>30</maxContacts>-->
+        <fdir1>1 0 0</fdir1>
+         <maxVel>0.0</maxVel>
+        <minDepth>0.001</minDepth>
         <material>Gazebo/Orange</material>
     </gazebo>
     <gazebo reference="r4_foot_ft_link">
-        <kp>100000.0</kp>
-        <kd>100.0</kd>
-        <mu1>0.9</mu1>
-        <mu2>0.9</mu2>
-        <!--<maxContacts>30</maxContacts>-->
-        <!-- <fdir1>1 0 0</fdir1> -->
-         <maxVel>1.0</maxVel>
-        <minDepth>0.0001</minDepth>
+        <kp>1e7</kp>
+        <kd>1e5</kd>
+        <mu1>1.5</mu1>
+        <mu2>1.5</mu2>
+        <!--<maxContacts>30</maxContacts>-->
+        <fdir1>1 0 0</fdir1>
+         <maxVel>0.0</maxVel>
+        <minDepth>0.001</minDepth>
         <material>Gazebo/Orange</material>
     </gazebo>
