Commit message: Completely fixed CAD model

File: huron_description/urdf/huron_inertia.xacro (robot description, xacro)
@@ -5,5 +5,5 @@
     <xacro:macro name="insert_inertia_base_link">
       <origin
-        xyz="4.7319E-09 5.4338E-07 0.026975"
+        xyz="-1.3585E-07 5.07E-07 0.026975"
         rpy="0 0 0" />
       <mass
@@ -11,8 +11,8 @@
       <inertia
         ixx="0.00319"
-        ixy="7.149E-11"
-        ixz="6.0313E-11"
+        ixy="-1.7776E-09"
+        ixz="-1.7316E-09"
         iyy="0.010531"
-        iyz="6.926E-09"
+        iyz="6.4623E-09"
         izz="0.012315" />
     </xacro:macro>
@@ -41,5 +41,5 @@
       <inertia
         ixx="0.0022702"
-        ixy="-2.5061E-10"
+        ixy="-2.4951E-10"
         ixz="6.6464E-06"
         iyy="0.0026746"
@@ -56,8 +56,8 @@
       <inertia
         ixx="0.00098222"
-        ixy="-9.9265E-08"
-        ixz="4.9766E-09"
+        ixy="-9.9267E-08"
+        ixz="4.9764E-09"
         iyy="0.00097045"
-        iyz="-9.7282E-08"
+        iyz="-9.7285E-08"
         izz="0.00092365" />
     </xacro:macro>
@@ -65,14 +65,14 @@
     <xacro:macro name="insert_inertia_l_hip_pitch_link">
       <origin
-        xyz="0.26752 4.6211E-05 0.053152"
+        xyz="0.25103 -7.7295E-06 0.053135"
         rpy="0 0 0" />
       <mass
         value="4.2544" />
       <inertia
-        ixx="0.0034527"
-        ixy="-3.1056E-08"
+        ixx="0.0034501"
+        ixy="-1.1102E-07"
         ixz="0.0019797"
-        iyy="0.010032"
-        iyz="-1.4618E-10"
+        iyy="0.010035"
+        iyz="-4.8767E-10"
         izz="0.01009" />
     </xacro:macro>
@@ -80,5 +80,5 @@
     <xacro:macro name="insert_inertia_l_knee_pitch_link">
       <origin
-        xyz="0.13547 0.00068516 0.00486"
+        xyz="0.13397 0.00066001 0.0028723"
         rpy="0 0 0" />
       <mass
@@ -95,5 +95,5 @@
     <xacro:macro name="insert_inertia_l_ankle_pitch_link">
       <origin
-        xyz="-0.029808 0.001045 3.1135E-08"
+        xyz="-0.029808 0.001045 3.1134E-08"
         rpy="0 0 0" />
       <mass
@@ -104,5 +104,5 @@
         ixz="1.1633E-12"
         iyy="0.0045125"
-        iyz="6.7196E-10"
+        iyz="6.7197E-10"
         izz="0.0049235" />
     </xacro:macro>
@@ -110,15 +110,15 @@
     <xacro:macro name="insert_inertia_l_ankle_roll_link">
       <origin
-        xyz="0.073422 -5.3261E-05 0.063946"
-        rpy="0 0 0" />
-      <mass
-        value="1.8533" />
-      <inertia
-        ixx="0.008682"
-        ixy="-1.0255E-05"
-        ixz="0.00024351"
-        iyy="0.0084057"
-        iyz="0.00012332"
-        izz="0.0013019" />
+        xyz="0.07353 6.708E-05 0.063947"
+        rpy="0 0 0" />
+      <mass
+        value="1.8633" />
+      <inertia
+        ixx="0.0086824"
+        ixy="-9.8353E-06"
+        ixz="0.00024334"
+        iyy="0.0084059"
+        iyz="0.00012379"
+        izz="0.0013021" />
     </xacro:macro>
     <!-- Left foot sensors -->
@@ -126,60 +126,60 @@
     <xacro:macro name="insert_inertia_l1_foot_ft_link">
       <origin
-        xyz="7.3272E-06 0.0048383 4.6103E-08"
-        rpy="0 0 0" />
-      <mass
-        value="0.0086322" />
-      <inertia
-        ixx="3.8994E-07"
-        ixy="2.9118E-10"
-        ixz="2.9784E-10"
-        iyy="5.8221E-07"
-        iyz="1.8321E-12"
-        izz="3.4261E-07" />
+        xyz="-5.7176E-15 0.0047713 3.2752E-15"
+        rpy="0 0 0" />
+      <mass
+        value="0.0061011" />
+      <inertia
+        ixx="3.1713E-07"
+        ixy="3.8307E-22"
+        ixz="-1.1921E-22"
+        iyy="4.8773E-07"
+        iyz="-1.0683E-22"
+        izz="3.1713E-07" />
     </xacro:macro>
     <!-- l2_foot_ft link  -->
     <xacro:macro name="insert_inertia_l2_foot_ft_link">
       <origin
-        xyz="7.32716003928879E-06 0.00483832570565201 4.61026197218217E-08"
-        rpy="0 0 0" />
-      <mass
-        value="0.00863223621815312" />
-      <inertia
-        ixx="3.89940334430996E-07"
-        ixy="2.91176476412897E-10"
-        ixz="2.9783895900032E-10"
-        iyy="5.82213619517231E-07"
-        iyz="1.83208753538184E-12"
-        izz="3.4260620679022E-07" />
+        xyz="-4.46864767411626E-15 0.00477126123234917 2.4980018054066E-15"
+        rpy="0 0 0" />
+      <mass
+        value="0.00610112058812606" />
+      <inertia
+        ixx="3.17133668071686E-07"
+        ixy="4.81665130591134E-22"
+        ixz="-8.8406170379935E-23"
+        iyy="4.87731969834605E-07"
+        iyz="-8.74913874421171E-23"
+        izz="3.17133668071686E-07" />
     </xacro:macro>
     <!-- l3_foot_ft link 3 -->
     <xacro:macro name="insert_inertia_l3_foot_ft_link">
       <origin
-        xyz="7.32716003956635E-06 0.00483832570565224 4.61026188336433E-08"
-        rpy="0 0 0" />
-      <mass
-        value="0.00863223621815312" />
-      <inertia
-        ixx="3.89940334430996E-07"
-        ixy="2.9117647641293E-10"
-        ixz="2.97838959000262E-10"
-        iyy="5.82213619517231E-07"
-        iyz="1.83208753540344E-12"
-        izz="3.4260620679022E-07" />
+        xyz="-2.19269047363468E-15 0.00477126123234894 1.4432899320127E-15"
+        rpy="0 0 0" />
+      <mass
+        value="0.00610112058812606" />
+      <inertia
+        ixx="3.17133668071686E-07"
+        ixy="4.98475719906322E-22"
+        ixz="-6.41076334805219E-23"
+        iyy="4.87731969834605E-07"
+        iyz="-7.83706170725903E-23"
+        izz="3.17133668071686E-07" />
     </xacro:macro>
     <!-- l4_foot_ft link 4 -->
     <xacro:macro name="insert_inertia_l4_foot_ft_link">
       <origin
-        xyz="7.32716003670753E-06 0.00483832570565246 4.61026209985782E-08"
-        rpy="0 0 0" />
-      <mass
-        value="0.00863223621815312" />
-      <inertia
-        ixx="3.89940334430996E-07"
-        ixy="2.91176476412812E-10"
-        ixz="2.97838959000613E-10"
-        iyy="5.82213619517231E-07"
-        iyz="1.83208753537968E-12"
-        izz="3.42606206790219E-07" />
+        xyz="-8.32667268468867E-16 0.00477126123234917 6.66133814775094E-16"
+        rpy="0 0 0" />
+      <mass
+        value="0.00610112058812606" />
+      <inertia
+        ixx="3.17133668071686E-07"
+        ixy="3.66436341457745E-22"
+        ixz="5.6860083747849E-23"
+        iyy="4.87731969834605E-07"
+        iyz="-1.13521885241387E-22"
+        izz="3.17133668071686E-07" />
     </xacro:macro>
     <!-- Right leg -->
@@ -193,8 +193,8 @@
       <inertia
         ixx="0.0022729"
-        ixy="-5.6517E-10"
+        ixy="-5.6494E-10"
         ixz="6.6464E-06"
         iyy="0.0026746"
-        iyz="5.6889E-09"
+        iyz="5.69E-09"
         izz="0.0012354" />
     </xacro:macro>
@@ -202,5 +202,5 @@
     <xacro:macro name="insert_inertia_r_hip_roll_link">
       <origin
-        xyz="-0.07196 0.0061152 -0.00052563"
+        xyz="-0.071945 0.0061152 -0.00052563"
         rpy="0 0 0" />
       <mass
@@ -208,8 +208,8 @@
       <inertia
         ixx="0.00098222"
-        ixy="9.8947E-08"
-        ixz="9.2484E-09"
+        ixy="9.8944E-08"
+        ixz="9.2479E-09"
         iyy="0.00097045"
-        iyz="9.7414E-08"
+        iyz="9.7418E-08"
         izz="0.00092365" />
     </xacro:macro>
@@ -217,5 +217,5 @@
     <xacro:macro name="insert_inertia_r_hip_pitch_link">
       <origin
-        xyz="0.26753 4.9957E-05 -0.053132"
+        xyz="0.25103 -6.5307E-08 -0.05311"
         rpy="0 0 0" />
       <mass
@@ -223,8 +223,8 @@
       <inertia
         ixx="0.0034501"
-        ixy="-2.7593E-09"
+        ixy="1.1101E-07"
         ixz="-0.0019797"
         iyy="0.010035"
-        iyz="2.5351E-10"
+        iyz="-7.0796E-10"
         izz="0.01009" />
     </xacro:macro>
@@ -232,5 +232,5 @@
     <xacro:macro name="insert_inertia_r_knee_pitch_link">
       <origin
-        xyz="0.13396 0.00063335 -0.00486"
+        xyz="0.13396 0.0006585 -0.0028723"
         rpy="0 0 0" />
       <mass
@@ -254,5 +254,5 @@
         ixx="0.0025143"
         ixy="-0.00025651"
-        ixz="1.5321E-12"
+        ixz="1.5318E-12"
         iyy="0.0045125"
         iyz="9.9589E-10"
@@ -262,15 +262,15 @@
     <xacro:macro name="insert_inertia_r_ankle_roll_link">
       <origin
-        xyz="0.073422 7.2094E-05 0.063933"
-        rpy="0 0 0" />
-      <mass
-        value="1.8533" />
-      <inertia
-        ixx="0.0086813"
-        ixy="1.0356E-05"
-        ixz="0.00024346"
-        iyy="0.0084051"
-        iyz="-0.00012301"
-        izz="0.0013018" />
+        xyz="0.07353 -7.0757E-05 0.063933"
+        rpy="0 0 0" />
+      <mass
+        value="1.8633" />
+      <inertia
+        ixx="0.0086817"
+        ixy="9.8525E-06"
+        ixz="0.00024324"
+        iyy="0.0084053"
+        iyz="-0.00012345"
+        izz="0.0013019" />
     </xacro:macro>
     <!-- Right foot sensors -->
@@ -278,60 +278,60 @@
     <xacro:macro name="insert_inertia_r1_foot_ft_link">
       <origin
-        xyz="-8.7899E-06 0.0048383 -9.7784E-08"
-        rpy="0 0 0" />
-      <mass
-        value="0.0086322" />
-      <inertia
-        ixx="3.8994E-07"
-        ixy="-3.4931E-10"
-        ixz="5.2655E-10"
-        iyy="5.8221E-07"
-        iyz="-3.8859E-12"
-        izz="3.4261E-07" />
+        xyz="4.02455846426619E-16 0.00477126123234806 2.77555756156289E-16"
+        rpy="0 0 0" />
+      <mass
+        value="0.00610112058812607" />
+      <inertia
+        ixx="3.17133668071686E-07"
+        ixy="-4.44802942503628E-22"
+        ixz="-5.13396248201841E-23"
+        iyy="4.87731969834605E-07"
+        iyz="6.29534110948095E-22"
+        izz="3.17133668071686E-07" />
     </xacro:macro>
     <!-- r2_foot_ft link  -->
     <xacro:macro name="insert_inertia_r2_foot_ft_link">
       <origin
-        xyz="-8.78991381628169E-06 0.00483832326857458 -9.77840948768183E-08"
-        rpy="0 0 0" />
-      <mass
-        value="0.00863223621815318" />
-      <inertia
-        ixx="3.89936544476746E-07"
-        ixy="-3.49305164752985E-10"
-        ixz="5.26550951245735E-10"
-        iyy="5.82213425821568E-07"
-        iyz="-3.88587306925662E-12"
-        izz="3.42610190440137E-07" />
+        xyz="2.45636844198316E-15 0.00477126123234772 -5.55111512312578E-17"
+        rpy="0 0 0" />
+      <mass
+        value="0.00610112058812607" />
+      <inertia
+        ixx="3.17133668071686E-07"
+        ixy="-4.50854564995024E-22"
+        ixz="-3.37723169777971E-23"
+        iyy="4.87731969834605E-07"
+        iyz="6.62187087857084E-22"
+        izz="3.17133668071686E-07" />
     </xacro:macro>
     <!-- r_foot_ft link 3 -->
     <xacro:macro name="insert_inertia_r3_foot_ft_link">
       <origin
-        xyz="-8.78991381587924E-06 0.00483832326857436 -9.7784095154374E-08"
-        rpy="0 0 0" />
-      <mass
-        value="0.00863223621815318" />
-      <inertia
-        ixx="3.89936544476746E-07"
-        ixy="-3.49305164752997E-10"
-        ixz="5.26550951245753E-10"
-        iyy="5.82213425821568E-07"
-        iyz="-3.88587306930208E-12"
-        izz="3.42610190440137E-07" />
+        xyz="1.84574577843932E-15 0.00477126123234928 -1.11022302462516E-16"
+        rpy="0 0 0" />
+      <mass
+        value="0.00610112058812607" />
+      <inertia
+        ixx="3.17133668071686E-07"
+        ixy="-4.50482113604524E-22"
+        ixz="-5.92683031466877E-23"
+        iyy="4.87731969834605E-07"
+        iyz="6.6444452379759E-22"
+        izz="3.17133668071686E-07" />
     </xacro:macro>
     <!-- r_foot_ft link 4 -->
     <xacro:macro name="insert_inertia_r4_foot_ft_link">
       <origin
-        xyz="-8.78991381597638E-06 0.00483832326857403 -9.7784095154374E-08"
-        rpy="0 0 0" />
-      <mass
-        value="0.00863223621815318" />
-      <inertia
-        ixx="3.89936544476746E-07"
-        ixy="-3.49305164753006E-10"
-        ixz="5.26550951245779E-10"
-        iyy="5.82213425821568E-07"
-        iyz="-3.88587306929652E-12"
-        izz="3.42610190440137E-07" />
+        xyz="1.80411241501588E-15 0.00477126123234772 -1.66533453693773E-16"
+        rpy="0 0 0" />
+      <mass
+        value="0.00610112058812607" />
+      <inertia
+        ixx="3.17133668071686E-07"
+        ixy="-4.47159964907589E-22"
+        ixz="1.84653258585498E-23"
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
File: huron_description/urdf/huron_left_leg.xacro (robot description, xacro)
@@ -6,5 +6,7 @@
         <!-- left hip yaw joint -->
         <joint name="l_hip_yaw_joint" type="revolute">
-          <origin xyz="-0.0775 0 -0.14512" rpy="0 0 -0.0" />
+          <origin
+            xyz="-0.0775000000000011 0 -0.1451242"
+            rpy="0 0 0" />
           <parent link="${parent}" />
           <child link="l_hip_yaw_link" />
@@ -17,5 +19,5 @@
           <dynamics
             damping="0.5"
-            friction="5" />
+            friction="8" />
         </joint>
         <xacro:insert_transmission name="l_hip_yaw_joint"/>
@@ -52,5 +54,5 @@
           <dynamics
             damping="0.5"
-            friction="5" />
+            friction="8" />
         </joint>
         <xacro:insert_transmission name="l_hip_roll_joint"/>
@@ -72,5 +74,5 @@
           type="revolute">
           <origin
-            xyz="0 0 0"
+            xyz="1.6665E-05 -0.0165 -5E-05"
             rpy="${-pi/2} 0 ${-pi/2}" />
           <parent
@@ -87,5 +89,5 @@
           <dynamics
             damping="0.5"
-            friction="5" />
+            friction="8" />
         </joint>
         <xacro:insert_transmission name="l_hip_pitch_joint"/>
@@ -107,5 +109,5 @@
           type="revolute">
           <origin
-            xyz="0.512778478308813 5.00027201116859E-05 1.66647320003488E-05"
+            xyz="0.49628 0 0"
             rpy="0 0 0" />
           <parent
@@ -122,5 +124,5 @@
           <dynamics
             damping="0.5"
-            friction="5" />
+            friction="8" />
         </joint>
         <xacro:insert_transmission name="l_knee_pitch_joint"/>
@@ -142,5 +144,5 @@
           type="revolute">
           <origin
-            xyz="0.3715 3.1633E-05 0.0025"
+            xyz="0.37 0 0"
             rpy="0 0 0.0" />
           <parent
@@ -157,5 +159,5 @@
           <dynamics
             damping="0.5"
-            friction="2.0" />
+            friction="4" />
         </joint>
         <xacro:insert_transmission name="l_ankle_pitch_joint"/>
@@ -192,5 +194,5 @@
           <dynamics
             damping="0.5"
-            friction="2.0" />
+            friction="4" />
         </joint>
         <xacro:insert_transmission name="l_ankle_roll_joint"/>
@@ -210,5 +212,5 @@
         <joint name="l1_ft_fixed" type="revolute">
             <origin
-              xyz="0.0983282135717449 0.0206816111121677 0.127875866180865"
+              xyz="0.098297 0.02083 0.12788"
               rpy="0 0 ${pi/2}" />
             <axis xyz="0 0 1"/>
@@ -236,5 +238,5 @@
         <joint name="l2_ft_fixed" type="revolute">
             <origin
-              xyz="0.0982752085863122 -0.0143183487516882 0.127875866180865"
+              xyz="0.098297 -0.01417 0.12788"
               rpy="0 0 ${pi/2}" />
             <axis xyz="0 0 1"/>
@@ -262,5 +264,5 @@
         <joint name="l3_ft_fixed" type="revolute">
             <origin
-              xyz="0.0982716792139032 -0.0166488444898757 0"
+              xyz="0.098297 -0.0165 0"
               rpy="0 0 ${pi/2}" />
             <axis xyz="0 0 1"/>
@@ -288,5 +290,5 @@
         <joint name="l4_ft_fixed" type="revolute">
             <origin
-              xyz="0.0983224252792114 0.0168595176863209 0"
+              xyz="0.098297 0.017008 0"
               rpy="0 0 ${pi/2}" />
             <axis xyz="0 0 1"/>

File: huron_description/urdf/huron_right_leg.xacro (robot description, xacro)
@@ -9,5 +9,5 @@
           type="revolute">
           <origin
-            xyz="0.0774999999999944 0 -0.1451242"
+            xyz="0.0775 0 -0.14512"
             rpy="0 0 ${pi}" />
           <parent
@@ -24,5 +24,5 @@
           <dynamics
             damping="0.5"
-            friction="5" />
+            friction="8" />
         </joint>
         <xacro:insert_transmission name="r_hip_yaw_joint"/>
@@ -59,5 +59,5 @@
           <dynamics
             damping="0.5"
-            friction="5" />
+            friction="8" />
         </joint>
         <xacro:insert_transmission name="r_hip_roll_joint"/>
@@ -79,5 +79,5 @@
           type="revolute">
           <origin
-            xyz="0 0 0"
+            xyz="-1.6665E-05 -0.0165 -5E-05"
             rpy="${-pi/2} 0 ${-pi/2}" />
           <parent
@@ -94,5 +94,5 @@
           <dynamics
             damping="0.5"
-            friction="5" />
+            friction="8" />
         </joint>
         <xacro:insert_transmission name="r_hip_pitch_joint"/>
@@ -114,5 +114,5 @@
           type="revolute">
           <origin
-            xyz="0.512778478308813 4.99999999867273E-05 -1.66647320091612E-05"
+            xyz="0.49628 0 0"
             rpy="0 0 0" />
           <parent
@@ -129,5 +129,5 @@
           <dynamics
             damping="0.5"
-            friction="5" />
+            friction="8" />
         </joint>
         <xacro:insert_transmission name="r_knee_pitch_joint"/>
@@ -149,5 +149,5 @@
           type="revolute">
           <origin
-            xyz="0.370000000000006 -3.16358749707368E-05 -0.00249999999999943"
+            xyz="0.37 0 0"
             rpy="0 0 0.0" />
           <parent
@@ -164,5 +164,5 @@
           <dynamics
             damping="0.5"
-            friction="2.0" />
+            friction="4" />
         </joint>
         <xacro:insert_transmission name="r_ankle_pitch_joint"/>
@@ -199,5 +199,5 @@
           <dynamics
             damping="0.5"
-            friction="2.0" />
+            friction="4" />
         </joint>
         <xacro:insert_transmission name="r_ankle_roll_joint"/>
@@ -217,5 +217,5 @@
         <joint name="r1_ft_fixed" type="revolute">
             <origin
-              xyz="0.0982708740959065 0.0143480673989493 0.127875866180863"
+              xyz="0.098297 0.01417 0.12788"
               rpy="0 0 ${pi/2}" />
             <axis xyz="0 0 1"/>
@@ -243,5 +243,5 @@
         <joint name="r2_ft_fixed" type="revolute">
             <origin
-              xyz="0.0983344633797905 -0.0206518748353312 0.127875866180863"
+              xyz="0.098297 -0.02083 0.12788"
               rpy="0 0 ${pi/2}" />
             <axis xyz="0 0 1"/>
@@ -269,5 +269,5 @@
         <joint name="r3_ft_fixed" type="revolute">
             <origin
-              xyz="0.0983275192522874 -0.0168297833346846 0"
+              xyz="0.098297 -0.017008 0"
               rpy="0 0 ${pi/2}" />
             <axis xyz="0 0 1"/>
@@ -295,5 +295,5 @@
         <joint name="r4_ft_fixed" type="revolute">
             <origin
-              xyz="0.0982666399609057 0.0166785619632585 0"
+              xyz="0.098297 0.0165 0"
               rpy="0 0 ${pi/2}" />
             <axis xyz="0 0 1"/>

File: huron_description/urdf/huron_visuals.xacro (robot description, xacro)
@@ -74,5 +74,5 @@
         <origin xyz="0 0 0" rpy=" 0 0 0" />
         <geometry>
-            <mesh filename="package://huron_description/meshes/r_foot_ft.STL" scale="1 1 1" />
+            <mesh filename="package://huron_description/meshes/l1_foot_ft_link.STL" scale="1 1 1" />
         </geometry>
         <material name="green"/>
@@ -82,5 +82,5 @@
         <origin xyz="0 0 0" rpy=" 0 0 0" />
         <geometry>
-            <mesh filename="package://huron_description/meshes/r_foot_ft.STL" scale="1 1 1" />
+            <mesh filename="package://huron_description/meshes/l2_foot_ft_link.STL" scale="1 1 1" />
         </geometry>
         <material name="green"/>
@@ -90,5 +90,5 @@
         <origin xyz="0 0 0" rpy=" 0 0 0" />
         <geometry>
-            <mesh filename="package://huron_description/meshes/r_foot_ft.STL" scale="1 1 1" />
+            <mesh filename="package://huron_description/meshes/l3_foot_ft_link.STL" scale="1 1 1" />
         </geometry>
         <material name="green"/>
@@ -98,5 +98,5 @@
         <origin xyz="0 0 0" rpy=" 0 0 0" />
         <geometry>
-            <mesh filename="package://huron_description/meshes/r_foot_ft.STL" scale="1 1 1" />
+            <mesh filename="package://huron_description/meshes/l4_foot_ft_link.STL" scale="1 1 1" />
         </geometry>
         <material name="green"/>
@@ -159,7 +159,7 @@
         <origin xyz="0 0 0" rpy=" 0 0 0" />
         <geometry>
-            <mesh filename="package://huron_description/meshes/r_foot_ft.STL" scale="1 1 1" />
+            <mesh filename="package://huron_description/meshes/r1_foot_ft_link.STL" scale="1 1 1" />
         </geometry>
-        <material name="grey"/>
+        <material name="green"/>
     </xacro:macro>
     <!-- r2_foot_ft link  -->
@@ -167,7 +167,7 @@
         <origin xyz="0 0 0" rpy=" 0 0 0" />
         <geometry>
-            <mesh filename="package://huron_description/meshes/r_foot_ft.STL" scale="1 1 1" />
+            <mesh filename="package://huron_description/meshes/r2_foot_ft_link.STL" scale="1 1 1" />
         </geometry>
-        <material name="grey"/>
+        <material name="green"/>
     </xacro:macro>
     <!-- r3_foot_ft link 3-->
@@ -175,7 +175,7 @@
         <origin xyz="0 0 0" rpy=" 0 0 0" />
         <geometry>
-            <mesh filename="package://huron_description/meshes/r_foot_ft.STL" scale="1 1 1" />
+            <mesh filename="package://huron_description/meshes/r3_foot_ft_link.STL" scale="1 1 1" />
         </geometry>
-        <material name="grey"/>
+        <material name="green"/>
     </xacro:macro>
     <!-- r4_foot_ft link 4 -->
@@ -183,7 +183,7 @@
         <origin xyz="0 0 0" rpy=" 0 0 0" />
         <geometry>
-            <mesh filename="package://huron_description/meshes/r_foot_ft.STL" scale="1 1 1" />
+            <mesh filename="package://huron_description/meshes/r4_foot_ft_link.STL" scale="1 1 1" />
         </geometry>
-        <material name="grey"/>
+        <material name="green"/>
     </xacro:macro>
     <!-- Foot base -->
