Commit message: WIP

File: huron_description/urdf/huron.urdf (robot description, URDF)
Before this commit: robot huron, 26 links, 25 joints
Links:
- removed link l1_foot_ft_link
- removed link l2_foot_ft_link
- removed link l3_foot_ft_link
- removed link l4_foot_ft_link
- removed link l_foot_v_ft_link
- removed link r1_foot_ft_link
- removed link r2_foot_ft_link
- removed link r3_foot_ft_link
- removed link r4_foot_ft_link
- removed link r_foot_v_ft_link
Joints:
- removed joint l1_ft_fixed
- removed joint l2_ft_fixed
- removed joint l3_ft_fixed
- removed joint l4_ft_fixed
- removed joint lv_ft_fixed
- removed joint r1_ft_fixed
- removed joint r2_ft_fixed
- removed joint r3_ft_fixed
- removed joint r4_ft_fixed
- removed joint rv_ft_fixed

File: huron_description/urdf/huron_gazebo.xacro (robot description, xacro)
@@ -41,5 +41,5 @@
     <gazebo>
     <plugin name="r1_ft_sensor" filename="libgazebo_ros_ft_sensor.so">
-        <updateRate>50.0</updateRate>
+        <updateRate>100.0</updateRate>
         <topicName>/huron/sensor/r1_ft_sensor</topicName>
         <jointName>r_ankle_roll_joint</jointName>
@@ -52,5 +52,5 @@
     <gazebo>
     <plugin name="l1_ft_sensor" filename="libgazebo_ros_ft_sensor.so">
-        <updateRate>50.0</updateRate>
+        <updateRate>100.0</updateRate>
         <topicName>/huron/sensor/l1_ft_sensor</topicName>
         <jointName>l_ankle_roll_joint</jointName>
