Commit message: Added foot sensors to the model, tested output

File: huron_description/urdf/huron.xacro (robot description, xacro)
@@ -38,5 +38,5 @@
     <!-- imu joint -->
     <joint name="imu_fixed" type="fixed">
-        <origin xyz="0.0 0 0.45" rpy="0 0 0"/>
+        <origin xyz="0 0 0" rpy="0 0 0"/>
         <parent link="base_footprint"/>
         <child link="imu_link"/>

File: huron_description/urdf/huron_gazebo.xacro (robot description, xacro)
@@ -36,12 +36,11 @@
         </sensor>
     </gazebo>
-    <?comment
     <gazebo reference ="r1_ft_fixed">
-    	<provideFeedback> true</provideFeedback>
+    	<provideFeedback>true</provideFeedback>
     </gazebo>
     <gazebo>
     <plugin name="r1_ft_sensor" filename="libgazebo_ros_ft_sensor.so">
         <updateRate>100.0</updateRate>
-        <topicName>/robotis/sensor/r1_ft_sensor</topicName>
+        <topicName>/huron/sensor/r1_ft_sensor</topicName>
         <jointName>r1_ft_fixed</jointName>
         <gaussianNoise>0.0</gaussianNoise>
@@ -49,10 +48,10 @@
     </gazebo>
     <gazebo reference ="r2_ft_fixed">
-    	<provideFeedback> true</provideFeedback>
+    	<provideFeedback>true</provideFeedback>
     </gazebo>
     <gazebo>
     <plugin name="r2_ft_sensor" filename="libgazebo_ros_ft_sensor.so">
         <updateRate>100.0</updateRate>
-        <topicName>/robotis/sensor/r2_ft_sensor</topicName>
+        <topicName>/huron/sensor/r2_ft_sensor</topicName>
         <jointName>r2_ft_fixed</jointName>
         <gaussianNoise>0.0</gaussianNoise>
@@ -60,10 +59,10 @@
     </gazebo>
     <gazebo reference ="r3_ft_fixed">
-    	<provideFeedback> true</provideFeedback>
+    	<provideFeedback>true</provideFeedback>
     </gazebo>
     <gazebo>
     <plugin name="r3_ft_sensor" filename="libgazebo_ros_ft_sensor.so">
         <updateRate>100.0</updateRate>
-        <topicName>/robotis/sensor/r3_ft_sensor</topicName>
+        <topicName>/huron/sensor/r3_ft_sensor</topicName>
         <jointName>r3_ft_fixed</jointName>
         <gaussianNoise>0.0</gaussianNoise>
@@ -71,10 +70,10 @@
     </gazebo>
     <gazebo reference ="r4_ft_fixed">
-    	<provideFeedback> true</provideFeedback>
+    	<provideFeedback>true</provideFeedback>
     </gazebo>
     <gazebo>
     <plugin name="r4_ft_sensor" filename="libgazebo_ros_ft_sensor.so">
         <updateRate>100.0</updateRate>
-        <topicName>/robotis/sensor/r4_ft_sensor</topicName>
+        <topicName>/huron/sensor/r4_ft_sensor</topicName>
         <jointName>r4_ft_fixed</jointName>
         <gaussianNoise>0.0</gaussianNoise>
@@ -82,10 +81,10 @@
     </gazebo>
     <gazebo reference ="l1_ft_fixed">
-    	<provideFeedback> true</provideFeedback>
+    	<provideFeedback>true</provideFeedback>
     </gazebo>
     <gazebo>
     <plugin name="l1_ft_sensor" filename="libgazebo_ros_ft_sensor.so">
         <updateRate>100.0</updateRate>
-        <topicName>/robotis/sensor/l1_ft_sensor</topicName>
+        <topicName>/huron/sensor/l1_ft_sensor</topicName>
         <jointName>l1_ft_fixed</jointName>
         <gaussianNoise>0.0</gaussianNoise>
@@ -93,10 +92,10 @@
     </gazebo>
     <gazebo reference ="l2_ft_fixed">
-    	<provideFeedback> true</provideFeedback>
+    	<provideFeedback>true</provideFeedback>
     </gazebo>
     <gazebo>
     <plugin name="l2_ft_sensor" filename="libgazebo_ros_ft_sensor.so">
         <updateRate>100.0</updateRate>
-        <topicName>/robotis/sensor/l2_ft_sensor</topicName>
+        <topicName>/huron/sensor/l2_ft_sensor</topicName>
         <jointName>l2_ft_fixed</jointName>
         <gaussianNoise>0.0</gaussianNoise>
@@ -104,10 +103,10 @@
     </gazebo>
     <gazebo reference ="l3_ft_fixed">
-    	<provideFeedback> true</provideFeedback>
+    	<provideFeedback>true</provideFeedback>
     </gazebo>
     <gazebo>
     <plugin name="l3_ft_sensor" filename="libgazebo_ros_ft_sensor.so">
         <updateRate>100.0</updateRate>
-        <topicName>/robotis/sensor/l3_ft_sensor</topicName>
+        <topicName>/huron/sensor/l3_ft_sensor</topicName>
         <jointName>l3_ft_fixed</jointName>
         <gaussianNoise>0.0</gaussianNoise>
@@ -115,15 +114,14 @@
     </gazebo>
     <gazebo reference ="l4_ft_fixed">
-    	<provideFeedback> true</provideFeedback>
+    	<provideFeedback>true</provideFeedback>
     </gazebo>
     <gazebo>
     <plugin name="r4_ft_sensor" filename="libgazebo_ros_ft_sensor.so">
         <updateRate>100.0</updateRate>
-        <topicName>/robotis/sensor/l4_ft_sensor</topicName>
+        <topicName>/huron/sensor/l4_ft_sensor</topicName>
         <jointName>l4_ft_fixed</jointName>
         <gaussianNoise>0.0</gaussianNoise>
     </plugin>
     </gazebo>
-      ?>
     <!-- World -->
     <gazebo reference="world"></gazebo>
@@ -183,5 +181,4 @@
         <material>Gazebo/Blue</material>
     </gazebo>
-    <?comment
     <gazebo reference="l1_foot_ft_link">
         <kp>100000.0</kp>
@@ -193,5 +190,5 @@
          <maxVel>1.0</maxVel>
         <minDepth>0.0001</minDepth>
-        <material>Gazebo/white</material>
+        <material>Gazebo/Black</material>
     </gazebo>
     <gazebo reference="l2_foot_ft_link">
@@ -204,5 +201,5 @@
          <maxVel>1.0</maxVel>
         <minDepth>0.0001</minDepth>
-        <material>Gazebo/white</material>
+        <material>Gazebo/Black</material>
     </gazebo>
     <gazebo reference="l3_foot_ft_link">
@@ -215,5 +212,5 @@
          <maxVel>1.0</maxVel>
         <minDepth>0.0001</minDepth>
-        <material>Gazebo/white</material>
+        <material>Gazebo/Black</material>
     </gazebo>
     <gazebo reference="l4_foot_ft_link">
@@ -226,7 +223,6 @@
          <maxVel>1.0</maxVel>
         <minDepth>0.0001</minDepth>
-        <material>Gazebo/white</material>
-    </gazebo>
-    ?>
+        <material>Gazebo/Black</material>
+    </gazebo>
     <!-- Right Leg -->
     <gazebo reference="r_hip_yaw_link">
@@ -271,5 +267,4 @@
         <material>Gazebo/Blue</material>
     </gazebo>
-    <?comment
     <gazebo reference="r1_foot_ft_link">
         <kp>100000.0</kp>
@@ -281,5 +276,5 @@
          <maxVel>1.0</maxVel>
         <minDepth>0.0001</minDepth>
-        <material>Gazebo/white</material>
+        <material>Gazebo/Black</material>
     </gazebo>
     <gazebo reference="r2_foot_ft_link">
@@ -292,5 +287,5 @@
          <maxVel>1.0</maxVel>
         <minDepth>0.0001</minDepth>
-        <material>Gazebo/white</material>
+        <material>Gazebo/Black</material>
     </gazebo>
     <gazebo reference="r3_foot_ft_link">
@@ -303,5 +298,5 @@
          <maxVel>1.0</maxVel>
         <minDepth>0.0001</minDepth>
-        <material>Gazebo/white</material>
+        <material>Gazebo/Black</material>
     </gazebo>
     <gazebo reference="r4_foot_ft_link">
@@ -314,6 +309,5 @@
          <maxVel>1.0</maxVel>
         <minDepth>0.0001</minDepth>
-        <material>Gazebo/white</material>
-    </gazebo>
-    ?>
+        <material>Gazebo/Black</material>
+    </gazebo>
 </robot>

File: huron_description/urdf/huron_inertia.xacro (robot description, xacro)
@@ -110,21 +110,61 @@
     <!-- l1_foot_ft link -->
     <xacro:macro name="insert_inertia_l1_foot_ft_link">
-        <mass value="0.03875"/>
-        <inertia ixx="0.00052206" ixy="0" ixz="0.00001" iyy="0.00047025" iyz="0" izz="0.00009087" />
+      <origin
+        xyz="6.5681E-06 0.0048368 0.00012069"
+        rpy="0 0 0" />
+      <mass
+        value="0.0086322" />
+      <inertia
+        ixx="3.8994E-07"
+        ixy="2.5351E-10"
+        ixz="3.0416E-10"
+        iyy="5.8206E-07"
+        iyz="5.9744E-09"
+        izz="3.4276E-07" />
     </xacro:macro>
     <!-- l2_foot_ft link  -->
     <xacro:macro name="insert_inertia_l2_foot_ft_link">
-        <mass value="0.03875"/>
-        <inertia ixx="0.00052206" ixy="0" ixz="0.00001" iyy="0.00047025" iyz="0" izz="0.00009087" />
+      <origin
+        xyz="6.56809560273253E-06 0.00483682139671537 0.000120685375128327"
+        rpy="0 0 0" />
+      <mass
+        value="0.00863223621815319" />
+      <inertia
+        ixx="3.89940248965647E-07"
+        ixy="2.53506346419819E-10"
+        ixz="3.04161588773098E-10"
+        iyy="5.82064646347941E-07"
+        iyz="5.97441467814794E-09"
+        izz="3.42755265424868E-07" />
     </xacro:macro>
     <!-- l3_foot_ft link 3 -->
     <xacro:macro name="insert_inertia_l3_foot_ft_link">
-        <mass value="0.03875"/>
-        <inertia ixx="0.00052206" ixy="0" ixz="0.00001" iyy="0.00047025" iyz="0" izz="0.00009087" />
+      <origin
+        xyz="6.56809560273253E-06 0.00483682139671548 0.000120685375128382"
+        rpy="0 0 0" />
+      <mass
+        value="0.00863223621815319" />
+      <inertia
+        ixx="3.89940248965648E-07"
+        ixy="2.53506346419837E-10"
+        ixz="3.04161588773088E-10"
+        iyy="5.82064646347941E-07"
+        iyz="5.97441467814795E-09"
+        izz="3.42755265424868E-07" />
     </xacro:macro>
     <!-- l4_foot_ft link 4 -->
     <xacro:macro name="insert_inertia_l4_foot_ft_link">
-        <mass value="0.03875"/>
-        <inertia ixx="0.00052206" ixy="0" ixz="0.00001" iyy="0.00047025" iyz="0" izz="0.00009087" />
+      <origin
+        xyz="6.5681E-06 0.0048368 0.00012069"
+        rpy="0 0 0" />
+      <mass
+        value="0.0086322" />
+      <inertia
+        ixx="3.8994E-07"
+        ixy="2.5351E-10"
+        ixz="3.0416E-10"
+        iyy="5.8206E-07"
+        iyz="5.9744E-09"
+        izz="3.4276E-07" />
     </xacro:macro>
     <!-- Right leg -->
@@ -222,21 +262,61 @@
     <!-- r1_foot_ft link -->
     <xacro:macro name="insert_inertia_r1_foot_ft_link">
-        <mass value="0.03875"/>
-        <inertia ixx="0.00052206" ixy="0" ixz="0.00001" iyy="0.00047025" iyz="0" izz="0.00009087" />
+      <origin
+        xyz="-9.3029E-06 0.0048381 4.6013E-05"
+        rpy="0 0 0" />
+      <mass
+        value="0.0086322" />
+      <inertia
+        ixx="3.8994E-07"
+        ixy="-3.7469E-10"
+        ixz="5.2298E-10"
+        iyy="5.8219E-07"
+        iyz="2.2796E-09"
+        izz="3.4263E-07" />
     </xacro:macro>
     <!-- r2_foot_ft link  -->
     <xacro:macro name="insert_inertia_r2_foot_ft_link">
-        <mass value="0.03875"/>
-        <inertia ixx="0.00052206" ixy="0" ixz="0.00001" iyy="0.00047025" iyz="0" izz="0.00009087" />
+      <origin
+        xyz="-9.3029E-06 0.0048381 4.6013E-05"
+        rpy="0 0 0" />
+      <mass
+        value="0.0086322" />
+      <inertia
+        ixx="3.8994E-07"
+        ixy="-3.7469E-10"
+        ixz="5.2298E-10"
+        iyy="5.8219E-07"
+        iyz="2.2796E-09"
+        izz="3.4263E-07" />
     </xacro:macro>
     <!-- r_foot_ft link 3 -->
     <xacro:macro name="insert_inertia_r3_foot_ft_link">
-        <mass value="0.03875"/>
-        <inertia ixx="0.00052206" ixy="0" ixz="0.00001" iyy="0.00047025" iyz="0" izz="0.00009087" />
+      <origin
+        xyz="-9.3029E-06 0.0048381 4.6013E-05"
+        rpy="0 0 0" />
+      <mass
+        value="0.0086322" />
+      <inertia
+        ixx="3.8994E-07"
+        ixy="-3.7469E-10"
+        ixz="5.2298E-10"
+        iyy="5.8219E-07"
+        iyz="2.2796E-09"
+        izz="3.4263E-07" />
     </xacro:macro>
     <!-- r_foot_ft link 4 -->
     <xacro:macro name="insert_inertia_r4_foot_ft_link">
-        <mass value="0.03875"/>
-        <inertia ixx="0.00052206" ixy="0" ixz="0.00001" iyy="0.00047025" iyz="0" izz="0.00009087" />
+      <origin
+        xyz="-9.3029E-06 0.0048381 4.6013E-05"
+        rpy="0 0 0" />
+      <mass
+        value="0.0086322" />
+      <inertia
+        ixx="3.8994E-07"
+        ixy="-3.7469E-10"
+        ixz="5.2298E-10"
+        iyy="5.8219E-07"
+        iyz="2.2796E-09"
+        izz="3.4263E-07" />
     </xacro:macro>
 </robot>

File: huron_description/urdf/huron_left_leg.xacro (robot description, xacro)
@@ -207,8 +207,9 @@
             </inertial>
         </link>
-        <?comment
         <!-- left ft fixed joint 1 -->
         <joint name="l1_ft_fixed" type="revolute">
-            <origin xyz="0.045 0.006 0.09" rpy="0 0  1.57"/>
+            <origin
+              xyz="0.098328 0.020682 0.12788"
+              rpy="-0.024938 0.00629 1.5706" />
             <axis xyz="0 0 1"/>
             <parent link="l_ankle_roll_link"/>
@@ -234,5 +235,7 @@
         <!-- left ft fixed joint 2 -->
         <joint name="l2_ft_fixed" type="revolute">
-            <origin xyz="0.045  -0.006  0.09" rpy="0 0  1.57"/>
+            <origin
+              xyz="0.098275 -0.014318 0.12788"
+              rpy="-0.024938 0.00629 1.5706" />
             <axis xyz="0 0 1"/>
             <parent link="l_ankle_roll_link"/>
@@ -258,5 +261,7 @@
         <!-- left ft fixed joint 3 -->
         <joint name="l3_ft_fixed" type="revolute">
-            <origin xyz="0.045  -0.008  -0.09" rpy="0 0  1.57"/>
+            <origin
+              xyz="0.098272 -0.016649 0"
+              rpy="-0.024938 0.00629 1.5706" />
             <axis xyz="0 0 1"/>
             <parent link="l_ankle_roll_link"/>
@@ -282,5 +287,7 @@
         <!-- left ft fixed joint 4 -->
         <joint name="l4_ft_fixed" type="revolute">
-            <origin xyz="0.045  0.008  -0.09" rpy="0 0  1.57"/>
+            <origin
+              xyz="0.098322 0.01686 0"
+              rpy="-0.024938 0.00629 1.5706" />
             <axis xyz="0 0 1"/>
             <parent link="l_ankle_roll_link"/>
@@ -312,5 +319,4 @@
         <!-- left foot ft link -->
         <link name="l_foot_v_ft_link"></link>
-      ?>
     </xacro:macro>
 </robot>

File: huron_description/urdf/huron_right_leg.xacro (robot description, xacro)
@@ -215,8 +215,9 @@
         </link>
         <!-- Right foot sensors -->
-        <?comment
         <!-- right ft fixed joint 1 -->
         <joint name="r1_ft_fixed" type="revolute">
-            <origin xyz="0.045 0.006 0.09" rpy="0 0  1.57"/>
+            <origin
+              xyz="0.098271 0.014348 0.12788"
+              rpy="-0.0095317 0.011124 1.5707" />
             <axis xyz="0 0 1"/>
             <parent link="r_ankle_roll_link"/>
@@ -242,5 +243,7 @@
         <!-- right ft fixed joint 2 -->
         <joint name="r2_ft_fixed" type="revolute">
-            <origin xyz="0.045  -0.006  0.09" rpy="0 0  1.57"/>
+            <origin
+              xyz="0.098334 -0.020652 0.12788"
+              rpy="-0.0095317 0.011124 1.5707" />
             <axis xyz="0 0 1"/>
             <parent link="r_ankle_roll_link"/>
@@ -266,5 +269,7 @@
         <!-- right ft fixed joint 3 -->
         <joint name="r3_ft_fixed" type="revolute">
-            <origin xyz="0.045  -0.008  -0.09" rpy="0 0  1.57"/>
+            <origin
+              xyz="0.098328 -0.01683 0"
+              rpy="-0.0095317 0.011124 1.5707" />
             <axis xyz="0 0 1"/>
             <parent link="r_ankle_roll_link"/>
@@ -290,5 +295,7 @@
         <!-- right ft fixed joint 4 -->
         <joint name="r4_ft_fixed" type="revolute">
-            <origin xyz="0.045  0.008  -0.09" rpy="0 0  1.57"/>
+            <origin
+              xyz="0.098267 0.016679 0"
+              rpy="-0.0095317 0.011124 1.5707" />
             <axis xyz="0 0 1"/>
             <parent link="r_ankle_roll_link"/>
@@ -312,5 +319,5 @@
 	    </inertial>
         </link>
-                <!-- right ft fixed joint -->
+        <!-- right ft fixed joint -->
         <joint name="rv_ft_fixed" type="fixed">
             <origin xyz="0.0 0.0 0.0" rpy="0 0 0"/>
@@ -326,5 +333,4 @@
         <!-- right foot ft link -->
         <link name="r_foot_v_ft_link"></link>
-      ?>
     </xacro:macro>
 </robot>

File: huron_description/urdf/huron_visuals.xacro (robot description, xacro)
@@ -62,10 +62,9 @@
         </material>
     </xacro:macro>
-    <?comment
     <!-- l1_foot_ft link -->
     <xacro:macro name="insert_mesh_l1_foot_ft_link">
         <origin xyz="0 0 0" rpy=" 0 0 0" />
         <geometry>
-            <mesh filename="package://huron_description/meshes/r_foot_ft.STL" scale="0.05 0.05 0.05" />
+            <mesh filename="package://huron_description/meshes/r_foot_ft.STL" scale="1 1 1" />
         </geometry>
         <material name="grey"/>
@@ -75,5 +74,5 @@
         <origin xyz="0 0 0" rpy=" 0 0 0" />
         <geometry>
-            <mesh filename="package://huron_description/meshes/r_foot_ft.STL" scale="0.05 0.05 0.05" />
+            <mesh filename="package://huron_description/meshes/r_foot_ft.STL" scale="1 1 1" />
         </geometry>
         <material name="grey"/>
@@ -83,5 +82,5 @@
         <origin xyz="0 0 0" rpy=" 0 0 0" />
         <geometry>
-            <mesh filename="package://huron_description/meshes/r_foot_ft.STL" scale="0.05 0.05 0.05" />
+            <mesh filename="package://huron_description/meshes/r_foot_ft.STL" scale="1 1 1" />
         </geometry>
         <material name="grey"/>
@@ -91,9 +90,8 @@
         <origin xyz="0 0 0" rpy=" 0 0 0" />
         <geometry>
-            <mesh filename="package://huron_description/meshes/r_foot_ft.STL" scale="0.05 0.05 0.05" />
+            <mesh filename="package://huron_description/meshes/r_foot_ft.STL" scale="1 1 1" />
         </geometry>
         <material name="grey"/>
     </xacro:macro>
-        ?>
     <!-- right hip yaw link -->
     <xacro:macro name="insert_mesh_r_hip_yaw_link">
@@ -149,10 +147,9 @@
     </xacro:macro>
     <!-- Right foot sensors -->
-    <?comment
     <!-- r1_foot_ft link -->
     <xacro:macro name="insert_mesh_r1_foot_ft_link">
         <origin xyz="0 0 0" rpy=" 0 0 0" />
         <geometry>
-            <mesh filename="package://huron_description/meshes/r_foot_ft.STL" scale="0.05 0.05 0.05" />
+            <mesh filename="package://huron_description/meshes/r_foot_ft.STL" scale="1 1 1" />
         </geometry>
         <material name="grey"/>
@@ -162,5 +159,5 @@
         <origin xyz="0 0 0" rpy=" 0 0 0" />
         <geometry>
-            <mesh filename="package://huron_description/meshes/r_foot_ft.STL" scale="0.05 0.05 0.05" />
+            <mesh filename="package://huron_description/meshes/r_foot_ft.STL" scale="1 1 1" />
         </geometry>
         <material name="grey"/>
@@ -170,5 +167,5 @@
         <origin xyz="0 0 0" rpy=" 0 0 0" />
         <geometry>
-            <mesh filename="package://huron_description/meshes/r_foot_ft.STL" scale="0.05 0.05 0.05" />
+            <mesh filename="package://huron_description/meshes/r_foot_ft.STL" scale="1 1 1" />
         </geometry>
         <material name="grey"/>
@@ -178,8 +175,7 @@
         <origin xyz="0 0 0" rpy=" 0 0 0" />
         <geometry>
-            <mesh filename="package://huron_description/meshes/r_foot_ft.STL" scale="0.05 0.05 0.05" />
+            <mesh filename="package://huron_description/meshes/r_foot_ft.STL" scale="1 1 1" />
         </geometry>
         <material name="grey"/>
     </xacro:macro>
-        ?>
 </robot>
