Commit message: Added floating joint link for pinocchio, and re-added force sensor frames for contacts (no collisions)

File: huron_description/urdf/huron_cheat.urdf (robot description, URDF)
Before this commit: robot huron, 27 links, 26 joints
Links:
- removed link base_link
- added link base
- added link world
Joints:
- added joint world_fixed: type floating, parent world, child base, origin xyz=0 0 0 rpy=0 0 0
- joint base_fixed: parent base_link -> base

File: huron_description/urdf/huron_left_leg.xacro (robot description, xacro)
@@ -5,5 +5,5 @@
     <xacro:macro name="huron_left_leg" params="parent dxl_effort dxl_speed">
         <!-- left hip yaw joint -->
-        <joint name="l_hip_yaw_joint" type="fixed">
+        <joint name="l_hip_yaw_joint" type="revolute">
           <origin
             xyz="-0.0775 0 -0.1451242"
@@ -37,5 +37,5 @@
         <joint
           name="l_hip_roll_joint"
-          type="fixed">
+          type="revolute">
           <origin
             xyz="0 0 0"
@@ -209,4 +209,116 @@
             </inertial>
         </link>
+        <!-- left ft fixed joint 1 -->
+        <joint name="l1_ft_fixed" type="fixed">
+            <origin
+              xyz="0.0983282135717449 0.0206816111121677 0.127875866180865"
+              rpy="0 0 ${pi/2}" />
+            <axis xyz="0 0 1"/>
+            <parent link="l_ankle_roll_link"/>
+            <child link="l1_foot_ft_link"/>
+            <limit
+            lower="0"
+            upper="0"
+            effort="100"
+            velocity="100" />
+        </joint>
+        <!-- left foot ft link 1 -->
+        <link name="l1_foot_ft_link">
+	    <visual>
+		<xacro:insert_mesh_l1_foot_ft_link />
+	    </visual>
+            <!-- <collision>
+                <xacro:insert_mesh_l1_foot_ft_link />
+            </collision>
+	    <inertial>
+		<xacro:insert_inertia_l1_foot_ft_link />
+	    </inertial> -->
+        </link>
+        <!-- left ft fixed joint 2 -->
+        <joint name="l2_ft_fixed" type="fixed">
+            <origin
+              xyz="0.0982752085863122 -0.0143183487516882 0.127875866180865"
+              rpy="0 0 ${pi/2}" />
+            <axis xyz="0 0 1"/>
+            <parent link="l_ankle_roll_link"/>
+            <child link="l2_foot_ft_link"/>
+            <limit
+            lower="0"
+            upper="0"
+            effort="100"
+            velocity="100" />
+        </joint>
+        <!-- left foot ft link 2 -->
+        <link name="l2_foot_ft_link">
+	    <visual>
+		<xacro:insert_mesh_l2_foot_ft_link />
+	    </visual>
+            <!-- <collision>
+                <xacro:insert_mesh_l2_foot_ft_link />
+            </collision>
+	    <inertial>
+		<xacro:insert_inertia_l2_foot_ft_link />
+	    </inertial> -->
+        </link>
+        <!-- left ft fixed joint 3 -->
+        <joint name="l3_ft_fixed" type="fixed">
+            <origin
+              xyz="0.0982716792139032 -0.0166488444898757 0"
+              rpy="0 0 ${pi/2}" />
+            <axis xyz="0 0 1"/>
+            <parent link="l_ankle_roll_link"/>
+            <child link="l3_foot_ft_link"/>
+            <limit
+            lower="0"
+            upper="0"
+            effort="100"
+            velocity="100" />
+        </joint>
+        <!-- left foot ft link 3 -->
+        <link name="l3_foot_ft_link">
+	    <visual>
+		<xacro:insert_mesh_l3_foot_ft_link />
+	    </visual>
+            <!-- <collision>
+                <xacro:insert_mesh_l3_foot_ft_link />
+            </collision>
+	    <inertial>
+		<xacro:insert_inertia_l3_foot_ft_link />
+	    </inertial> -->
+        </link>
+        <!-- left ft fixed joint 4 -->
+        <joint name="l4_ft_fixed" type="fixed">
+            <origin
+              xyz="0.0983224252792114 0.0168595176863209 0"
+              rpy="0 0 ${pi/2}" />
+            <axis xyz="0 0 1"/>
+            <parent link="l_ankle_roll_link"/>
+            <child link="l4_foot_ft_link"/>
+            <limit
+            lower="0"
+            upper="0"
+            effort="100"
+            velocity="100" />
+        </joint>
+        <!-- left foot ft link 4 -->
+        <link name="l4_foot_ft_link">
+	    <visual>
+		<xacro:insert_mesh_l4_foot_ft_link />
+	    </visual>
+            <!-- <collision>
+                <xacro:insert_mesh_l4_foot_ft_link />
+            </collision>
+	    <inertial>
+		<xacro:insert_inertia_l4_foot_ft_link />
+	    </inertial> -->
+        </link>
+        <!-- left ft fixed joint -->
+        <joint name="lv_ft_fixed" type="fixed">
+            <origin xyz="-0.0165 0 0.055" rpy="0 0 0"/>
+            <parent link="l4_foot_ft_link"/>
+            <child link="l_foot_v_ft_link"/>
+        </joint>
+        <!-- left foot ft link -->
+        <link name="l_foot_v_ft_link"></link>
     </xacro:macro>
 </robot>

File: huron_description/urdf/huron_right_leg.xacro (robot description, xacro)
@@ -7,5 +7,5 @@
         <joint
           name="r_hip_yaw_joint"
-          type="fixed">
+          type="revolute">
           <origin
             xyz="0.0775 0 -0.14512"
@@ -42,5 +42,5 @@
         <joint
           name="r_hip_roll_joint"
-          type="fixed">
+          type="revolute">
           <origin
             xyz="0 0 0"
@@ -214,4 +214,122 @@
             </inertial>
         </link>
+       <!-- right ft fixed joint 1 -->
+        <joint name="r1_ft_fixed" type="fixed">
+            <origin
+              xyz="0.0982708740959065 0.0143480673989493 0.127875866180863"
+              rpy="0 0 ${pi/2}" />
+            <axis xyz="0 0 1"/>
+            <parent link="r_ankle_roll_link"/>
+            <child link="r1_foot_ft_link"/>
+            <limit
+            lower="0"
+            upper="0"
+            effort="100"
+            velocity="100" />
+        </joint>
+        <!-- right foot ft link 1 -->
+        <link name="r1_foot_ft_link">
+	    <visual>
+		<xacro:insert_mesh_r1_foot_ft_link />
+	    </visual>
+            <!-- <collision>
+                <xacro:insert_mesh_r1_foot_ft_link />
+            </collision>
+	    <inertial>
+		<xacro:insert_inertia_r1_foot_ft_link />
+	    </inertial> -->
+        </link>
+        <!-- right ft fixed joint 2 -->
+        <joint name="r2_ft_fixed" type="fixed">
+            <origin
+              xyz="0.0983344633797905 -0.0206518748353312 0.127875866180863"
+              rpy="0 0 ${pi/2}" />
+            <axis xyz="0 0 1"/>
+            <parent link="r_ankle_roll_link"/>
+            <child link="r2_foot_ft_link"/>
+            <limit
+            lower="0"
+            upper="0"
+            effort="100"
+            velocity="100" />
+        </joint>
+        <!-- right foot ft link 2 -->
+        <link name="r2_foot_ft_link">
+	    <visual>
+		<xacro:insert_mesh_r2_foot_ft_link />
+	    </visual>
+            <!-- <collision>
+                <xacro:insert_mesh_r2_foot_ft_link />
+            </collision>
+	    <inertial>
+		<xacro:insert_inertia_r2_foot_ft_link />
+	    </inertial> -->
+        </link>
+        <!-- right ft fixed joint 3 -->
+        <joint name="r3_ft_fixed" type="fixed">
+            <origin
+              xyz="0.0983275192522874 -0.0168297833346846 0"
+              rpy="0 0 ${pi/2}" />
+            <axis xyz="0 0 1"/>
+            <parent link="r_ankle_roll_link"/>
+            <child link="r3_foot_ft_link"/>
+            <limit
+            lower="0"
+            upper="0"
+            effort="100"
+            velocity="100" />
+        </joint>
+        <!-- right foot ft link 3 -->
+        <link name="r3_foot_ft_link">
+	    <visual>
+		<xacro:insert_mesh_r3_foot_ft_link />
+	    </visual>
+            <!-- <collision>
+                <xacro:insert_mesh_r3_foot_ft_link />
+            </collision>
+	    <inertial>
+		<xacro:insert_inertia_r3_foot_ft_link />
+	    </inertial> -->
+        </link>
+        <!-- right ft fixed joint 4 -->
+        <joint name="r4_ft_fixed" type="fixed">
+            <origin
+              xyz="0.0982666399609057 0.0166785619632585 0"
+              rpy="0 0 ${pi/2}" />
+            <axis xyz="0 0 1"/>
+            <parent link="r_ankle_roll_link"/>
+            <child link="r4_foot_ft_link"/>
+            <limit
+            lower="0"
+            upper="0"
+            effort="100"
+            velocity="100" />
+        </joint>
+        <!-- right4 foot ft link 4 -->
+        <link name="r4_foot_ft_link">
+	    <visual>
+		<xacro:insert_mesh_r4_foot_ft_link />
+	    </visual>
+            <!-- <collision>
+                <xacro:insert_mesh_r4_foot_ft_link />
+            </collision>
+	    <inertial>
+		<xacro:insert_inertia_r4_foot_ft_link />
+	    </inertial> -->
+        </link>
+        <!-- right ft fixed joint -->
+        <joint name="rv_ft_fixed" type="fixed">
+            <origin xyz="-0.0165 0 0.055" rpy="0 0 0"/>
+            <axis xyz="0 0 0"/>
+            <parent link="r4_foot_ft_link"/>
+            <child link="r_foot_v_ft_link"/>
+            <limit
+            lower="0"
+            upper="0"
+            effort="100"
+            velocity="100" />
+        </joint>
+        <!-- right foot ft link -->
+        <link name="r_foot_v_ft_link"></link>
     </xacro:macro>
 </robot>
